File: hardware/schematic/v1.0/CLOCK_INT_N/CLOCK_INT_N.kicad_sch (KiCad schematic)
At the start: 14 parts, among them J1 Conn_Coaxial, U1 ADF4360-8, U2 OCXO-10M

Commit message: sch commit
Parts:
- added U3: ADF4002, Package_CSP:LFCSP-20-1EP_4x4mm_P0.5mm_EP2.1x2.1mm, symbol Counter:ADF4002
Changed lines of the file:
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@@
+	)
+	(symbol
+		(lib_id "Counter:ADF4002")
+		(at 212.09 50.8 0)
+		(unit 1)
+		(body_style 1)
+		(exclude_from_sim no)
+		(in_bom yes)
+		(on_board yes)
+		(in_pos_files yes)
+		(dnp no)
+		(fields_autoplaced yes)
+		(property "Reference" "U3"
+			(at 242.57 51.9998 0)
+			(show_name no)
+			(do_not_autoplace no)
+			(effects
+				(font
+					(size 1.27 1.27)
+				)
+			)
+		)
+		(property "Value" "ADF4002"
+			(at 242.57 54.5398 0)
+			(show_name no)
+			(do_not_autoplace no)
+			(effects
+				(font
+					(size 1.27 1.27)
+				)
+			)
+		)
+		(property "Footprint" "Package_CSP:LFCSP-20-1EP_4x4mm_P0.5mm_EP2.1x2.1mm"
+			(at 223.266 39.878 0)
+			(hide yes)
+			(show_name no)
+			(do_not_autoplace no)
+			(effects
+				(font
+					(size 1.27 1.27)
+				)
+			)
+		)
+		(property "Datasheet" ""
+			(at 212.09 50.8 0)
+			(hide yes)
+			(show_name no)
+			(do_not_autoplace no)
+			(effects
+				(font
+					(size 1.27 1.27)
+				)
+			)
+		)
+		(property "Description" ""
+			(at 212.09 50.8 0)
+			(hide yes)
+			(show_name no)
+			(do_not_autoplace no)
+			(effects
+				(font
+					(size 1.27 1.27)
+				)
+			)
+		)
+		(pin "5"
+		)
+		(pin "7"
+		)
+		(pin "12"
+		)
+		(pin "15"
+		)
+		(pin "9"
+		)
+		(pin "6"
+		)
+		(pin "13"
+		)
+		(pin "18"
+		)
+		(pin "20"
+		)
+		(pin "14"
+		)
+		(pin "1"
+		)
+		(pin "4"
+		)
+		(pin "2"
+		)
+		(pin "3"
+		)
+		(pin "8"
+		)
+		(pin "10"
+		)
+		(pin "16"
+		)
+		(pin "17"
+		)
+		(pin "19"
+		)
+		(pin "21"
+		)
+		(pin "11"
+		)
+		(instances
+			(project "CLOCK_INT_N"
+				(path "/6bffb4aa-8563-4398-b7a2-aaa6bc3ae230"
+					(reference "U3")
+					(unit 1)
+				)
+			)
+		)
 	)
 	(symbol

Commit message: sch
Parts:
- added C4: 100pF, symbol Device:C
- added C5: 1nF, symbol Device:C
- added C6, C7, C8, C9: (no value), symbol Device:C
- added J2: Conn_Coaxial, Connector_Coaxial:SMA_Amphenol_132289_EdgeMount, symbol Connector:Conn_Coaxial
- added R10, R9: (no value), Resistor_SMD:R_0402_1005Metric, symbol Device:R
- added R11, R12, R13: 330, Resistor_SMD:R_0402_1005Metric, symbol Device:R
- added R14, R15, R16: 10K, Resistor_SMD:R_0402_1005Metric, symbol Device:R
- added R7: 5.1K, Resistor_SMD:R_0402_1005Metric, symbol Device:R
- added R8: 0, Resistor_SMD:R_0201_0603Metric, symbol Device:R
Connections:
- net GND: now also U2.2 (GND), U3.1 (CPGND), U3.2 (AGND), U3.21 (EP), U3.3 (AGND), C4.1, C6.2, C7.2, C8.2, C9.2, J2.2 (Ext), R14.2, R15.2, R16.2, R7.1
- net VCTRL: now reaches U2.3 (VCTRL)
- net VCTRL: now also C8.1, C9.1, R10.1
- net at U3.19 (RSET): now also R7.2
- net CP: now reaches U3.20 (CP)
- net CP: now also C6.1, R10.2, R9.2
- net at U3.4 (RFINB): now also C4.2
- net 10MHZ ExtRef: now reaches U3.8 (REFIN)
- net 10MHZ ExtRef: now also R8.2
- net at U1.17 (CLK): now also R12.1, R16.1
- net at U1.18 (DATA): now also R11.1, R15.1
- net at U1.19 (LE): now also R13.2, R14.1
- new net: C5.2, J2.1 (In)
- new net: C5.1, R8.1
- new net: C7.1, R9.1
- new net CLK: R12.2
- new net DATA: R11.2
- new net LE: R13.1
Other:
- note added: "LOOP FILTER"

Commit message: sch commit
Parts:
- added R17, R18, R19: 330, Resistor_SMD:R_0402_1005Metric, symbol Device:R
- added R20, R21, R22: 10K, Resistor_SMD:R_0402_1005Metric, symbol Device:R
Connections:
- net CLK: now also R18.2
- net DATA: now also R17.2
- net GND: now also R20.1, R21.1, R22.1
- net LE: now also R19.2
- net at U3.12 (CLK): now also R18.1, R20.2
- net at U3.13 (DATA): now also R17.1, R21.2
- net at U3.14 (LE): now also R19.1, R22.2
