File: hardware/schematic/v1.0/CLOCK/CLOCK.kicad_sch (KiCad schematic)
At the start: 11 parts, among them J1 Conn_Coaxial, J2 Conn_Coaxial, J3 Conn_Coaxial, J4 Conn_Coaxial, J5 Conn_Coaxial, U1 LMK5B12204, U2 LMK1C1102

Commit message: Update schematic and configuration files
Parts:
- added C1, C2, C3, C4: 100nF, Capacitor_SMD:C_0402_1005Metric, symbol Device:C
- added R3, R6: Open, symbol Device:R
- added R4, R5, R7, R8: 49.9, symbol Device:R
- added R9: 0, Resistor_SMD:R_0402_1005Metric, symbol Device:R
Connections:
- net GND: now also J2.2 (Ext), J3.2 (Ext), J4.2 (Ext), J5.2 (Ext), U1.49 (EPAD), U1.8 (REFSEL), R4.2, R5.1, R7.2, R8.1, R9.1
- net CAP_DIG: now reaches U1.3 (CAP_DIG)
- net XO_P: now reaches U1.31 (XO_P)
- net XO_N: now reaches U1.32 (XO_N)
- net VDD_DIG: now reaches U1.4 (VDD_DIG)
- net OUT2_N: now reaches U1.41 (OUT2_N)
- net OUT2_N: now also C2.1, R3.2
- net OUT2_P: now reaches U1.42 (OUT2_P)
- net OUT2_P: now also C1.1, R3.1
- net OUT3_N: now reaches U1.44 (OUT3_N)
- net OUT3_N: now also C4.1, R6.2
- net OUT3_P: now reaches U1.45 (OUT3_P)
- net OUT3_P: now also C3.1, R6.1
- net VDD_IN: now reaches U1.5 (VDD_IN)
- net at U1.9 (HW_SW_CTRL): now also R9.2
- net at J2.1 (In): now also C1.2, R4.1
- net at J4.1 (In): now also C3.2, R7.1
- net at J3.1 (In): now also C2.2, R5.2
- net at J5.1 (In): now also C4.2, R8.2
- no-connect marks 6 -> 10
Other:
- moved on the sheet: J2, J3

Commit message: Update schematic files and remove lock file
Parts:
- added C5: 100nF, Capacitor_SMD:C_0402_1005Metric, symbol Device:C
Connections:
- net GND: now also J1.2 (Ext)
- net at J1.1 (In): now also C5.1
Changed lines of the file:
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@@
 	(wire
 		(pts
+			(xy 50.8 77.47) (xy 52.07 77.47)
+		)
+		(stroke
+			(width 0)
+			(type default)
+		)
+	)
+	(wire
+		(pts
 			(xy 224.79 92.71) (xy 229.87 92.71)
 		)
@@
 	)
 	(symbol
+		(lib_id "Device:C")
+		(at 55.88 77.47 90)
+		(unit 1)
+		(body_style 1)
+		(exclude_from_sim no)
+		(in_bom yes)
+		(on_board yes)
+		(in_pos_files yes)
+		(dnp no)
+		(fields_autoplaced yes)
+		(property "Reference" "C5"
+			(at 55.88 69.85 90)
+			(show_name no)
+			(do_not_autoplace no)
+			(effects
+				(font
+					(size 1.27 1.27)
+				)
+			)
+		)
+		(property "Value" "100nF"
+			(at 55.88 72.39 90)
+			(show_name no)
+			(do_not_autoplace no)
+			(effects
+				(font
+					(size 1.27 1.27)
+				)
+			)
+		)
+		(property "Footprint" "Capacitor_SMD:C_0402_1005Metric"
+			(at 59.69 76.5048 0)
+			(hide yes)
+			(show_name no)
+			(do_not_autoplace no)
+			(effects
+				(font
+					(size 1.27 1.27)
+				)
+			)
+		)
+		(property "Datasheet" ""
+			(at 55.88 77.47 0)
+			(hide yes)
+			(show_name no)
+			(do_not_autoplace no)
+			(effects
+				(font
+					(size 1.27 1.27)
+				)
+			)
+		)
+		(property "Description" "Unpolarized capacitor"
+			(at 55.88 77.47 0)
+			(hide yes)
+			(show_name no)
+			(do_not_autoplace no)
+			(effects
+				(font
+					(size 1.27 1.27)
+				)
+			)
+		)
+		(pin "1"
+		)
+		(pin "2"
+		)
+		(instances
+			(project "CLOCK"
+				(path "/a8714d66-6565-4fb4-a698-a884e68083d2"
+					(reference "C5")
+					(unit 1)
+				)
+			)
+		)
+	)
+	(symbol
 		(lib_id "power:GND")
 		(at 242.57 54.61 0)
@@
 					(unit 1)
 				)
+			)
+		)
+	)
+	(symbol
+		(lib_id "power:GND")
+		(at 45.72 82.55 0)
+		(unit 1)
+		(body_style 1)
+		(exclude_from_sim no)
+		(in_bom yes)
+		(on_board yes)
+		(in_pos_files yes)
+		(dnp no)
+		(fields_autoplaced yes)
+		(property "Reference" "#PWR013"
+			(at 45.72 88.9 0)
+			(hide yes)
+			(show_name no)
+			(do_not_autoplace no)
+			(effects
+				(font
+					(size 1.27 1.27)
+				)
+			)
+		)
+		(property "Value" "GND"
+			(at 45.72 87.63 0)
+			(show_name no)
+			(do_not_autoplace no)
+			(effects
+				(font
+					(size 1.27 1.27)
+				)
+			)
+		)
+		(property "Footprint" ""
+			(at 45.72 82.55 0)
+			(hide yes)
+			(show_name no)
+			(do_not_autoplace no)
+			(effects
+				(font
+					(size 1.27 1.27)
+				)
+			)
+		)
+		(property "Datasheet" ""
+			(at 45.72 82.55 0)
+			(hide yes)
+			(show_name no)
+			(do_not_autoplace no)
+			(effects
+				(font
+					(size 1.27 1.27)
+				)
+			)
+		)
+		(property "Description" "Power symbol creates a global label with name \"GND\" , ground"
+			(at 45.72 82.55 0)
+			(hide yes)
+			(show_name no)
+			(do_not_autoplace no)
+			(effects
+				(font
+					(size 1.27 1.27)
+				)
+			)
+		)
+		(pin "1"
+		)
+		(instances
+			(project "CLOCK"
+				(path "/a8714d66-6565-4fb4-a698-a884e68083d2"
+					(reference "#PWR013")
+					(unit 1)
+				)

Commit message: sch commit
Parts:
- added R10, R12: 10K, Resistor_SMD:R_0402_1005Metric, symbol Device:R
- added R11, R13: 0, Resistor_SMD:R_0402_1005Metric, symbol Device:R
- added R14, R15: 1K, Resistor_SMD:R_0402_1005Metric, symbol Device:R
- added U3: LMK1C1102, Package_SON:WSON-8-1EP_2x2mm_P0.5mm_EP0.9x1.6mm, symbol Counter:LMK1C1102
Connections:
- net +3.3V: now also R10.2, R12.2, R14.1
- net GND: now also U2.4 (GND), R13.1, R15.1, U3.4 (GND)
- net PRIREF_N: now also R13.2
- net PRIREF_P: now also R14.2, R15.2, U3.3 (Y0)
- net at U2.2 (1G): now also R10.1
- net at U2.8 (Y1): now also R11.1
- new net: R12.1, U3.2 (1G)
- new net: R11.2, U3.1 (CLKIN)
- no-connect marks 10 -> 15
Other:
- moved on the sheet: C5, D1, D2, J1, R1, R2, R9, U1, U2

Commit message: sch update commit
Parts:
- added C10, C7: 1uF, Capacitor_SMD:C_0402_1005Metric, symbol Device:C
- added C11, C8: 100nF, Capacitor_SMD:C_0402_1005Metric, symbol Device:C
- added C6, C9: 10uF, Capacitor_SMD:C_0402_1005Metric, symbol Device:C
- added FB1, FB2: 80 ohm@100mhz, Inductor_SMD:L_0603_1608Metric, symbol Device:FerriteBead_Small
- added J6: Conn_Coaxial, Connector_Coaxial:SMA_Amphenol_132289_EdgeMount, symbol Connector:Conn_Coaxial
- added R16, R17, R19, R20: 1K, Resistor_SMD:R_0402_1005Metric, symbol Device:R
- added R18, R21: 0, Resistor_SMD:R_0402_1005Metric, symbol Device:R
- renumbered D2 to D1, D1 to D2
Connections:
- net +3.3V: now also C6.2, C9.2, FB1.1, FB2.1, R16.2, R19.2
- net GND: now also C10.1, C11.1, C6.1, C7.1, C8.1, C9.1, J6.2 (Ext), R17.1, R20.1
- net OUT3_N: no longer C4.1
- net at J5.1 (In), R8.2: no longer C4.2
- net at U3.6 (VDD): now also C10.2, C11.2, FB2.2
- net at U2.1 (CLKIN): now also R18.1
- net at U2.3 (Y0): now also R19.1, R20.2, R21.1
- net at U2.6 (VDD): now also C7.2, C8.2, FB1.2
- net at C5.2: now also R16.1, R17.2, R18.2
- new net: J6.1 (In), R21.2
Other:
- note added: "10MHZ REF IN"
- note added: "10MHZ REF OUT"
- moved on the sheet: C4, C5, J1, R10, R11, R12, R13, R14, R15, U2, U3

Commit message: sch update commit
Parts:
- added C12, C13, C14, C15, C17, C18, C19, C27: 100nF, Capacitor_SMD:C_0402_1005Metric, symbol Device:C
- added C16: 1uF, Capacitor_SMD:C_0402_1005Metric, symbol Device:C
- added C20, C21, C22, C23, C24, C25: 10uF, Capacitor_SMD:C_0402_1005Metric, symbol Device:C
- added C26: 470nF, Capacitor_SMD:C_0402_1005Metric, symbol Device:C
- added FB3, FB4, FB5: 600 ohm@100mhz, symbol Device:FerriteBead_Small
- added FB6: 80 ohm@100mhz, symbol Device:FerriteBead_Small
- added J10, J7, J8, J9: Conn_Coaxial, symbol Connector:Conn_Coaxial
- added R22, R23: Open, symbol Device:R
- added R24, R25, R26, R27: 49.9, symbol Device:R
- FB1: value 80 ohm@100mhz -> 600 ohm@100mhz; footprint Inductor_SMD:L_0603_1608Metric -> (none)
Connections:
- net +3.3V: now also C16.2, C17.2, C18.2, C19.2, FB3.1, FB4.1, FB5.1, FB6.1
- net CAP_DIG: now also C23.2
- net GND: now also C16.1, C17.1, C18.1, C19.1, C20.1, C21.1, C22.1, C23.1, C24.1, C25.1, C26.1, C27.1, J10.2 (Ext), J7.2 (Ext), J8.2 (Ext), J9.2 (Ext), R24.2, R25.2, R26.1, R27.1
- net OUT3_N: now also C4.2
- net at J5.1 (In), R8.2: now also C4.1
- net at C7.2, C8.2, U2.6 (VDD): now also FB6.2; no longer FB1.2
- net OUT0_N: now reaches U1.16 (OUT0_N)
- net OUT0_N: now also C13.1, R22.2
- net OUT0_P: now reaches U1.17 (OUT0_P)
- net OUT0_P: now also C12.1, R22.1
- net OUT1_P: now reaches U1.20 (OUT1_P)
- net OUT1_P: now also C14.1, R23.1
- net OUT1_N: now reaches U1.21 (OUT1_N)
- net OUT1_N: now also C15.2, R23.2
- net VDD_PLL1: now reaches U1.27 (VDD_PLL1)
- net CAP_PLL1: now reaches U1.28 (CAP_PLL1)
- net CAP_PLL1: now also C24.2
- net LF1: now reaches U1.29 (LF1)
- net LF1: now also C26.2
- net LF2: now reaches U1.34 (LF2)
- net LF2: now also C27.2
- net CAP_PLL2: now reaches U1.35 (CAP_PLL2)
- net CAP_PLL2: now also C25.2
- net VDD_PLL2: now reaches U1.36 (VDD_PLL2)
- new net: C15.1, J10.1 (In), R27.2
- new net: C14.2, J9.1 (In), R25.1
- new net: C12.2, J7.1 (In), R24.1
- new net: C13.2, J8.1 (In), R26.2
- new net VDD: C20.2, FB3.2
- new net VDDDIG: FB1.2
- new net VDDO0_1: C21.2, FB4.2
- new net VDDO2_3: C22.2, FB5.2
Other:
- moved on the sheet: C1, C2, C3, C4, D1, D2, J2, J3, J4, J5, R1, R2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

Commit message: sch update commit
Parts:
- added C28, C29, C30, C31, C32, C33, C34, C35, C36, C37: 100nF, Capacitor_SMD:C_0402_1005Metric, symbol Device:C
Connections:
- net VDDO_0 is gone; now on net VDDO0_1: U1.18 (VDDO_0)
- net VDDO_1 is gone; now on net VDDO0_1: U1.19 (VDDO_1)
- net VDDO_2 is gone; now on net VDDO2_3: U1.37 (VDDO_2), U1.40 (VDDO_2)
- net VDDO_3 is gone; now on net VDDO2_3: U1.43 (VDDO_3), U1.46 (VDDO_3)
- net VDD_DIG is gone; now on net VDDDIG: U1.4 (VDD_DIG)
- net VDD_IN is gone; now on net VDD: U1.5 (VDD_IN)
- net VDD_PLL1 is gone; now on net VDD: U1.27 (VDD_PLL1)
- net VDD_PLL2 is gone; now on net VDD: U1.36 (VDD_PLL2)
- net GND: now also C28.1, C29.1, C30.1, C31.1, C32.1, C33.1, C34.1, C35.1, C36.1, C37.1
- net VDD: now also C29.2, C30.2, C31.2
- net VDDDIG: now also C28.2
- net VDDO0_1: now also C32.2, C33.2
- net VDDO2_3: now also C34.2, C35.2, C36.2, C37.2
Other:
- note added: "10MHZ Ext Ref"
- moved on the sheet: C1, C10, C11, C12, C13, C14, C15, C2, C3, C4, C5, C6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

Commit message: sch update
Parts:
- added C38: 2.2uF, Capacitor_SMD:C_0603_1608Metric, symbol Device:C
- added C39: 10nF, Capacitor_SMD:C_0402_1005Metric, symbol Device:C
- added C40: 1uF, Capacitor_SMD:C_0402_1005Metric, symbol Device:C
- added C41: 100nF, Capacitor_SMD:C_0402_1005Metric, symbol Device:C
- added J11: USB_C_Receptacle_USB2.0_16P, Connector_USB:USB_C_Receptacle_Palconn_UTC16-G, symbol Connector:USB_C_Receptacle_USB2.0_16P
- added J12: Conn_01x04_Socket, Connector_PinSocket_2.54mm:PinSocket_1x04_P2.54mm_Vertical, symbol Connector:Conn_01x04_Socket
- added J13: Conn_01x10_Socket, Connector_PinSocket_2.54mm:PinSocket_1x10_P2.54mm_Vertical, symbol Connector:Conn_01x10_Socket
- added R28: 0, Resistor_SMD:R_0402_1005Metric, symbol Device:R
- added U4: TPS78633, Package_TO_SOT_SMD:SOT-223-6, symbol Counter:TPS78633
Connections:
- net +3.3V: now also C40.1, C41.1, J12.1 (Pin_1), J12.2 (Pin_2), U4.4 (OUT)
- net GND: now also C38.1, C39.2, C40.2, C41.2, J12.3 (Pin_3), J12.4 (Pin_4), J13.10 (Pin_10), J13.9 (Pin_9), U4.3 (GND), U4.6 (TAB)
- net GPIO0: now also J13.3 (Pin_3)
- net GPIO1: now also J13.4 (Pin_4)
- net PDN: now also J13.5 (Pin_5)
- net SCL: now also J13.2 (Pin_2)
- net SDA: now also J13.1 (Pin_1)
- net SIG_2: now reaches R12.1, U3.2 (1G)
- net SIG_1: now reaches R10.1, U2.2 (1G)
- new net: C38.2, R28.2, U4.1 (EN)
- new net: C39.1, U4.5 (NR/FB)
- new net: J11.A1 (GND), J11.A12 (GND), J11.B1 (GND), J11.B12 (GND)
- new net: J11.A4 (VBUS), J11.A9 (VBUS), J11.B4 (VBUS), J11.B9 (VBUS)
- new net +5V: R28.1, U4.2 (IN)
Other:
- note added: "SOCKET"
- note added: "USB C"
- moved on the sheet: C21, R10, R12

Commit message: sch update
Parts:
- added C42: 2.2uF, Capacitor_SMD:C_0603_1608Metric, symbol Device:C
- added C43: 10nF, Capacitor_SMD:C_0402_1005Metric, symbol Device:C
- added C44: 1uF, Capacitor_SMD:C_0402_1005Metric, symbol Device:C
- added C45, C46: 100nF, Capacitor_SMD:C_0402_1005Metric, symbol Device:C
- added C47: 10uF, Capacitor_SMD:C_0402_1005Metric, symbol Device:C
- added R29: 0, Resistor_SMD:R_0402_1005Metric, symbol Device:R
- added R30, R31: 5.1K, Resistor_SMD:R_0402_1005Metric, symbol Device:R
- added U5: TPS78633, Package_TO_SOT_SMD:SOT-223-6, symbol Counter:TPS78633
- added U6: OCXO-10M, Connector:Joint-Tech_C5080WR-04P_1x04_P5.08mm_Vertical, symbol Counter:OCXO-10M
Connections:
- net +5V is gone; now on net VBUS: R28.1, U4.2 (IN)
- net +3.3V: now also C44.1, C45.1, U5.4 (OUT), U6.5 (VCC)
- net GND: now also J11.A1 (GND), J11.A12 (GND), J11.B1 (GND), J11.B12 (GND), J11.SH (SHIELD), C42.1, C43.2, C44.2, C45.2, C46.2, C47.1, R30.2, R31.1, U5.3 (GND), U5.6 (TAB), U6.2 (GND)
- net VBUS: now reaches J11.A4 (VBUS), J11.A9 (VBUS), J11.B4 (VBUS), J11.B9 (VBUS)
- net VBUS: now also C46.1, C47.2, R29.1, U5.2 (IN)
- net at J11.A5 (CC1): now also R30.1
- net at J11.B5 (CC2): now also R31.2
- new net: C42.2, R29.2, U5.1 (EN)
- new net: C43.1, U5.5 (NR/FB)
- no-connect marks 15 -> 21
Other:
- note added: "OCXO"
- moved on the sheet: J11
