File: hardware/schematic/v1.0/CLOCK/CLOCK.kicad_sch (KiCad schematic)
At the start: 105 parts, among them J1 Conn_Coaxial, J10 Conn_Coaxial, J11 USB_C_Receptacle_USB2.0_16P, J12 Conn_01x04_Socket, J13 Conn_01x10_Socket, J2 Conn_Coaxial, J3 Conn_Coaxial, J4 Conn_Coaxial, J5 Conn_Coaxial, J6 Conn_Coaxial, J7 Conn_Coaxial, J8 Conn_Coaxial, J9 Conn_Coaxial, U1 LMK5B12204, U2 LMK1C1102, U3 LMK1C1102, U4 TPS78633, U5 TPS78633, U6 OCXO-10M

Commit message: sch update
Connections:
- net GPIO2: now also J13.5 (Pin_5)
- net PDN: now also J13.6 (Pin_6); no longer J13.5 (Pin_5)
- net STATUS0: now also J13.7 (Pin_7)
- net STATUS1: now also J13.8 (Pin_8)
- net VDD: now also U1.33 (VDD_XO)
Changed lines of the file:
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@@
 	(wire
 		(pts
+			(xy 193.04 232.41) (xy 194.31 232.41)
+		)
+		(stroke
+			(width 0)
+			(type default)
+		)
+	)
+	(wire
+		(pts
 			(xy 293.37 113.03) (xy 306.07 113.03)
 		)
@@
 	(wire
 		(pts
+			(xy 193.04 234.95) (xy 194.31 234.95)
+		)
+		(stroke
+			(width 0)
+			(type default)
+		)
+	)
+	(wire
+		(pts
 			(xy 113.03 227.33) (xy 113.03 226.06)
 		)
@@
 	(wire
 		(pts
+			(xy 193.04 229.87) (xy 194.31 229.87)
+		)
+		(stroke
+			(width 0)
+			(type default)
+		)
+	)
+	(wire
+		(pts
 			(xy 125.73 31.75) (xy 125.73 33.02)
 		)
@@
 		)
 	)
+	(global_label "VDD"
+		(shape input)
+		(at 170.18 87.63 0)
+		(fields_autoplaced yes)
+		(effects
+			(font
+				(size 1.27 1.27)
+			)
+			(justify left)
+		)
+		(property "Intersheetrefs" "${INTERSHEET_REFS}"
+			(at 176.7938 87.63 0)
+			(hide yes)
+			(show_name no)
+			(do_not_autoplace no)
+			(effects
+				(font
+					(size 1.27 1.27)
+				)
+				(justify left)
+			)
+		)
+	)
 	(global_label "OUT2_N"
 		(shape input)
@@
 		)
 	)
+	(global_label "STATUS0"
+		(shape input)
+		(at 193.04 232.41 180)
+		(fields_autoplaced yes)
+		(effects
+			(font
+				(size 1.27 1.27)
+			)
+			(justify right)
+		)
+		(property "Intersheetrefs" "${INTERSHEET_REFS}"
+			(at 182.072 232.41 0)
+			(hide yes)
+			(show_name no)
+			(do_not_autoplace no)
+			(effects
+				(font
+					(size 1.27 1.27)
+				)
+				(justify right)
+			)
+		)
+	)
 	(global_label "VDDO_1"
 		(shape input)
@@
 		)
 	)
+	(global_label "PDN"
+		(shape output)
+		(at 193.04 229.87 180)
+		(fields_autoplaced yes)
+		(effects
+			(font
+				(size 1.27 1.27)
+			)
+			(justify right)
+		)
+		(property "Intersheetrefs" "${INTERSHEET_REFS}"
+			(at 186.1843 229.87 0)
+			(hide yes)
+			(show_name no)
+			(do_not_autoplace no)
+			(effects
+				(font
+					(size 1.27 1.27)
+				)
+				(justify right)
+			)
+		)
+	)
 	(global_label "VDD"
 		(shape output)
@@
 		)
 	)
+	(global_label "STATUS1"
+		(shape input)
+		(at 193.04 234.95 180)
+		(fields_autoplaced yes)
+		(effects
+			(font
+				(size 1.27 1.27)
+			)
+			(justify right)
+		)
+		(property "Intersheetrefs" "${INTERSHEET_REFS}"
+			(at 182.072 234.95 0)
+			(hide yes)
+			(show_name no)
+			(do_not_autoplace no)
+			(effects
+				(font
+					(size 1.27 1.27)
+				)
+				(justify right)
+			)
+		)
+	)
 	(global_label "CAP_DIG"
 		(shape input)
@@
 		)
 	)
-	(global_label "PDN"
+	(global_label "GPIO2"
 		(shape output)
 		(at 193.04 227.33 180)
@@
 		)
 		(property "Intersheetrefs" "${INTERSHEET_REFS}"
-			(at 186.1843 227.33 0)
+			(at 184.37 227.33 0)
 			(hide yes)
 			(show_name no)

Commit message: sch update
Parts:
- removed J12: Conn_01x04_Socket, Connector_PinSocket_2.54mm:PinSocket_1x04_P2.54mm_Vertical, symbol Connector:Conn_01x04_Socket
- removed J13: Conn_01x10_Socket, Connector_PinSocket_2.54mm:PinSocket_1x10_P2.54mm_Vertical, symbol Connector:Conn_01x10_Socket
- added J14: Conn_01x16_Socket, Connector_PinSocket_2.54mm:PinSocket_1x16_P2.54mm_Vertical, symbol Connector:Conn_01x16_Socket
Connections:
- net +3.3V: now also J14.3 (Pin_3), J14.4 (Pin_4)
- net GND: now also J14.5 (Pin_5), J14.6 (Pin_6)
- net GPIO0: now also J14.9 (Pin_9)
- net GPIO1: now also J14.10 (Pin_10)
- net GPIO2: now also J14.11 (Pin_11)
- net PDN: now also J14.12 (Pin_12)
- net SCL: now also J14.8 (Pin_8)
- net SDA: now also J14.7 (Pin_7)
- net STATUS0: now also J14.13 (Pin_13)
- net STATUS1: now also J14.14 (Pin_14)
- net VBUS renamed +5V
- net +5V: now also J14.1 (Pin_1), J14.2 (Pin_2)

Commit message: sch update
Parts:
- U6: footprint Connector:Joint-Tech_C5080WR-04P_1x04_P5.08mm_Vertical -> Counter:DOPFITKR2-10M
Connections:
- net XO_N is gone; now on net GND: U1.32 (XO_N)
- net XO_P: now also U6.1 (RF)
Changed lines of the file:
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@@
 	(wire
 		(pts
+			(xy 304.8 213.36) (xy 323.85 213.36)
+		)
+		(stroke
+			(width 0.508)
+			(type default)
+		)
+	)
+	(wire
+		(pts
 			(xy 66.04 201.93) (xy 66.04 213.36)
 		)
@@
 	(wire
 		(pts
+			(xy 312.42 215.9) (xy 312.42 222.25)
+		)
+		(stroke
+			(width 0)
+			(type default)
+		)
+	)
+	(wire
+		(pts
 			(xy 143.51 121.92) (xy 143.51 123.19)
 		)
@@
 		)
 	)
+	(wire
+		(pts
+			(xy 304.8 215.9) (xy 312.42 215.9)
+		)
+		(stroke
+			(width 0)
+			(type default)
+		)
+	)
 	(polyline
 		(pts
@@
 		)
 	)
+	(global_label "XO_P"
+		(shape output)
+		(at 304.8 213.36 180)
+		(fields_autoplaced yes)
+		(effects
+			(font
+				(size 1.27 1.27)
+			)
+			(justify right)
+		)
+		(property "Intersheetrefs" "${INTERSHEET_REFS}"
+			(at 297.0372 213.36 0)
+			(hide yes)
+			(show_name no)
+			(do_not_autoplace no)
+			(effects
+				(font
+					(size 1.27 1.27)
+				)
+				(justify right)
+			)
+		)
+	)
 	(global_label "VDDO_3"
 		(shape input)
@@
 		)
 	)
+	(global_label "XO_N"
+		(shape output)
+		(at 304.8 215.9 180)
+		(fields_autoplaced yes)
+		(effects
+			(font
+				(size 1.27 1.27)
+			)
+			(justify right)
+		)
+		(property "Intersheetrefs" "${INTERSHEET_REFS}"
+			(at 296.9767 215.9 0)
+			(hide yes)
+			(show_name no)
+			(do_not_autoplace no)
+			(effects
+				(font
+					(size 1.27 1.27)
+				)
+				(justify right)
+			)
+		)
+	)
 	(global_label "OUT3_N"
 		(shape output)
@@
 	)
 	(symbol
+		(lib_id "Counter:OCXO-10M")
+		(at 332.74 217.17 0)
+		(unit 1)
+		(body_style 1)
+		(exclude_from_sim no)
+		(in_bom yes)
+		(on_board yes)
+		(in_pos_files yes)
+		(dnp no)
+		(fields_autoplaced yes)
+		(property "Reference" "U6"
+			(at 332.74 205.74 0)
+			(show_name no)
+			(do_not_autoplace no)
+			(effects
+				(font
+					(size 1.27 1.27)
+				)
+			)
+		)
+		(property "Value" "OCXO-10M"
+			(at 332.74 208.28 0)
+			(show_name no)
+			(do_not_autoplace no)
+			(effects
+				(font
+					(size 1.27 1.27)
+				)
+			)
+		)
+		(property "Footprint" "Counter:DOPFITKR2-10M"
+			(at 332.74 217.17 0)
+			(hide yes)
+			(show_name no)
+			(do_not_autoplace no)
+			(effects
+				(font
+					(size 1.27 1.27)
+				)
+			)
+		)
+		(property "Datasheet" ""
+			(at 332.74 217.17 0)
+			(hide yes)
+			(show_name no)
+			(do_not_autoplace no)
+			(effects
+				(font
+					(size 1.27 1.27)
+				)
+			)
+		)
+		(property "Description" ""
+			(at 332.74 217.17 0)
+			(hide yes)
+			(show_name no)
+			(do_not_autoplace no)
+			(effects
+				(font
+					(size 1.27 1.27)
+				)
+			)
+		)
+		(pin "3"
+		)
+		(pin "2"
+		)
+		(pin "1"
+		)
+		(pin "5"
+		)
+		(pin "4"
+		)
+		(instances
+			(project "CLOCK"
+				(path "/a8714d66-6565-4fb4-a698-a884e68083d2"
+					(reference "U6")
+					(unit 1)
+				)
+			)
+		)
+	)
+	(symbol
 		(lib_id "power:GND")
 		(at 311.15 96.52 0)
@@
 	(symbol
 		(lib_id "power:GND")
+		(at 312.42 222.25 0)
+		(unit 1)
+		(body_style 1)
+		(exclude_from_sim no)
+		(in_bom yes)
+		(on_board yes)
+		(in_pos_files yes)
+		(dnp no)
+		(fields_autoplaced yes)
+		(property "Reference" "#PWR0113"
+			(at 312.42 228.6 0)
+			(hide yes)
+			(show_name no)
+			(do_not_autoplace no)
+			(effects
+				(font
+					(size 1.27 1.27)
+				)
+			)
+		)
+		(property "Value" "GND"
+			(at 312.42 227.33 0)
+			(hide yes)
+			(show_name no)
+			(do_not_autoplace no)
+			(effects
+				(font
+					(size 1.27 1.27)
+				)
+			)
+		)
+		(property "Footprint" ""
+			(at 312.42 222.25 0)
+			(hide yes)
+			(show_name no)
+			(do_not_autoplace no)
+			(effects
+				(font
+					(size 1.27 1.27)
+				)
+			)
+		)
+		(property "Datasheet" ""
+			(at 312.42 222.25 0)
+			(hide yes)
+			(show_name no)
+			(do_not_autoplace no)
+			(effects
+				(font
+					(size 1.27 1.27)
+				)
+			)
+		)
+		(property "Description" "Power symbol creates a global label with name \"GND\" , ground"
+			(at 312.42 222.25 0)
+			(hide yes)
+			(show_name no)
+			(do_not_autoplace no)
+			(effects
+				(font
+					(size 1.27 1.27)
+				)
+			)
+		)
+		(pin "1"
+		)
+		(instances
+			(project "CLOCK"
+				(path "/a8714d66-6565-4fb4-a698-a884e68083d2"
+					(reference "#PWR0113")
+					(unit 1)
+				)
+			)
+		)
+	)
+	(symbol
+		(lib_id "power:GND")
 		(at 300.99 82.55 180)
 		(unit 1)
@@
 					(unit 1)
 				)
-			)
-		)
-	)
-	(symbol
-		(lib_id "Counter:OCXO-10M")
-		(at 332.74 217.17 0)
-		(unit 1)
-		(body_style 1)
-		(exclude_from_sim no)
-		(in_bom yes)
-		(on_board yes)
-		(in_pos_files yes)
-		(dnp no)
-		(fields_autoplaced yes)
-		(property "Reference" "U6"
-			(at 332.74 205.74 0)
-			(show_name no)
-			(do_not_autoplace no)
-			(effects
-				(font
-					(size 1.27 1.27)
-				)
-			)
-		)
-		(property "Value" "OCXO-10M"
-			(at 332.74 208.28 0)
-			(show_name no)
-			(do_not_autoplace no)
-			(effects
-				(font
-					(size 1.27 1.27)
-				)
-			)
-		)
-		(property "Footprint" "Connector:Joint-Tech_C5080WR-04P_1x04_P5.08mm_Vertical"
-			(at 332.74 217.17 0)
-			(hide yes)
-			(show_name no)
-			(do_not_autoplace no)
-			(effects
-				(font
-					(size 1.27 1.27)
-				)
-			)
-		)
-		(property "Datasheet" ""
-			(at 332.74 217.17 0)
-			(hide yes)
-			(show_name no)
-			(do_not_autoplace no)
-			(effects
-				(font
-					(size 1.27 1.27)
-				)
-			)
-		)
-		(property "Description" ""
-			(at 332.74 217.17 0)
-			(hide yes)
-			(show_name no)
-			(do_not_autoplace no)
-			(effects
-				(font
-					(size 1.27 1.27)
-				)
-			)
-		)
-		(pin "1"
-		)
-		(pin "4"
-		)
-		(pin "3"
-		)
-		(pin "5"
-		)
-		(pin "2"
-		)
-		(instances
-			(project "CLOCK"
-				(path "/a8714d66-6565-4fb4-a698-a884e68083d2"
-					(reference "U6")
-					(unit 1)
-				)

Commit message: sch update
Parts:
- added C48: 10uF, Capacitor_SMD:C_0603_1608Metric, symbol Device:C
- added C49, C51: 100nF, Capacitor_SMD:C_0402_1005Metric, symbol Device:C
- added C50: 1uF, Capacitor_SMD:C_0402_1005Metric, symbol Device:C
- added R32: 3296W-1-103_C48997937, Counter:3296W-1-103_C48997937, symbol Counter:3296W-1-103_C48997937
- added R33: 1K, Resistor_SMD:R_0402_1005Metric, symbol Device:R
- FB1, FB3, FB4, FB5: value 600 ohm@100mhz -> 220 ohm@100mhz
Connections:
- net +3.3V: now also C48.2, C49.1, C50.2
- net GND: now also C48.1, C49.2, C50.1, C51.2, R32.1
- net at U6.3 (VCTRL): now also C51.1, R33.2
- net at U6.4 (VREF): now also R32.3
- new net: R32.2, R33.1
Other:
- note added: "50 OHM TRACE"

Commit message: sch update
Parts:
- added H1: HX_PH254-01-03-Z-L11_5_PCB_PIN_HEADER, Counter:HX_PH254-01-03-Z-L11_5_PCB_PIN_HEADER, symbol JLCImport:HX_PH254-01-03-Z-L11_5_PCB_PIN_HEADER
- C44: value 1uF -> 10uF; footprint Capacitor_SMD:C_0402_1005Metric -> Capacitor_SMD:C_0805_2012Metric
Connections:
- net +3.3V: no longer C44.1, C45.1, C48.2, C49.1, C50.2, U5.4 (OUT), U6.5 (VCC)
- net +5V: now also H1.3
- new net: C48.2, C49.1, C50.2, H1.2, U6.5 (VCC)
- new net +3.3V_OCXO: C44.1, C45.1, H1.1, U5.4 (OUT)
- no-connect marks 21 -> 23
Other:
- moved on the sheet: C42, C43, C44, C45, R29, U5

Commit message: sch update
Parts:
- added TP1: Volt TestPoint, TestPoint:TestPoint_Loop_D1.80mm_Drill1.0mm_Beaded, symbol Connector:TestPoint
Connections:
- net at C48.2, C49.1, C50.2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: now also TP1.1
Changed lines of the file:
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@@
 	)
 	(junction
+		(at 342.9 213.36)
+		(diameter 0)
+		(color 0 0 0 0)
+	)
+	(junction
 		(at 265.43 191.77)
 		(diameter 0)
@@
 	(wire
 		(pts
+			(xy 342.9 213.36) (xy 346.71 213.36)
+		)
+		(stroke
+			(width 0)
+			(type default)
+		)
+	)
+	(wire
+		(pts
 			(xy 341.63 227.33) (xy 344.17 227.33)
 		)
@@
 	(wire
 		(pts
+			(xy 342.9 200.66) (xy 342.9 213.36)
+		)
+		(stroke
+			(width 0)
+			(type default)
+		)
+	)
+	(wire
+		(pts
 			(xy 43.18 118.11) (xy 43.18 119.38)
 		)
@@
 	(wire
 		(pts
-			(xy 341.63 213.36) (xy 346.71 213.36)
+			(xy 341.63 213.36) (xy 342.9 213.36)
 		)
 		(stroke
@@
 					(unit 1)
 				)
+			)
+		)
+	)
+	(symbol
+		(lib_id "Connector:TestPoint")
+		(at 342.9 200.66 0)
+		(unit 1)
+		(body_style 1)
+		(exclude_from_sim no)
+		(in_bom yes)
+		(on_board yes)
+		(in_pos_files yes)
+		(dnp no)
+		(fields_autoplaced yes)
+		(property "Reference" "TP1"
+			(at 345.44 196.0879 0)
+			(show_name no)
+			(do_not_autoplace no)
+			(effects
+				(font
+					(size 1.27 1.27)
+				)
+				(justify left)
+			)
+		)
+		(property "Value" "Volt TestPoint"
+			(at 345.44 198.6279 0)
+			(show_name no)
+			(do_not_autoplace no)
+			(effects
+				(font
+					(size 1.27 1.27)
+				)
+				(justify left)
+			)
+		)
+		(property "Footprint" "TestPoint:TestPoint_Loop_D1.80mm_Drill1.0mm_Beaded"
+			(at 347.98 200.66 0)
+			(hide yes)
+			(show_name no)
+			(do_not_autoplace no)
+			(effects
+				(font
+					(size 1.27 1.27)
+				)
+			)
+		)
+		(property "Datasheet" ""
+			(at 347.98 200.66 0)
+			(hide yes)
+			(show_name no)
+			(do_not_autoplace no)
+			(effects
+				(font
+					(size 1.27 1.27)
+				)
+			)
+		)
+		(property "Description" "test point"
+			(at 342.9 200.66 0)
+			(hide yes)
+			(show_name no)
+			(do_not_autoplace no)
+			(effects
+				(font
+					(size 1.27 1.27)
+				)
+			)
+		)
+		(pin "1"
+		)
+		(instances
+			(project "CLOCK"
+				(path "/a8714d66-6565-4fb4-a698-a884e68083d2"
+					(reference "TP1")
+					(unit 1)
+				)
