File: hardware/schematic/v1.0/CLOCK/CLOCK.kicad_sch (KiCad schematic)
At the start: 131 parts, among them J1 Conn_Coaxial, J10 Conn_Coaxial, J12 Conn_Coaxial, J14 Conn_01x16_Socket, J2 Conn_Coaxial, J3 Conn_Coaxial, J4 Conn_Coaxial, J5 Conn_Coaxial, J6 Conn_Coaxial, J7 Conn_Coaxial, J8 Conn_Coaxial, J9 Conn_Coaxial, U1 LMK5B12204, U2 LMK1C1102, U3 LMK1C1102, U4 TPS78633, U5 TPS78633, U6 OCXO-10M, U7 TPS63020DSJR

Commit message: sch update
Parts:
- removed L1: 2.2uH, symbol Device:L
- added L1: 2.2uH, JLCImport:FNR4030S2R2MT, symbol JLCImport:FNR4030S2R2MT
Connections:
- net at U7.6 (L2), U7.7 (L2): now also L1.2
- net at U7.8 (L1), U7.9 (L1): now also L1.1
Changed lines of the file:
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@@
 	)
 	(junction
+		(at 327.66 110.49)
+		(diameter 0)
+		(color 0 0 0 0)
+	)
+	(junction
 		(at 144.78 208.28)
 		(diameter 0)
@@
 	)
 	(junction
-		(at 327.66 110.49)
-		(diameter 0)
-		(color 0 0 0 0)
-	)
-	(junction
 		(at 222.25 128.27)
 		(diameter 0)
@@
 	)
 	(junction
-		(at 317.5 110.49)
-		(diameter 0)
-		(color 0 0 0 0)
-	)
-	(junction
 		(at 363.22 63.5)
 		(diameter 0)
@@
 	)
 	(junction
+		(at 317.5 110.49)
+		(diameter 0)
+		(color 0 0 0 0)
+	)
+	(junction
 		(at 93.98 257.81)
 		(diameter 0)
@@
 	(wire
 		(pts
-			(xy 317.5 110.49) (xy 317.5 105.41)
+			(xy 317.5 110.49) (xy 317.5 106.68)
 		)
 		(stroke
@@
 	(wire
 		(pts
-			(xy 317.5 105.41) (xy 318.77 105.41)
-		)
-		(stroke
-			(width 0)
-			(type default)
-		)
-	)
-	(wire
-		(pts
 			(xy 295.91 78.74) (xy 300.99 78.74)
 		)
@@
 	(wire
 		(pts
-			(xy 326.39 105.41) (xy 327.66 105.41)
-		)
-		(stroke
-			(width 0)
-			(type default)
-		)
-	)
-	(wire
-		(pts
 			(xy 171.45 92.71) (xy 170.18 92.71)
 		)
@@
 	(wire
 		(pts
-			(xy 327.66 105.41) (xy 327.66 110.49)
+			(xy 327.66 106.68) (xy 327.66 110.49)
 		)
 		(stroke
@@
 	)
 	(symbol
+		(lib_id "JLCImport:FNR4030S2R2MT")
+		(at 322.58 106.68 0)
+		(unit 1)
+		(body_style 1)
+		(exclude_from_sim no)
+		(in_bom yes)
+		(on_board yes)
+		(in_pos_files yes)
+		(dnp no)
+		(property "Reference" "L1"
+			(at 322.5523 100.33 0)
+			(show_name no)
+			(do_not_autoplace no)
+			(effects
+				(font
+					(size 1.27 1.27)
+				)
+			)
+		)
+		(property "Value" "2.2uH"
+			(at 322.58 104.14 0)
+			(show_name no)
+			(do_not_autoplace no)
+			(effects
+				(font
+					(size 1.27 1.27)
+				)
+			)
+		)
+		(property "Footprint" "JLCImport:FNR4030S2R2MT"
+			(at 324.612 109.474 0)
+			(hide yes)
+			(show_name no)
+			(do_not_autoplace no)
+			(effects
+				(font
+					(size 1.27 1.27)
+				)
+			)
+		)
+		(property "Datasheet" "https://www.lcsc.com/datasheet/lcsc_datasheet_2304140030_cjiang--Changjiang-Microelectronics-Tech-FNR4030S2R2MT_C167869.pdf"
+			(at 324.612 109.474 0)
+			(hide yes)
+			(show_name no)
+			(do_not_autoplace no)
+			(effects
+				(font
+					(size 1.27 1.27)
+				)
+			)
+		)
+		(property "Description" "2.2uH 3.2A 39mΩ 5.8A Magnetic Shielded Inductor ±20% SMD,4x4mm Power Inductors ROHS"
+			(at 324.612 109.474 0)
+			(hide yes)
+			(show_name no)
+			(do_not_autoplace no)
+			(effects
+				(font
+					(size 1.27 1.27)
+				)
+			)
+		)
+		(property "LCSC" "C167869"
+			(at 322.58 106.68 0)
+			(hide yes)
+			(show_name no)
+			(do_not_autoplace no)
+			(effects
+				(font
+					(size 1.27 1.27)
+				)
+			)
+		)
+		(property "Manufacturer" "cjiang (Changjiang Microelectronics Tech)"
+			(at 324.612 109.474 0)
+			(hide yes)
+			(show_name no)
+			(do_not_autoplace no)
+			(effects
+				(font
+					(size 1.27 1.27)
+				)
+			)
+		)
+		(property "Manufacturer Part" "FNR4030S2R2MT"
+			(at 324.612 109.474 0)
+			(hide yes)
+			(show_name no)
+			(do_not_autoplace no)
+			(effects
+				(font
+					(size 1.27 1.27)
+				)
+			)
+		)
+		(pin "1"
+		)
+		(pin "2"
+		)
+		(instances
+			(project "CLOCK"
+				(path "/a8714d66-6565-4fb4-a698-a884e68083d2"
+					(reference "L1")
+					(unit 1)
+				)
+			)
+		)
+	)
+	(symbol
 		(lib_id "power:GND")
 		(at 322.58 209.55 270)
@@
 					(unit 1)
 				)
-			)
-		)
-	)
-	(symbol
-		(lib_id "Device:L")
-		(at 322.58 105.41 90)
-		(unit 1)
-		(body_style 1)
-		(exclude_from_sim no)
-		(in_bom yes)
-		(on_board yes)
-		(in_pos_files yes)
-		(dnp no)
-		(property "Reference" "L1"
-			(at 319.024 104.14 90)
-			(show_name no)
-			(do_not_autoplace no)
-			(effects
-				(font
-					(size 1.27 1.27)
-				)
-				(justify left)
-			)
-		)
-		(property "Value" "2.2uH"
-			(at 326.898 103.378 90)
-			(show_name no)
-			(do_not_autoplace no)
-			(effects
-				(font
-					(size 1.27 1.27)
-				)
-				(justify left)
-			)
-		)
-		(property "Footprint" ""
-			(at 322.58 105.41 0)
-			(hide yes)
-			(show_name no)
-			(do_not_autoplace no)
-			(effects
-				(font
-					(size 1.27 1.27)
-				)
-			)
-		)
-		(property "Datasheet" ""
-			(at 322.58 105.41 0)
-			(hide yes)
-			(show_name no)
-			(do_not_autoplace no)
-			(effects
-				(font
-					(size 1.27 1.27)
-				)
-			)
-		)
-		(property "Description" "Inductor"
-			(at 322.58 105.41 0)
-			(hide yes)
-			(show_name no)
-			(do_not_autoplace no)
-			(effects
-				(font
-					(size 1.27 1.27)
-				)
-			)
-		)
-		(pin "1"
-		)
-		(pin "2"
-		)
-		(instances
-			(project "CLOCK"
-				(path "/a8714d66-6565-4fb4-a698-a884e68083d2"
-					(reference "L1")
-					(unit 1)
-				)

Commit message: sch and pcb update
Parts:
- removed J14: Conn_01x16_Socket, Connector_PinSocket_2.54mm:PinSocket_1x16_P2.54mm_Vertical, symbol Connector:Conn_01x16_Socket
- removed R13: 0, Resistor_SMD:R_0402_1005Metric, symbol Device:R
- added H2, H3, H4, H5: MountingHole_Pad, MountingHole:MountingHole_3.2mm_M3_Pad, symbol Mechanical:MountingHole_Pad
- added J11, J13: Conn_01x06_Socket, Connector_PinSocket_2.54mm:PinSocket_1x06_P2.54mm_Vertical, symbol Connector:Conn_01x06_Socket
- added J14: Conn_01x02_Socket, Connector_PinSocket_2.54mm:PinSocket_1x02_P2.54mm_Vertical, symbol Connector:Conn_01x02_Socket
Connections:
- net PRIREF_N is gone; now on net GND: U1.7 (PRIREF_N)
- net +3.3V: now also J11.3 (Pin_3), J11.4 (Pin_4)
- net +5V_OCXO: now also J11.1 (Pin_1), J11.2 (Pin_2)
- net GND: now also H2.1, H3.1, H4.1, H5.1, J11.5 (Pin_5), J11.6 (Pin_6)
- net GPIO0: now also J13.4 (Pin_4)
- net GPIO1: now also J13.5 (Pin_5)
- net GPIO2: now also J13.6 (Pin_6)
- net PDN: now also J13.3 (Pin_3)
- net SCL: now also J13.2 (Pin_2)
- net SDA: now also J13.1 (Pin_1)
- net STATUS0: now also J14.1 (Pin_1)
- net STATUS1: now also J14.2 (Pin_2)
- no-connect marks 20 -> 18

Commit message: sch and pcb update
Other:
- note added: "HOLE"
- moved on the sheet: H2, H3, H4, H5
Changed lines of the file:
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@@
 		)
 	)
+	(text "HOLE"
+		(exclude_from_sim no)
+		(at 288.036 278.892 0)
+		(effects
+			(font
+				(size 2.54 2.54)
+			)
+		)
+	)
 	(text "OCXO"
 		(exclude_from_sim no)
@@
 		)
 	)
+	(polyline
+		(pts
+			(xy 228.6 245.11) (xy 228.6 283.21)
+		)
+		(stroke
+			(width 0)
+			(type dash)
+		)
+	)
 	(wire
 		(pts
@@
 	(polyline
 		(pts
+			(xy 228.6 245.11) (xy 297.18 245.11)
+		)
+		(stroke
+			(width 0)
+			(type dash)
+		)
+	)
+	(polyline
+		(pts
 			(xy 173.99 175.26) (xy 173.99 242.57)
 		)
@@
 		)
 	)
+	(polyline
+		(pts
+			(xy 297.18 245.11) (xy 297.18 283.21)
+		)
+		(stroke
+			(width 0)
+			(type dash)
+		)
+	)
 	(wire
 		(pts
@@
 		)
 	)
+	(polyline
+		(pts
+			(xy 228.6 283.21) (xy 297.18 283.21)
+		)
+		(stroke
+			(width 0)
+			(type dash)
+		)
+	)
 	(wire
 		(pts
@@
 	(symbol
 		(lib_id "power:GND")
-		(at 240.03 276.86 0)
+		(at 240.03 273.05 0)
 		(unit 1)
 		(body_style 1)
@@
 		(fields_autoplaced yes)
 		(property "Reference" "#PWR0135"
-			(at 240.03 283.21 0)
+			(at 240.03 279.4 0)
 			(hide yes)
 			(show_name no)
@@
 		)
 		(property "Value" "GND"
-			(at 240.03 281.94 0)
+			(at 240.03 278.13 0)
 			(hide yes)
 			(show_name no)
@@
 		)
 		(property "Footprint" ""
-			(at 240.03 276.86 0)
+			(at 240.03 273.05 0)
 			(hide yes)
 			(show_name no)
@@
 		)
 		(property "Datasheet" ""
-			(at 240.03 276.86 0)
+			(at 240.03 273.05 0)
 			(hide yes)
 			(show_name no)
@@
 		)
 		(property "Description" "Power symbol creates a global label with name \"GND\" , ground"
-			(at 240.03 276.86 0)
+			(at 240.03 273.05 0)
 			(hide yes)
 			(show_name no)
@@
 	(symbol
 		(lib_id "power:GND")
-		(at 273.05 276.86 0)
+		(at 273.05 273.05 0)
 		(unit 1)
 		(body_style 1)
@@
 		(fields_autoplaced yes)
 		(property "Reference" "#PWR0137"
-			(at 273.05 283.21 0)
+			(at 273.05 279.4 0)
 			(hide yes)
 			(show_name no)
@@
 		)
 		(property "Value" "GND"
-			(at 273.05 281.94 0)
+			(at 273.05 278.13 0)
 			(hide yes)
 			(show_name no)
@@
 		)
 		(property "Footprint" ""
-			(at 273.05 276.86 0)
+			(at 273.05 273.05 0)
 			(hide yes)
 			(show_name no)
@@
 		)
 		(property "Datasheet" ""
-			(at 273.05 276.86 0)
+			(at 273.05 273.05 0)
 			(hide yes)
 			(show_name no)
@@
 		)
 		(property "Description" "Power symbol creates a global label with name \"GND\" , ground"
-			(at 273.05 276.86 0)
+			(at 273.05 273.05 0)
 			(hide yes)
 			(show_name no)
@@
 	(symbol
 		(lib_id "Mechanical:MountingHole_Pad")
-		(at 273.05 274.32 0)
+		(at 273.05 270.51 0)
 		(unit 1)
 		(body_style 1)
@@
 		(fields_autoplaced yes)
 		(property "Reference" "H5"
-			(at 275.59 271.7799 0)
+			(at 275.59 267.9699 0)
 			(show_name no)
 			(do_not_autoplace no)
@@
 		)
 		(property "Value" "MountingHole_Pad"
-			(at 275.59 274.3199 0)
+			(at 275.59 270.5099 0)
 			(show_name no)
 			(do_not_autoplace no)
@@
 		)
 		(property "Footprint" "MountingHole:MountingHole_3.2mm_M3_Pad"
-			(at 273.05 274.32 0)
+			(at 273.05 270.51 0)
 			(hide yes)
 			(show_name no)
@@
 		)
 		(property "Datasheet" ""
-			(at 273.05 274.32 0)
+			(at 273.05 270.51 0)
 			(hide yes)
 			(show_name no)
@@
 		)
 		(property "Description" "Mounting Hole with connection"
-			(at 273.05 274.32 0)
+			(at 273.05 270.51 0)
 			(hide yes)
 			(show_name no)
@@
 	(symbol
 		(lib_id "Mechanical:MountingHole_Pad")
-		(at 273.05 259.08 0)
+		(at 273.05 255.27 0)
 		(unit 1)
 		(body_style 1)
@@
 		(fields_autoplaced yes)
 		(property "Reference" "H3"
-			(at 275.59 256.5399 0)
+			(at 275.59 252.7299 0)
 			(show_name no)
 			(do_not_autoplace no)
@@
 		)
 		(property "Value" "MountingHole_Pad"
-			(at 275.59 259.0799 0)
+			(at 275.59 255.2699 0)
 			(show_name no)
 			(do_not_autoplace no)
@@
 		)
 		(property "Footprint" "MountingHole:MountingHole_3.2mm_M3_Pad"
-			(at 273.05 259.08 0)
+			(at 273.05 255.27 0)
 			(hide yes)
 			(show_name no)
@@
 		)
 		(property "Datasheet" ""
-			(at 273.05 259.08 0)
+			(at 273.05 255.27 0)
 			(hide yes)
 			(show_name no)
@@
 		)
 		(property "Description" "Mounting Hole with connection"
-			(at 273.05 259.08 0)
+			(at 273.05 255.27 0)
 			(hide yes)
 			(show_name no)
@@
 	(symbol
 		(lib_id "Mechanical:MountingHole_Pad")
-		(at 240.03 274.32 0)
+		(at 240.03 270.51 0)
 		(unit 1)
 		(body_style 1)
@@
 		(fields_autoplaced yes)
 		(property "Reference" "H4"
-			(at 242.57 271.7799 0)
+			(at 242.57 267.9699 0)
 			(show_name no)
 			(do_not_autoplace no)
@@
 		)
 		(property "Value" "MountingHole_Pad"
-			(at 242.57 274.3199 0)
+			(at 242.57 270.5099 0)
 			(show_name no)
 			(do_not_autoplace no)
@@
 		)
 		(property "Footprint" "MountingHole:MountingHole_3.2mm_M3_Pad"
-			(at 240.03 274.32 0)
+			(at 240.03 270.51 0)
 			(hide yes)
 			(show_name no)
@@
 		)
 		(property "Datasheet" ""
-			(at 240.03 274.32 0)
+			(at 240.03 270.51 0)
 			(hide yes)
 			(show_name no)
@@
 		)
 		(property "Description" "Mounting Hole with connection"
-			(at 240.03 274.32 0)
+			(at 240.03 270.51 0)
 			(hide yes)
 			(show_name no)
@@
 	(symbol
 		(lib_id "Mechanical:MountingHole_Pad")
-		(at 240.03 259.08 0)
+		(at 240.03 255.27 0)
 		(unit 1)
 		(body_style 1)
@@
 		(fields_autoplaced yes)
 		(property "Reference" "H2"
-			(at 242.57 256.5399 0)
+			(at 242.57 252.7299 0)
 			(show_name no)
 			(do_not_autoplace no)
@@
 		)
 		(property "Value" "MountingHole_Pad"
-			(at 242.57 259.0799 0)
+			(at 242.57 255.2699 0)
 			(show_name no)
 			(do_not_autoplace no)
@@
 		)
 		(property "Footprint" "MountingHole:MountingHole_3.2mm_M3_Pad"
-			(at 240.03 259.08 0)
+			(at 240.03 255.27 0)
 			(hide yes)
 			(show_name no)
@@
 		)
 		(property "Datasheet" ""
-			(at 240.03 259.08 0)
+			(at 240.03 255.27 0)
 			(hide yes)
 			(show_name no)
@@
 		)
 		(property "Description" "Mounting Hole with connection"
-			(at 240.03 259.08 0)
+			(at 240.03 255.27 0)
 			(hide yes)
 			(show_name no)
@@
 	(symbol
 		(lib_id "power:GND")
-		(at 273.05 261.62 0)
+		(at 273.05 257.81 0)
 		(unit 1)
 		(body_style 1)
@@
 		(fields_autoplaced yes)
 		(property "Reference" "#PWR0136"
-			(at 273.05 267.97 0)
+			(at 273.05 264.16 0)
 			(hide yes)
 			(show_name no)
@@
 		)
 		(property "Value" "GND"
-			(at 273.05 266.7 0)
+			(at 273.05 262.89 0)
 			(hide yes)
 			(show_name no)
@@
 		)
 		(property "Footprint" ""
-			(at 273.05 261.62 0)
+			(at 273.05 257.81 0)
 			(hide yes)
 			(show_name no)
@@
 		)
 		(property "Datasheet" ""
-			(at 273.05 261.62 0)
+			(at 273.05 257.81 0)
 			(hide yes)
 			(show_name no)
@@
 		)
 		(property "Description" "Power symbol creates a global label with name \"GND\" , ground"
-			(at 273.05 261.62 0)
+			(at 273.05 257.81 0)
 			(hide yes)
 			(show_name no)
@@
 	(symbol
 		(lib_id "power:GND")
-		(at 240.03 261.62 0)
+		(at 240.03 257.81 0)
 		(unit 1)
 		(body_style 1)
@@
 		(fields_autoplaced yes)
 		(property "Reference" "#PWR0134"
-			(at 240.03 267.97 0)
+			(at 240.03 264.16 0)
 			(hide yes)
 			(show_name no)
@@
 		)
 		(property "Value" "GND"
-			(at 240.03 266.7 0)
+			(at 240.03 262.89 0)
 			(hide yes)
 			(show_name no)
@@
 		)
 		(property "Footprint" ""
-			(at 240.03 261.62 0)
+			(at 240.03 257.81 0)
 			(hide yes)
 			(show_name no)
@@
 		)
 		(property "Datasheet" ""
-			(at 240.03 261.62 0)
+			(at 240.03 257.81 0)
 			(hide yes)
 			(show_name no)
@@
 		)
 		(property "Description" "Power symbol creates a global label with name \"GND\" , ground"
-			(at 240.03 261.62 0)
+			(at 240.03 257.81 0)
 			(hide yes)
 			(show_name no)

Commit message: sch and pcb update
Parts:
- added R13, R22, R23, R32: DNP, Resistor_SMD:R_0402_1005Metric, symbol Device:R
- R24, R25, R26, R27, R4, R5, R7, R8: footprint Resistor_SMD:R_0603_1608Metric -> Resistor_SMD:R_0402_1005Metric
Connections:
- net OUT0_N: now also R13.2
- net OUT0_P: now also R13.1
- net OUT1_N: now also R22.2
- net OUT1_P: now also R22.1
- net OUT2_N: now also R23.2
- net OUT2_P: now also R23.1
- net OUT3_N: now also R32.2
- net OUT3_P: now also R32.1

Commit message: sch and pcb update
Parts:
- added TP2: TestPoint, TestPoint:TestPoint_Loop_D1.80mm_Drill1.0mm_Beaded, symbol Connector:TestPoint
Connections:
- net GND: now also TP2.1
Changed lines of the file:
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@@
 	)
 	(symbol
+		(lib_id "Connector:TestPoint")
+		(at 365.76 234.95 0)
+		(unit 1)
+		(body_style 1)
+		(exclude_from_sim no)
+		(in_bom yes)
+		(on_board yes)
+		(in_pos_files yes)
+		(dnp no)
+		(fields_autoplaced yes)
+		(property "Reference" "TP2"
+			(at 368.3 230.3779 0)
+			(show_name no)
+			(do_not_autoplace no)
+			(effects
+				(font
+					(size 1.27 1.27)
+				)
+				(justify left)
+			)
+		)
+		(property "Value" "TestPoint"
+			(at 368.3 232.9179 0)
+			(show_name no)
+			(do_not_autoplace no)
+			(effects
+				(font
+					(size 1.27 1.27)
+				)
+				(justify left)
+			)
+		)
+		(property "Footprint" "TestPoint:TestPoint_Loop_D1.80mm_Drill1.0mm_Beaded"
+			(at 370.84 234.95 0)
+			(hide yes)
+			(show_name no)
+			(do_not_autoplace no)
+			(effects
+				(font
+					(size 1.27 1.27)
+				)
+			)
+		)
+		(property "Datasheet" ""
+			(at 370.84 234.95 0)
+			(hide yes)
+			(show_name no)
+			(do_not_autoplace no)
+			(effects
+				(font
+					(size 1.27 1.27)
+				)
+			)
+		)
+		(property "Description" "test point"
+			(at 365.76 234.95 0)
+			(hide yes)
+			(show_name no)
+			(do_not_autoplace no)
+			(effects
+				(font
+					(size 1.27 1.27)
+				)
+			)
+		)
+		(pin "1"
+		)
+		(instances
+			(project "CLOCK"
+				(path "/a8714d66-6565-4fb4-a698-a884e68083d2"
+					(reference "TP2")
+					(unit 1)
+				)
+			)
+		)
+	)
+	(symbol
 		(lib_id "power:+3.3V")
 		(at 76.2 222.25 90)
@@
 					(unit 1)
 				)
+			)
+		)
+	)
+	(symbol
+		(lib_id "power:GND")
+		(at 365.76 234.95 0)
+		(unit 1)
+		(body_style 1)
+		(exclude_from_sim no)
+		(in_bom yes)
+		(on_board yes)
+		(in_pos_files yes)
+		(dnp no)
+		(fields_autoplaced yes)
+		(property "Reference" "#PWR0138"
+			(at 365.76 241.3 0)
+			(hide yes)
+			(show_name no)
+			(do_not_autoplace no)
+			(effects
+				(font
+					(size 1.27 1.27)
+				)
+			)
+		)
+		(property "Value" "GND"
+			(at 365.76 240.03 0)
+			(hide yes)
+			(show_name no)
+			(do_not_autoplace no)
+			(effects
+				(font
+					(size 1.27 1.27)
+				)
+			)
+		)
+		(property "Footprint" ""
+			(at 365.76 234.95 0)
+			(hide yes)
+			(show_name no)
+			(do_not_autoplace no)
+			(effects
+				(font
+					(size 1.27 1.27)
+				)
+			)
+		)
+		(property "Datasheet" ""
+			(at 365.76 234.95 0)
+			(hide yes)
+			(show_name no)
+			(do_not_autoplace no)
+			(effects
+				(font
+					(size 1.27 1.27)
+				)
+			)
+		)
+		(property "Description" "Power symbol creates a global label with name \"GND\" , ground"
+			(at 365.76 234.95 0)
+			(hide yes)
+			(show_name no)
+			(do_not_autoplace no)
+			(effects
+				(font
+					(size 1.27 1.27)
+				)
+			)
+		)
+		(pin "1"
+		)
+		(instances
+			(project "CLOCK"
+				(path "/a8714d66-6565-4fb4-a698-a884e68083d2"
+					(reference "#PWR0138")
+					(unit 1)
+				)

Commit message: add main ctrl
Parts:
- removed C1, C11, C12, C13, C14, C15, C17, C18, C19, C2, C27, C28, C29, C3, C30, C31, C32, C33, C34, C35, C36, C37, C4, C41, C45, C46, C49, C5, C51, C52, C54, C56, C62, C8: 100nF, Capacitor_SMD:C_0402_1005Metric, symbol Device:C
- removed C10, C16, C40, C50, C59, C7: 1uF, Capacitor_SMD:C_0402_1005Metric, symbol Device:C
- removed C20, C21, C22, C23, C24, C25, C47, C6, C60, C61, C63, C9: 10uF, Capacitor_SMD:C_0402_1005Metric, symbol Device:C
- removed C26: 470nF, Capacitor_SMD:C_0402_1005Metric, symbol Device:C
- removed C38, C42: 2.2uF, Capacitor_SMD:C_0603_1608Metric, symbol Device:C
- removed C39, C43: 10nF, Capacitor_SMD:C_0402_1005Metric, symbol Device:C
- removed C44: 10uF, Capacitor_SMD:C_0805_2012Metric, symbol Device:C
- removed C48, C53, C57: 10uF, Capacitor_SMD:C_0603_1608Metric, symbol Device:C
- removed C55: 22uF, Capacitor_SMD:C_0805_2012Metric, symbol Device:C
- removed C58: 1uF, Capacitor_SMD:C_0603_1608Metric, symbol Device:C
- removed D1, D2: LED, LED_SMD:LED_0603_1608Metric, symbol Device:LED
- removed FB1, FB10, FB3, FB4, FB5, FB7, FB9: 220 ohm@100mhz, Inductor_SMD:L_0603_1608Metric, symbol Device:FerriteBead_Small
- removed FB2, FB6: 80 ohm@100mhz, Inductor_SMD:L_0603_1608Metric, symbol Device:FerriteBead_Small
- removed FB8: 600 ohm@100mhz, Inductor_SMD:L_0603_1608Metric, symbol Device:FerriteBead_Small
- removed H1: HX_PH254-01-03-Z-L11_5_PCB_PIN_HEADER, JLCImport:HX_PH254-01-03-Z-L11_5_PCB_PIN_HEADER, symbol JLCImport:HX_PH254-01-03-Z-L11_5_PCB_PIN_HEADER
- removed H2, H3, H4, H5: MountingHole_Pad, MountingHole:MountingHole_3.2mm_M3_Pad, symbol Mechanical:MountingHole_Pad
- removed J1, J10, J12, J2, J3, J4, J5, J6, J7, J8, J9: Conn_Coaxial, Connector_Coaxial:SMA_Amphenol_132289_EdgeMount, symbol Connector:Conn_Coaxial
- removed J11, J13: Conn_01x06_Socket, Connector_PinSocket_2.54mm:PinSocket_1x06_P2.54mm_Vertical, symbol Connector:Conn_01x06_Socket
- removed J14: Conn_01x02_Socket, Connector_PinSocket_2.54mm:PinSocket_1x02_P2.54mm_Vertical, symbol Connector:Conn_01x02_Socket
- removed L1: 2.2uH, JLCImport:FNR4030S2R2MT, symbol JLCImport:FNR4030S2R2MT
- removed R1, R2: 4.7K, Resistor_SMD:R_0603_1608Metric, symbol Device:R
- removed R10, R12: 10K, Resistor_SMD:R_0402_1005Metric, symbol Device:R
- removed R11, R18, R21, R28, R29, R9: 0, Resistor_SMD:R_0402_1005Metric, symbol Device:R
- removed R13, R22, R23, R32: DNP, Resistor_SMD:R_0402_1005Metric, symbol Device:R
- removed R14, R15, R16, R17, R19, R20, R33, R34: 1K, Resistor_SMD:R_0402_1005Metric, symbol Device:R
- removed R24, R25, R26, R27, R4, R5, R7, R8: 49.9, Resistor_SMD:R_0402_1005Metric, symbol Device:R
- removed R3: 3296W-1-103_C48997937, Counter:3296W-1-103_C48997937, symbol Counter:3296W-1-103_C48997937
- removed R30, R31: 5.1K, Resistor_SMD:R_0402_1005Metric, symbol Device:R
- removed R36: 909K, Resistor_SMD:R_0402_1005Metric, symbol Device:R
- removed R37: 100K, Resistor_SMD:R_0402_1005Metric, symbol Device:R
- removed R38: 10, Resistor_SMD:R_0402_1005Metric, symbol Device:R
- removed TP1: Volt TestPoint, TestPoint:TestPoint_Pad_D1.0mm, symbol Connector:TestPoint
- removed TP2: TestPoint, TestPoint:TestPoint_Loop_D1.80mm_Drill1.0mm_Beaded, symbol Connector:TestPoint
- removed U1: LMK5B12204, Package_DFN_QFN:VQFN-48-1EP_7x7mm_P0.5mm_EP5.15x5.15mm_ThermalVias, symbol Counter:LMK5B12204
- removed U2, U3: LMK1C1102, Package_SON:WSON-8-1EP_2x2mm_P0.5mm_EP0.9x1.6mm, symbol Counter:LMK1C1102
- removed U4, U5: TPS78633, JLCImport:TPS78633DCQR, symbol Counter:TPS78633
- removed U6: OCXO-10M, JLCImport:DOPFITKR2-10M, symbol Counter:OCXO-10M
- removed U7: TPS63020DSJR, JLCImport:TPS63020DSJR, symbol Counter:TPS63020DSJR
- removed USB1: TYPE-C_16PIN_2MD_073, JLCImport:TYPE-C_16PIN_2MD_073, symbol JLCImport:TYPE-C_16PIN_2MD_073
Connections:
- no-connect marks 18 -> 0
Other:
- added sheet CLOCK_GEN (CLOCK_GEN.kicad_sch)
- added sheet MAIN_CTRL (MAIN_CTRL.kicad_sch)
- note removed: "10MHZ Ext Ref"
- note removed: "10MHZ REF IN"
- note removed: "10MHZ REF OUT"
- note removed: "50 OHM TRACE"
- note removed: "HOLE"
- note removed: "LDO"
- note removed: "OCXO"
- note removed: "SOCKET"
- note removed: "USB C"

Commit message: sch update
Other:
- sheet CLOCK_GEN ports: added none; removed GPIO0, GPIO1, GPIO2
- sheet MAIN_CTRL ports: added none; removed GPIO0, GPIO1, GPIO2
Changed lines of the file:
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@@
-	(wire
-		(pts
-			(xy 128.27 100.33) (xy 158.75 100.33)
-		)
-		(stroke
-			(width 0)
-			(type default)
-		)
-	)
 	(wire
 		(pts
@@
 	(wire
 		(pts
-			(xy 128.27 102.87) (xy 158.75 102.87)
-		)
-		(stroke
-			(width 0)
-			(type default)
-		)
-	)
-	(wire
-		(pts
 			(xy 128.27 93.98) (xy 158.75 93.98)
-		)
-		(stroke
-			(width 0)
-			(type default)
-		)
-	)
-	(wire
-		(pts
-			(xy 128.27 97.79) (xy 158.75 97.79)
 		)
 		(stroke
@@
 			)
 		)
-		(pin "GPIO0" input
-			(at 128.27 102.87 0)
-			(effects
-				(font
-					(size 1.27 1.27)
-				)
-				(justify right)
-			)
-		)
-		(pin "GPIO2" input
-			(at 128.27 97.79 0)
-			(effects
-				(font
-					(size 1.27 1.27)
-				)
-				(justify right)
-			)
-		)
 		(pin "SCL" input
 			(at 128.27 91.44 0)
@@
 			)
 		)
-		(pin "PDN" input
-			(at 128.27 93.98 0)
+		(pin "SDA" bidirectional
+			(at 128.27 88.9 0)
 			(effects
 				(font
@@
 			)
 		)
-		(pin "GPIO1" input
-			(at 128.27 100.33 0)
-			(effects
-				(font
-					(size 1.27 1.27)
-				)
-				(justify right)
-			)
-		)
-		(pin "SDA" bidirectional
-			(at 128.27 88.9 0)
+		(pin "PDN" input
+			(at 128.27 93.98 0)
 			(effects
 				(font
@@
 			)
 		)
-		(pin "GPIO0" output
-			(at 158.75 102.87 180)
-			(effects
-				(font
-					(size 1.27 1.27)
-				)
-				(justify left)
-			)
-		)
-		(pin "GPIO1" output
-			(at 158.75 100.33 180)
-			(effects
-				(font
-					(size 1.27 1.27)
-				)
-				(justify left)
-			)
-		)
 		(pin "PDN" output
 			(at 158.75 93.98 180)
@@
 			(effects
 				(font
-					(size 1.27 1.27)
-				)
-				(justify left)
-			)
-		)
-		(pin "GPIO2" output
-			(at 158.75 97.79 180)
-			(effects
-				(font
