File: hardware/schematic/v1.0/CLOCK/CLOCK.kicad_pcb (KiCad board)
At the start: 2 copper layers, 90 x 90 mm, 136 parts, among them J1 Conn_Coaxial, J10 Conn_Coaxial, J11 Conn_01x06_Socket, J12 Conn_Coaxial, J13 Conn_01x06_Socket, J14 Conn_01x02_Socket, J2 Conn_Coaxial, J3 Conn_Coaxial, J4 Conn_Coaxial, J5 Conn_Coaxial, J6 Conn_Coaxial, J7 Conn_Coaxial, J8 Conn_Coaxial, J9 Conn_Coaxial, U1 LMK5B12204, U2 LMK1C1102, U3 LMK1C1102, U4 TPS78633, U5 TPS78633, U6 OCXO-10M, U7 TPS63020DSJR

Commit message: sch and pcb update
Parts:
- moved H3 10.4 mm to (169.8, 58.4)
- moved H2 1.45 mm to (101.2, 58.4)
- moved H5 0.55 mm to (169.8, 137.3)
- moved H4 0.21 mm to (101.2, 137.3)
Changed lines of the file:
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@@
 	(footprint "MountingHole:MountingHole_3.2mm_M3_Pad"
 		(layer "F.Cu")
-		(at 101.9 59.65)
+		(at 101.25 58.35)
 		(descr "Mounting Hole 3.2mm, M3, generated by kicad-footprint-generator mountinghole.py")
 		(tags "mountinghole M3")
@@
 	(footprint "MountingHole:MountingHole_3.2mm_M3_Pad"
 		(layer "F.Cu")
-		(at 180.15 57.85)
+		(at 169.75 58.35)
 		(descr "Mounting Hole 3.2mm, M3, generated by kicad-footprint-generator mountinghole.py")
 		(tags "mountinghole M3")
@@
 	(footprint "MountingHole:MountingHole_3.2mm_M3_Pad"
 		(layer "F.Cu")
-		(at 101.4 137.2)
+		(at 101.25 137.35)
 		(descr "Mounting Hole 3.2mm, M3, generated by kicad-footprint-generator mountinghole.py")
 		(tags "mountinghole M3")
@@
 	(footprint "MountingHole:MountingHole_3.2mm_M3_Pad"
 		(layer "F.Cu")
-		(at 169.8 137.9)
+		(at 169.75 137.35)
 		(descr "Mounting Hole 3.2mm, M3, generated by kicad-footprint-generator mountinghole.py")
 		(tags "mountinghole M3")

Commit message: sch and pcb update
Parts:
- added R13: DNP, Resistor_SMD:R_0402_1005Metric, F.Cu at (119.2, 128.8)
- added R22: DNP, Resistor_SMD:R_0402_1005Metric, F.Cu at (150.6, 129.3)
- added R23: DNP, Resistor_SMD:R_0402_1005Metric, F.Cu at (150.7, 66.2)
- added R32: DNP, Resistor_SMD:R_0402_1005Metric, F.Cu at (119.2, 66.0)
- R24, R25, R26, R27, R4, R5, R7, R8: footprint Resistor_SMD:R_0603_1608Metric -> Resistor_SMD:R_0402_1005Metric
- moved R14 109.4 mm to (116.3, 89.1)
- moved R15 109.4 mm to (118.5, 89.1)
- moved J6 109.1 mm to (98.3, 89.3)
- moved R19 109.1 mm to (107.5, 87.6)
- moved R20 109.1 mm to (107.5, 90.8)
- moved R21 109.1 mm to (104.8, 89.4)
- moved C5 108.1 mm to (103.0, 75.8)
- moved C6 108.1 mm to (111.0, 84.1)
- moved C7 108.1 mm to (111.6, 81.0)
- moved C8 108.1 mm to (111.6, 79.7)
- moved J1 108.1 mm to (98.3, 75.8)
- moved R18 108.1 mm to (107.4, 75.8)
- moved C10 108.1 mm to (121.0, 80.5)
- moved C9 108.1 mm to (120.3, 83.8)
- moved R10 108.1 mm to (109.5, 73.4)
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Other:
- copper layers 2 -> 4

Commit message: sch and pcb update
Parts:
- added TP2: TestPoint, TestPoint:TestPoint_Loop_D1.80mm_Drill1.0mm_Beaded, F.Cu at (170.5, 106.8)
- moved J11 131.1 mm to (198.1, 113.0)
- moved J14 46.0 mm to (98.0, 65.0)
Changed lines of the file:
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@@
 		(capping no)
 		(filling no)
-		(zone_defaults)
 		(aux_axis_origin 95.75 52.85)
 		(grid_origin 95.75 52.85)
@@
 		)
 	)
+	(footprint "TestPoint:TestPoint_Loop_D1.80mm_Drill1.0mm_Beaded"
+		(layer "F.Cu")
+		(at 170.525 106.825)
+		(descr "wire loop with bead as test point, loop diameter 1.8mm, hole diameter 1.0mm")
+		(tags "test point wire loop bead")
+		(property "Reference" "TP2"
+			(at -0.025 -2.475 0)
+			(layer "F.SilkS")
+			(effects
+				(font
+					(size 0.5 0.5)
+					(thickness 0.1)
+				)
+			)
+		)
+		(property "Value" "TestPoint"
+			(at 0 -2.8 0)
+			(layer "F.Fab")
+			(hide yes)
+			(effects
+				(font
+					(size 1 1)
+					(thickness 0.15)
+				)
+			)
+		)
+		(property "Datasheet" ""
+			(at 0 0 0)
+			(unlocked yes)
+			(layer "F.Fab")
+			(hide yes)
+			(effects
+				(font
+					(size 1.27 1.27)
+					(thickness 0.15)
+				)
+			)
+		)
+		(property "Description" "test point"
+			(at 0 0 0)
+			(unlocked yes)
+			(layer "F.Fab")
+			(hide yes)
+			(effects
+				(font
+					(size 1.27 1.27)
+					(thickness 0.15)
+				)
+			)
+		)
+		(property ki_fp_filters "Pin* Test*")
+		(sheetname "/")
+		(sheetfile "CLOCK.kicad_sch")
+		(units
+			(unit
+				(name "A")
+				(pins "1")
+			)
+		)
+		(attr through_hole)
+		(duplicate_pad_numbers_are_jumpers no)
+		(fp_circle
+			(center 0 0)
+			(end 1.5 0)
+			(stroke
+				(width 0.12)
+				(type solid)
+			)
+			(fill no)
+			(layer "F.SilkS")
+		)
+		(fp_circle
+			(center 0 0)
+			(end 1.8 0)
+			(stroke
+				(width 0.05)
+				(type solid)
+			)
+			(fill no)
+			(layer "F.CrtYd")
+		)
+		(fp_line
+			(start -0.9 -0.2)
+			(end 0.9 -0.2)
+			(stroke
+				(width 0.12)
+				(type solid)
+			)
+			(layer "F.Fab")
+		)
+		(fp_line
+			(start -0.9 0.2)
+			(end -0.9 -0.2)
+			(stroke
+				(width 0.12)
+				(type solid)
+			)
+			(layer "F.Fab")
+		)
+		(fp_line
+			(start 0.9 -0.2)
+			(end 0.9 0.2)
+			(stroke
+				(width 0.12)
+				(type solid)
+			)
+			(layer "F.Fab")
+		)
+		(fp_line
+			(start 0.9 0.2)
+			(end -0.9 0.2)
+			(stroke
+				(width 0.12)
+				(type solid)
+			)
+			(layer "F.Fab")
+		)
+		(fp_circle
+			(center 0 0)
+			(end 1.3 0)
+			(stroke
+				(width 0.12)
+				(type solid)
+			)
+			(fill no)
+			(layer "F.Fab")
+		)
+		(fp_text user "${REFERENCE}"
+			(at -0.025 -2.475 0)
+			(layer "F.Fab")
+			(effects
+				(font
+					(size 0.5 0.5)
+					(thickness 0.1)
+				)
+			)
+		)
+		(pad "1" thru_hole circle
+			(at 0 0)
+			(size 2 2)
+			(drill 1)
+			(layers "*.Cu" "*.Mask")
+			(remove_unused_layers no)
+			(net "GND")
+			(pinfunction "1_1")
+			(pintype "passive")
+		)
+		(embedded_fonts no)
+		(model "${KICAD10_3DMODEL_DIR}/TestPoint.3dshapes/TestPoint_Loop_D1.80mm_Drill1.0mm_Beaded.step"
+			(offset
+				(xyz 0 0 0)
+			)
+			(scale
+				(xyz 1 1 1)
+			)
+			(rotate
+				(xyz 0 0 0)
+			)
+		)
+	)
 	(footprint "Capacitor_SMD:C_0402_1005Metric"
 		(layer "F.Cu")
@@
 	(footprint "Connector_PinSocket_2.54mm:PinSocket_1x02_P2.54mm_Vertical"
 		(layer "F.Cu")
-		(at 60.2 91.08)
+		(at 98.05 64.95)
 		(descr "Through hole straight socket strip, 1x02, 2.54mm pitch, single row (from Kicad 4.0.7), script generated")
 		(tags "Through hole socket strip THT 1x02 2.54mm single row")
@@
 	(footprint "Connector_PinSocket_2.54mm:PinSocket_1x06_P2.54mm_Vertical"
 		(layer "F.Cu")
-		(at 67.2 121.33)
+		(at 198.05 112.98)
 		(descr "Through hole straight socket strip, 1x06, 2.54mm pitch, single row (from Kicad 4.0.7), script generated")
 		(tags "Through hole socket strip THT 1x06 2.54mm single row")

Commit message: sch and pcb update
Parts:
- added C64: 100nF, Capacitor_SMD:C_0402_1005Metric, F.Cu at (204.3, 84.5)
- added C65: 100nF, Capacitor_SMD:C_0402_1005Metric, F.Cu at (202.2, 86.0)
- added C66: 100nF, Capacitor_SMD:C_0402_1005Metric, F.Cu at (201.1, 93.3)
- added C67: 100nF, Capacitor_SMD:C_0402_1005Metric, F.Cu at (212.2, 95.5)
- added C68: 100nF, Capacitor_SMD:C_0402_1005Metric, F.Cu at (213.8, 87.7)
- added C69: 100nF, Capacitor_SMD:C_0402_1005Metric, F.Cu at (200.9, 91.5)
- added C70: 20pF, Capacitor_SMD:C_0402_1005Metric, F.Cu at (196.1, 93.2)
- added C71: 20pF, Capacitor_SMD:C_0402_1005Metric, F.Cu at (195.9, 87.2)
- added J15: Conn_01x04_Pin, Connector_PinHeader_2.54mm:PinHeader_1x04_P2.54mm_Vertical, F.Cu at (225.2, 94.3)
- added R39: 10K, Resistor_SMD:R_0603_1608Metric, F.Cu at (209.3, 97.6)
- added U8: STM32F103CBTx, Package_QFP:LQFP-48_7x7mm_P0.5mm, F.Cu at (207.6, 90.7)
- added X1: X32258MOB4SI, JLCImport:X32258MOB4SI, F.Cu at (196.0, 90.3)
- moved C29 19.6 mm to (50.3, 60.5)
- moved C27 3.70 mm to (65.8, 60.1)
- moved U2 0.30 mm to (110.6, 76.6)
Connections:
- U2 pad 9: (no net) -> GND
- U3 pad 9: (no net) -> GND

Commit message: sch and pcb update
Parts:
- added J16: Conn_01x03_Pin, Connector_PinHeader_2.54mm:PinHeader_1x03_P2.54mm_Vertical, F.Cu at (217.7, 109.4)
- moved U2 0.56 mm to (110.6, 77.2)
- moved U3 0.54 mm to (118.4, 77.0)
Connections:
- U8 pad 12: unconnected-(U8-PA2-Pad12) -> /MAIN_CTRL/UART3_TXD
- U8 pad 13: unconnected-(U8-PA3-Pad13) -> /MAIN_CTRL/UART3_RXD

Commit message: sch and pcb update
Parts:
- C64, C65, C66, C67, C68, C69, C70, C71, R39, U8, X1: moved to B.Cu
- R36, R37: footprint Resistor_SMD:R_0402_1005Metric -> Resistor_SMD:R_0603_1608Metric
- moved FB10 111.8 mm to (147.2, 96.1), turned to -90 degrees
- moved C56 108.7 mm to (145.7, 105.1), turned to 45 degrees
- moved FB9 108.4 mm to (143.9, 92.5), turned to 135 degrees
- moved C62 107.3 mm to (149.0, 95.8), turned to 90 degrees
- moved FB7 106.0 mm to (144.5, 104.0), turned to -135 degrees
- moved C60 104.8 mm to (142.8, 105.5), turned to 135 degrees
- moved C18 104.1 mm to (134.7, 110.1)
- moved FB3 103.5 mm to (123.3, 94.6), turned to -45 degrees
- moved C59 103.5 mm to (144.7, 91.5), turned to -45 degrees
- moved C63 103.5 mm to (145.3, 96.6), turned to -90 degrees
- moved C61 100.1 mm to (142.2, 91.2), turned to -135 degrees
- moved C30 96.9 mm to (140.2, 102.8), turned to 135 degrees
- moved D1 94.5 mm to (123.7, 102.8), turned to 0 degrees
- moved D2 93.6 mm to (123.8, 104.8), turned to 0 degrees
- moved C16 93.0 mm to (124.8, 91.0), turned to 45 degrees
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
Commit message: sch update
Parts:
- J15: value Conn_01x04_Pin -> Conn_01x03_Pin; footprint Connector_PinHeader_2.54mm:PinHeader_1x04_P2.54mm_Vertical -> Connector_PinHeader_2.54mm:PinHeader_1x03_P2.54mm_Vertical
- moved J15 127.1 mm to (98.8, 108.0), turned to 0 degrees
- moved J16 87.0 mm to (134.7, 135.2)
- moved C64 78.5 mm to (130.6, 112.2)
- moved C66 78.5 mm to (133.8, 121.0)
- moved C69 78.5 mm to (133.9, 119.3)
- moved C70 78.5 mm to (138.8, 121.0)
- moved U8 78.5 mm to (127.3, 118.4)
- moved C65 78.5 mm to (132.7, 113.8)
- moved C67 78.5 mm to (122.7, 123.3)
- moved C68 78.5 mm to (121.2, 115.5)
- moved C71 78.5 mm to (139.0, 114.9)
- moved R39 78.5 mm to (125.6, 125.4)
- moved X1 78.5 mm to (138.9, 118.0)
Connections:
- J15 pad 1: +3.3V -> /MAIN_CTRL/SWDIO
- J15 pad 2: GND -> /MAIN_CTRL/SWCLK
- J15 pad 3: /MAIN_CTRL/SWDIO -> GND

Commit message: sch update
Parts:
- added H6: HX_PH254-01-03-Z-L11_5_PCB_PIN_HEADER, JLCImport:HX_PH254-01-03-Z-L11_5_PCB_PIN_HEADER, F.Cu at (112.5, 96.8)
- added H7: HX_PH254-01-03-Z-L11_5_PCB_PIN_HEADER, JLCImport:HX_PH254-01-03-Z-L11_5_PCB_PIN_HEADER, F.Cu at (117.0, 107.5)
- added R35: 0, Resistor_SMD:R_0402_1005Metric, F.Cu at (223.4, 92.7)
- added R40: 0, Resistor_SMD:R_0402_1005Metric, F.Cu at (223.4, 94.7)
- added R41: 0, Resistor_SMD:R_0402_1005Metric, F.Cu at (120.3, 107.6)
- added R42: 0, Resistor_SMD:R_0402_1005Metric, F.Cu at (223.4, 98.7)
- J13: value Conn_01x06_Socket -> Conn_01x04_Socket; footprint Connector_PinSocket_2.54mm:PinSocket_1x06_P2.54mm_Vertical -> Connector_PinHeader_2.54mm:PinHeader_1x04_P2.54mm_Vertical
- moved J13 70.8 mm to (98.2, 124.3)
- moved J11 31.9 mm to (190.9, 81.8)
Connections:
- J13 pad 1: SDA -> SCL
- J13 pad 2: SCL -> SDA
- J13 pad 4: GPIO0 -> GND
- U1 pad 12: GPIO0 -> Net-(U1-GPIO0/SYNCN)
- U1 pad 24: GPIO1 -> GND
- U1 pad 30: GPIO2 -> unconnected-(U1-GPIO2/SDO/_FINC-Pad30)
- U8 pad 25: GPIO0 -> unconnected-(U8-PB12-Pad25)
- U8 pad 26: GPIO1 -> unconnected-(U8-PB13-Pad26)
- U8 pad 27: GPIO2 -> unconnected-(U8-PB14-Pad27)
