File: hardware/schematic/v1.0/CLOCK/CLOCK.kicad_pcb (KiCad board)
At the start: 4 copper layers, 90 x 90 mm, 160 parts, among them J1 Conn_Coaxial, J10 Conn_Coaxial, J11 Conn_01x06_Socket, J12 Conn_Coaxial, J13 Conn_01x04_Socket, J14 Conn_01x02_Socket, J15 Conn_01x03_Pin, J16 Conn_01x03_Pin, J2 Conn_Coaxial, J3 Conn_Coaxial, J4 Conn_Coaxial, J5 Conn_Coaxial, J6 Conn_Coaxial, J7 Conn_Coaxial, J8 Conn_Coaxial, J9 Conn_Coaxial, U1 LMK5B12204, U2 LMK1C1102, U3 LMK1C1102, U4 TPS78633, U5 TPS78633, U6 OCXO-10M, U7 TPS63020DSJR, U8 STM32F103CBTx, X1 X32258MOB4SI

Commit message: sch and pcb update
Parts:
- added C72: 100nF, Capacitor_SMD:C_0402_1005Metric, F.Cu at (121.6, 109.6)
- added R6: 10K, Resistor_SMD:R_0603_1608Metric, F.Cu at (116.3, 96.0)
- R35, R40, R42: moved to B.Cu
- R41: value 0 -> 10K
- moved R40 126.1 mm to (102.2, 129.3)
- moved R35 126.0 mm to (102.1, 126.8), turned to 180 degrees
- moved R42 124.0 mm to (102.1, 124.2)
- moved R41 0.79 mm to (121.1, 107.5)
Connections:
- R35 pad 1: SDA -> Net-(U8-PB11)
- R40 pad 1: SCL -> PDN
- R40 pad 2: SCL -> Net-(U8-PB15)
- R42 pad 1: PDN -> SCL
- R42 pad 2: PDN -> Net-(U8-PB10)
- U8 pad 21: SCL -> Net-(U8-PB10)
- U8 pad 22: SDA -> Net-(U8-PB11)
- U8 pad 28: PDN -> Net-(U8-PB15)
