File: hardware/schematic/v1.0/CLOCK/CLOCK_GEN.kicad_sch (KiCad schematic)
At the start: 141 parts, among them J1 Conn_Coaxial, J10 Conn_Coaxial, J11 Conn_Coaxial, J12 Conn_Coaxial, J13 Conn_Coaxial, J14 Conn_Coaxial, J2 Conn_Coaxial, J3 Conn_01x06_Socket, J4 Conn_01x02_Socket, J5 Conn_01x06_Socket, J6 Conn_Coaxial, J7 Conn_Coaxial, J8 Conn_Coaxial, J9 Conn_Coaxial, U1 TPS78633, U2 LMK1C1102, U3 LMK1C1102, U4 LMK5B12204, U5 TPS78633, U6 TPS63020DSJR, U7 OCXO-10M

Commit message: sch and pcb update
Parts:
- renumbered C58 to C1, C27 to C10, C26 to C11, C50 to C12, C51 to C13, C48 to C14, C49 to C15, C5 to C16, C1 to C17, C6 to C18, C7 to C19, C59 to C2, C9 to C20, C13 to C21, C14 to C22, C25 to C24, C29 to C25, C32 to C26, C35 to C27, C20 to C28, C24 to C29, C56 to C3, C31 to C30, C37 to C31, C38 to C32, C39 to C33, C40 to C34, C41 to C35, C42 to C36, C43 to C37, C15 to C38, C17 to C39, C57 to C4, C19 to C40, C22 to C41, C28 to C42, C33 to C43, C34 to C44, C36 to C45, C45 to C46, C44 to C47, C62 to C48, C55 to C49, C8 to C5, C60 to C50, C54 to C51, C53 to C52, C46 to C53, C47 to C54, C61 to C55, C3 to C56, C63 to C57, C52 to C58, C4 to C59, C16 to C6, C11 to C60, C12 to C61, C2 to C62, C10 to C63, C18 to C7, C21 to C8, C30 to C9, FB5 to FB1, FB2 to FB10, FB9 to FB2, FB1 to FB3, FB6 to FB4, FB7 to FB5, FB8 to FB6, FB3 to FB7, FB10 to FB8, FB4 to FB9, H5 to H1, H1 to H2, H2 to H4, H4 to H5, J7 to J10, J3 to J11, J10 to J12, J5 to J13, J4 to J14, J13 to J2, J14 to J3, J11 to J4, J12 to J5, J2 to J6, J8 to J7, J9 to J8, J6 to J9, R15 to R1, R8 to R10, R9 to R11, R10 to R12, R20 to R13, R11 to R14, R13 to R15, R1 to R16, R2 to R17, R5 to R18, R6 to R19, R16 to R2, R7 to R20, R3 to R21, R19 to R22, R30 to R23, R23 to R24, R22 to R25, R25 to R26, R24 to R27, R4 to R28, R14 to R29, R28 to R3, R17 to R30, R18 to R31, R29 to R32, R27 to R33, R26 to R34, R31 to R36, R32 to R37, R21 to R38, R34 to R4, R36 to R5, R33 to R7, R35 to R8, R12 to R9, U4 to U1, U1 to U4, U7 to U6, U6 to U7
Other:
- moved on the sheet: C6, C7, C8, FB6, R14, R15

Commit message: sch and pcb update
Connections:
- net GND: now also U2.9 (EP), U3.9 (EP)
Changed lines of the file:
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@@
 	)
 	(symbol
-		(lib_id "Counter:LMK1C1102")
-		(at 111.76 200.66 0)
-		(unit 1)
-		(body_style 1)
-		(exclude_from_sim no)
-		(in_bom yes)
-		(on_board yes)
-		(in_pos_files yes)
-		(dnp no)
-		(property "Reference" "U3"
-			(at 112.522 199.644 0)
-			(show_name no)
-			(do_not_autoplace no)
-			(effects
-				(font
-					(size 1.27 1.27)
-				)
-			)
-		)
-		(property "Value" "LMK1C1102"
-			(at 120.396 199.644 0)
-			(show_name no)
-			(do_not_autoplace no)
-			(effects
-				(font
-					(size 1.27 1.27)
-				)
-			)
-		)
-		(property "Footprint" "Package_SON:WSON-8-1EP_2x2mm_P0.5mm_EP0.9x1.6mm"
-			(at 111.76 200.66 0)
-			(hide yes)
-			(show_name no)
-			(do_not_autoplace no)
-			(effects
-				(font
-					(size 1.27 1.27)
-				)
-			)
-		)
-		(property "Datasheet" ""
-			(at 111.76 200.66 0)
-			(hide yes)
-			(show_name no)
-			(do_not_autoplace no)
-			(effects
-				(font
-					(size 1.27 1.27)
-				)
-			)
-		)
-		(property "Description" ""
-			(at 111.76 200.66 0)
-			(hide yes)
-			(show_name no)
-			(do_not_autoplace no)
-			(effects
-				(font
-					(size 1.27 1.27)
-				)
-			)
-		)
-		(pin "5"
-		)
-		(pin "8"
-		)
-		(pin "7"
-		)
-		(pin "6"
-		)
-		(pin "3"
-		)
-		(pin "9"
-		)
-		(pin "1"
-		)
-		(pin "2"
-		)
-		(pin "4"
-		)
-		(instances
-			(project "CLOCK"
-				(path "/e8d80103-6a56-4030-bccc-c2b7ae1d549d/ad7e8003-daaa-4c55-9ec1-92ad34af2e50"
-					(reference "U3")
-					(unit 1)
-				)
-			)
-		)
-	)
-	(symbol
 		(lib_id "power:GND")
 		(at 119.38 215.9 0)
@@
 	)
 	(symbol
+		(lib_id "Counter:LMK1C1102")
+		(at 111.76 200.66 0)
+		(unit 1)
+		(body_style 1)
+		(exclude_from_sim no)
+		(in_bom yes)
+		(on_board yes)
+		(in_pos_files yes)
+		(dnp no)
+		(fields_autoplaced yes)
+		(property "Reference" "U3"
+			(at 118.745 195.58 0)
+			(show_name no)
+			(do_not_autoplace no)
+			(effects
+				(font
+					(size 1.27 1.27)
+				)
+			)
+		)
+		(property "Value" "LMK1C1102"
+			(at 118.745 198.12 0)
+			(show_name no)
+			(do_not_autoplace no)
+			(effects
+				(font
+					(size 1.27 1.27)
+				)
+			)
+		)
+		(property "Footprint" "Package_SON:WSON-8-1EP_2x2mm_P0.5mm_EP0.9x1.6mm"
+			(at 111.76 200.66 0)
+			(hide yes)
+			(show_name no)
+			(do_not_autoplace no)
+			(effects
+				(font
+					(size 1.27 1.27)
+				)
+			)
+		)
+		(property "Datasheet" ""
+			(at 111.76 200.66 0)
+			(hide yes)
+			(show_name no)
+			(do_not_autoplace no)
+			(effects
+				(font
+					(size 1.27 1.27)
+				)
+			)
+		)
+		(property "Description" ""
+			(at 111.76 200.66 0)
+			(hide yes)
+			(show_name no)
+			(do_not_autoplace no)
+			(effects
+				(font
+					(size 1.27 1.27)
+				)
+			)
+		)
+		(pin "3"
+		)
+		(pin "6"
+		)
+		(pin "4"
+		)
+		(pin "1"
+		)
+		(pin "5"
+		)
+		(pin "8"
+		)
+		(pin "2"
+		)
+		(pin "7"
+		)
+		(pin "9"
+		)
+		(instances
+			(project "CLOCK"
+				(path "/e8d80103-6a56-4030-bccc-c2b7ae1d549d/ad7e8003-daaa-4c55-9ec1-92ad34af2e50"
+					(reference "U3")
+					(unit 1)
+				)
+			)
+		)
+	)
+	(symbol
 		(lib_id "Device:C")
 		(at 354.33 27.94 90)
@@
 			)
 		)
-		(property "Description" "Ferrite bead"
+		(property "Description" "Ferrite bead, small symbol"
 			(at 364.49 118.11 0)
 			(hide yes)
@@
 	)
 	(symbol
-		(lib_id "Counter:LMK1C1102")
-		(at 74.93 200.66 0)
-		(unit 1)
-		(body_style 1)
-		(exclude_from_sim no)
-		(in_bom yes)
-		(on_board yes)
-		(in_pos_files yes)
-		(dnp no)
-		(property "Reference" "U2"
-			(at 75.692 199.644 0)
-			(show_name no)
-			(do_not_autoplace no)
-			(effects
-				(font
-					(size 1.27 1.27)
-				)
-			)
-		)
-		(property "Value" "LMK1C1102"
-			(at 83.566 199.644 0)
-			(show_name no)
-			(do_not_autoplace no)
-			(effects
-				(font
-					(size 1.27 1.27)
-				)
-			)
-		)
-		(property "Footprint" "Package_SON:WSON-8-1EP_2x2mm_P0.5mm_EP0.9x1.6mm"
-			(at 74.93 200.66 0)
-			(hide yes)
-			(show_name no)
-			(do_not_autoplace no)
-			(effects
-				(font
-					(size 1.27 1.27)
-				)
-			)
-		)
-		(property "Datasheet" ""
-			(at 74.93 200.66 0)
-			(hide yes)
-			(show_name no)
-			(do_not_autoplace no)
-			(effects
-				(font
-					(size 1.27 1.27)
-				)
-			)
-		)
-		(property "Description" ""
-			(at 74.93 200.66 0)
-			(hide yes)
-			(show_name no)
-			(do_not_autoplace no)
-			(effects
-				(font
-					(size 1.27 1.27)
-				)
-			)
-		)
-		(pin "3"
-		)
-		(pin "1"
-		)
-		(pin "5"
-		)
-		(pin "2"
-		)
-		(pin "6"
-		)
-		(pin "8"
-		)
-		(pin "7"
-		)
-		(pin "4"
-		)
-		(pin "9"
-		)
-		(instances
-			(project "CLOCK"
-				(path "/e8d80103-6a56-4030-bccc-c2b7ae1d549d/ad7e8003-daaa-4c55-9ec1-92ad34af2e50"
-					(reference "U2")
-					(unit 1)
-				)
-			)
-		)
-	)
-	(symbol
 		(lib_id "power:GND")
 		(at 91.44 163.83 0)
@@
 					(unit 1)
 				)
+			)
+		)
+	)
+	(symbol
+		(lib_id "Counter:LMK1C1102")
+		(at 74.93 200.66 0)
+		(unit 1)
+		(body_style 1)
+		(exclude_from_sim no)
+		(in_bom yes)
+		(on_board yes)
+		(in_pos_files yes)
+		(dnp no)
+		(fields_autoplaced yes)
+		(property "Reference" "U2"
+			(at 81.915 195.58 0)
+			(show_name no)
+			(do_not_autoplace no)
+			(effects
+				(font
+					(size 1.27 1.27)
+				)
+			)
+		)
+		(property "Value" "LMK1C1102"
+			(at 81.915 198.12 0)
+			(show_name no)
+			(do_not_autoplace no)
+			(effects
+				(font
+					(size 1.27 1.27)
+				)
+			)
+		)
+		(property "Footprint" "Package_SON:WSON-8-1EP_2x2mm_P0.5mm_EP0.9x1.6mm"
+			(at 74.93 200.66 0)
+			(hide yes)
+			(show_name no)
+			(do_not_autoplace no)
+			(effects
+				(font
+					(size 1.27 1.27)
+				)
+			)
+		)
+		(property "Datasheet" ""
+			(at 74.93 200.66 0)
+			(hide yes)
+			(show_name no)
+			(do_not_autoplace no)
+			(effects
+				(font
+					(size 1.27 1.27)
+				)
+			)
+		)
+		(property "Description" ""
+			(at 74.93 200.66 0)
+			(hide yes)
+			(show_name no)
+			(do_not_autoplace no)
+			(effects
+				(font
+					(size 1.27 1.27)
+				)
+			)
+		)
+		(pin "1"
+		)
+		(pin "4"
+		)
+		(pin "5"
+		)
+		(pin "8"
+		)
+		(pin "3"
+		)
+		(pin "2"
+		)
+		(pin "6"
+		)
+		(pin "7"
+		)
+		(pin "9"
+		)
+		(instances
+			(project "CLOCK"
+				(path "/e8d80103-6a56-4030-bccc-c2b7ae1d549d/ad7e8003-daaa-4c55-9ec1-92ad34af2e50"
+					(reference "U2")
+					(unit 1)
+				)

Commit message: sch and pcb update
Parts:
- R36, R37: footprint Resistor_SMD:R_0402_1005Metric -> Resistor_SMD:R_0603_1608Metric
Changed lines of the file:
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@@
 			)
 		)
-		(property "Footprint" "Resistor_SMD:R_0402_1005Metric"
+		(property "Footprint" "Resistor_SMD:R_0603_1608Metric"
 			(at 347.98 124.46 90)
 			(hide yes)
@@
 			)
 		)
-		(property "Footprint" "Resistor_SMD:R_0402_1005Metric"
+		(property "Footprint" "Resistor_SMD:R_0603_1608Metric"
 			(at 347.98 134.62 90)
 			(hide yes)
