File: hardware/schematic/v1.0/CLOCK/CLOCK_GEN.kicad_sch (KiCad schematic)
At the start: 141 parts, among them J1 Conn_Coaxial, J10 Conn_Coaxial, J11 Conn_01x06_Socket, J12 Conn_Coaxial, J13 Conn_01x06_Socket, J14 Conn_01x02_Socket, J2 Conn_Coaxial, J3 Conn_Coaxial, J4 Conn_Coaxial, J5 Conn_Coaxial, J6 Conn_Coaxial, J7 Conn_Coaxial, J8 Conn_Coaxial, J9 Conn_Coaxial, U1 LMK5B12204, U2 LMK1C1102, U3 LMK1C1102, U4 TPS78633, U5 TPS78633, U6 OCXO-10M, U7 TPS63020DSJR

Commit message: sch update
Parts:
- removed J13: Conn_01x06_Socket, Connector_PinSocket_2.54mm:PinSocket_1x06_P2.54mm_Vertical, symbol Connector:Conn_01x06_Socket
- added H6, H7: HX_PH254-01-03-Z-L11_5_PCB_PIN_HEADER, JLCImport:HX_PH254-01-03-Z-L11_5_PCB_PIN_HEADER, symbol JLCImport:HX_PH254-01-03-Z-L11_5_PCB_PIN_HEADER
- added J13: Conn_01x04_Socket, Connector_PinHeader_2.54mm:PinHeader_1x04_P2.54mm_Vertical, symbol Connector:Conn_01x04_Socket
- added R35, R40, R41, R42: 0, Resistor_SMD:R_0402_1005Metric, symbol Device:R
Connections:
- net GPIO1 is gone; now on net GND: U1.24 (GPIO1/SCS)
- net +3.3V: now also H6.1, H7.1
- net GND: now also H6.3, H7.3, J13.4 (Pin_4)
- net PDN: now also J13.3 (Pin_3), R41.2, R42.1, R42.2
- net SCL: now also J13.1 (Pin_1), R40.1, R40.2
- net SDA: now also J13.2 (Pin_2), R35.1, R35.2
- net GPIO0: no longer names the net of U1.12 (GPIO0/SYNCN)
- net GPIO0: now also H6.2
- net GPIO2: no longer names the net of U1.30 (GPIO2/SDO/_FINC)
- new net: H7.2, R41.1
- no-connect marks 18 -> 19
Other:
- note removed: "SOCKET"

Commit message: sch and pcb update
Parts:
- removed R35, R40, R42: 0, Resistor_SMD:R_0402_1005Metric, symbol Device:R
- added C72: 100nF, Capacitor_SMD:C_0402_1005Metric, symbol Device:C
- added R6: 10K, Resistor_SMD:R_0603_1608Metric, symbol Device:R
- R41: value 0 -> 10K
Connections:
- net +3.3V: now also R6.1
- net GND: now also C72.1
- net PDN: now also C72.2
- net at H6.2, U1.12 (GPIO0/SYNCN): now also R6.2
Other:
- moved on the sheet: H6, H7, R41
