File: hardware/schematic/v1.0/CLOCK/MAIN_CTRL.kicad_sch (KiCad schematic)
At the start: 1 part, among them U8 STM32F103CBTx

Commit message: sch update
Connections:
- net GPIO0: now also U8.25 (PB12)
- net GPIO1: now also U8.26 (PB13)
- net GPIO2: now also U8.27 (PB14)
- net PDN: now also U8.28 (PB15)
- net SCL: now also U8.21 (PB10)
- net SDA: now also U8.22 (PB11)
- net SWDIO: now reaches U8.34 (PA13)
- net SWCLK: now reaches U8.37 (PA14)
Changed lines of the file:
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@@
 	(generator_version "10.0")
 	(paper "A4")
+	(wire
+		(pts
+			(xy 83.82 121.92) (xy 87.63 121.92)
+		)
+		(stroke
+			(width 0)
+			(type default)
+		)
+	)
+	(wire
+		(pts
+			(xy 123.19 96.52) (xy 134.62 96.52)
+		)
+		(stroke
+			(width 0)
+			(type default)
+		)
+	)
+	(wire
+		(pts
+			(xy 83.82 116.84) (xy 87.63 116.84)
+		)
+		(stroke
+			(width 0)
+			(type default)
+		)
+	)
+	(wire
+		(pts
+			(xy 83.82 127) (xy 87.63 127)
+		)
+		(stroke
+			(width 0)
+			(type default)
+		)
+	)
+	(wire
+		(pts
+			(xy 83.82 114.3) (xy 87.63 114.3)
+		)
+		(stroke
+			(width 0)
+			(type default)
+		)
+	)
+	(wire
+		(pts
+			(xy 83.82 124.46) (xy 87.63 124.46)
+		)
+		(stroke
+			(width 0)
+			(type default)
+		)
+	)
+	(wire
+		(pts
+			(xy 123.19 93.98) (xy 134.62 93.98)
+		)
+		(stroke
+			(width 0)
+			(type default)
+		)
+	)
+	(wire
+		(pts
+			(xy 83.82 119.38) (xy 87.63 119.38)
+		)
+		(stroke
+			(width 0)
+			(type default)
+		)
+	)
+	(label "SWCLK"
+		(at 127 96.52 0)
+		(effects
+			(font
+				(size 1.27 1.27)
+			)
+			(justify left bottom)
+		)
+	)
+	(label "SWDIO"
+		(at 127 93.98 0)
+		(effects
+			(font
+				(size 1.27 1.27)
+			)
+			(justify left bottom)
+		)
+	)
 	(hierarchical_label "GPIO2"
 		(shape output)
-		(at 173.99 100.33 180)
+		(at 83.82 124.46 180)
 		(effects
 			(font
@@
 	(hierarchical_label "SCL"
 		(shape output)
-		(at 173.99 115.57 180)
+		(at 83.82 114.3 180)
 		(effects
 			(font
@@
 	(hierarchical_label "GPIO1"
 		(shape output)
-		(at 173.99 104.14 180)
+		(at 83.82 121.92 180)
 		(effects
 			(font
@@
 	(hierarchical_label "GPIO0"
 		(shape output)
-		(at 173.99 107.95 180)
+		(at 83.82 119.38 180)
 		(effects
 			(font
@@
 	(hierarchical_label "SDA"
 		(shape bidirectional)
-		(at 173.99 119.38 180)
+		(at 83.82 116.84 180)
 		(effects
 			(font
@@
 	(hierarchical_label "PDN"
 		(shape output)
-		(at 173.99 111.76 180)
+		(at 83.82 127 180)
 		(effects
 			(font

Commit message: sch update
Parts:
- added C64, C65, C66, C67, C68: 100nF, Capacitor_SMD:C_0402_1005Metric, symbol Device:C
Connections:
- net +3.3V: now reaches U8.1 (VBAT)
- net +3.3V: now also U8.24 (VDD), U8.36 (VDD), U8.48 (VDD), U8.9 (VDDA), C64.2, C65.2, C66.2, C67.2, C68.2
- net GND: now reaches U8.23 (VSS), U8.35 (VSS), U8.47 (VSS)
- net GND: now also U8.44 (BOOT0), U8.8 (VSSA), C64.1, C65.1, C66.1, C67.1, C68.1

Commit message: sch and pcb update
Parts:
- added C69: 100nF, Capacitor_SMD:C_0402_1005Metric, symbol Device:C
- added C70, C71: 20pF, Capacitor_SMD:C_0402_1005Metric, symbol Device:C
- added J15: Conn_01x04_Pin, Connector_PinHeader_2.54mm:PinHeader_1x04_P2.54mm_Vertical, symbol Connector:Conn_01x04_Pin
- added R39: 10K, Resistor_SMD:R_0603_1608Metric, symbol Device:R
- added X1: X32258MOB4SI, JLCImport:X32258MOB4SI, symbol JLCImport:X32258MOB4SI
Connections:
- net +3.3V: now also J15.1 (Pin_1)
- net GND: now also C69.2, C70.2, C71.2, J15.2 (Pin_2), R39.2, X1.2 (GND), X1.4 (GND); no longer U8.44 (BOOT0)
- net SWCLK: now also J15.4 (Pin_4)
- net SWDIO: now also J15.3 (Pin_3)
- net at U8.5 (PD0): now also C71.1, X1.1
- net at U8.6 (PD1): now also C70.1, X1.3
- net at U8.7 (NRST): now also C69.1
- new net: R39.1, U8.44 (BOOT0)
- no-connect marks 0 -> 27

Commit message: sch and pcb update
Parts:
- added J16: Conn_01x03_Pin, Connector_PinHeader_2.54mm:PinHeader_1x03_P2.54mm_Vertical, symbol Connector:Conn_01x03_Pin
Connections:
- net GND: now also J16.3 (Pin_3)
- net UART3_TXD: now reaches U8.12 (PA2)
- net UART3_TXD: now also J16.1 (Pin_1)
- net UART3_RXD: now reaches U8.13 (PA3)
- net UART3_RXD: now also J16.2 (Pin_2)
- no-connect marks 27 -> 25
Other:
- moved on the sheet: J15

Commit message: sch update
Parts:
- removed J15: Conn_01x04_Pin, Connector_PinHeader_2.54mm:PinHeader_1x04_P2.54mm_Vertical, symbol Connector:Conn_01x04_Pin
- added J15: Conn_01x03_Pin, Connector_PinHeader_2.54mm:PinHeader_1x03_P2.54mm_Vertical, symbol Connector:Conn_01x03_Pin
Connections:
- net GND: now also J15.3 (Pin_3)
- net SWCLK: now also J15.2 (Pin_2)
- net SWDIO: now also J15.1 (Pin_1)
Changed lines of the file:
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@@
+	(wire
+		(pts
+			(xy 170.18 100.33) (xy 179.07 100.33)
+		)
+		(stroke
+			(width 0)
+			(type default)
+		)
+	)
 	(wire
 		(pts
@@
 	(wire
 		(pts
-			(xy 170.18 105.41) (xy 172.72 105.41)
-		)
-		(stroke
-			(width 0)
-			(type default)
-		)
-	)
-	(wire
-		(pts
 			(xy 100.33 53.34) (xy 102.87 53.34)
 		)
@@
 	(wire
 		(pts
-			(xy 170.18 113.03) (xy 179.07 113.03)
-		)
-		(stroke
-			(width 0)
-			(type default)
-		)
-	)
-	(wire
-		(pts
 			(xy 143.51 43.18) (xy 156.21 43.18)
 		)
@@
 	(wire
 		(pts
-			(xy 170.18 110.49) (xy 179.07 110.49)
-		)
-		(stroke
-			(width 0)
-			(type default)
-		)
-	)
-	(wire
-		(pts
 			(xy 71.12 71.12) (xy 71.12 74.93)
 		)
@@
 	(wire
 		(pts
+			(xy 170.18 97.79) (xy 179.07 97.79)
+		)
+		(stroke
+			(width 0)
+			(type default)
+		)
+	)
+	(wire
+		(pts
 			(xy 105.41 134.62) (xy 105.41 135.89)
 		)
@@
 	(wire
 		(pts
-			(xy 170.18 107.95) (xy 177.8 107.95)
-		)
-		(stroke
-			(width 0)
-			(type default)
-		)
-	)
-	(wire
-		(pts
 			(xy 123.19 68.58) (xy 134.62 68.58)
 		)
@@
 	)
 	(label "SWCLK"
-		(at 172.72 113.03 0)
-		(effects
-			(font
-				(size 1.27 1.27)
-			)
-			(justify left bottom)
-		)
-	)
-	(label "SWDIO"
-		(at 172.72 110.49 0)
+		(at 172.72 100.33 0)
 		(effects
 			(font
@@
 	(label "UART3_TXD"
 		(at 171.45 67.31 0)
+		(effects
+			(font
+				(size 1.27 1.27)
+			)
+			(justify left bottom)
+		)
+	)
+	(label "SWDIO"
+		(at 172.72 97.79 0)
 		(effects
 			(font
@@
 	)
 	(symbol
+		(lib_id "Connector:Conn_01x03_Pin")
+		(at 165.1 100.33 0)
+		(unit 1)
+		(body_style 1)
+		(exclude_from_sim no)
+		(in_bom yes)
+		(on_board yes)
+		(in_pos_files yes)
+		(dnp no)
+		(property "Reference" "J15"
+			(at 172.466 107.95 0)
+			(show_name no)
+			(do_not_autoplace no)
+			(effects
+				(font
+					(size 1.27 1.27)
+				)
+			)
+		)
+		(property "Value" "Conn_01x03_Pin"
+			(at 172.466 110.49 0)
+			(show_name no)
+			(do_not_autoplace no)
+			(effects
+				(font
+					(size 1.27 1.27)
+				)
+			)
+		)
+		(property "Footprint" "Connector_PinHeader_2.54mm:PinHeader_1x03_P2.54mm_Vertical"
+			(at 165.1 100.33 0)
+			(hide yes)
+			(show_name no)
+			(do_not_autoplace no)
+			(effects
+				(font
+					(size 1.27 1.27)
+				)
+			)
+		)
+		(property "Datasheet" ""
+			(at 165.1 100.33 0)
+			(hide yes)
+			(show_name no)
+			(do_not_autoplace no)
+			(effects
+				(font
+					(size 1.27 1.27)
+				)
+			)
+		)
+		(property "Description" "Generic connector, single row, 01x03, script generated"
+			(at 165.1 100.33 0)
+			(hide yes)
+			(show_name no)
+			(do_not_autoplace no)
+			(effects
+				(font
+					(size 1.27 1.27)
+				)
+			)
+		)
+		(pin "3"
+		)
+		(pin "1"
+		)
+		(pin "2"
+		)
+		(instances
+			(project "CLOCK"
+				(path "/e8d80103-6a56-4030-bccc-c2b7ae1d549d/dc044937-6056-4220-ad80-6587bb362b58"
+					(reference "J15")
+					(unit 1)
+				)
+			)
+		)
+	)
+	(symbol
 		(lib_id "Device:C")
 		(at 170.18 46.99 180)
@@
 	)
 	(symbol
-		(lib_id "power:GND")
-		(at 177.8 107.95 90)
-		(unit 1)
-		(body_style 1)
-		(exclude_from_sim no)
-		(in_bom yes)
-		(on_board yes)
-		(in_pos_files yes)
-		(dnp no)
-		(fields_autoplaced yes)
-		(property "Reference" "#PWR0141"
-			(at 184.15 107.95 0)
-			(hide yes)
-			(show_name no)
-			(do_not_autoplace no)
-			(effects
-				(font
-					(size 1.27 1.27)
-				)
-			)
-		)
-		(property "Value" "GND"
-			(at 182.88 107.95 0)
-			(hide yes)
-			(show_name no)
-			(do_not_autoplace no)
-			(effects
-				(font
-					(size 1.27 1.27)
-				)
-			)
-		)
-		(property "Footprint" ""
-			(at 177.8 107.95 0)
-			(hide yes)
-			(show_name no)
-			(do_not_autoplace no)
-			(effects
-				(font
-					(size 1.27 1.27)
-				)
-			)
-		)
-		(property "Datasheet" ""
-			(at 177.8 107.95 0)
-			(hide yes)
-			(show_name no)
-			(do_not_autoplace no)
-			(effects
-				(font
-					(size 1.27 1.27)
-				)
-			)
-		)
-		(property "Description" "Power symbol creates a global label with name \"GND\" , ground"
-			(at 177.8 107.95 0)
-			(hide yes)
-			(show_name no)
-			(do_not_autoplace no)
-			(effects
-				(font
-					(size 1.27 1.27)
-				)
-			)
-		)
-		(pin "1"
-		)
-		(instances
-			(project "CLOCK"
-				(path "/e8d80103-6a56-4030-bccc-c2b7ae1d549d/dc044937-6056-4220-ad80-6587bb362b58"
-					(reference "#PWR0141")
-					(unit 1)
-				)
-			)
-		)
-	)
-	(symbol
 		(lib_id "Connector:Conn_01x03_Pin")
 		(at 165.1 69.85 0)
@@
 				(path "/e8d80103-6a56-4030-bccc-c2b7ae1d549d/dc044937-6056-4220-ad80-6587bb362b58"
 					(reference "J16")
-					(unit 1)
-				)
-			)
-		)
-	)
-	(symbol
-		(lib_id "Connector:Conn_01x04_Pin")
-		(at 165.1 107.95 0)
-		(unit 1)
-		(body_style 1)
-		(exclude_from_sim no)
-		(in_bom yes)
-		(on_board yes)
-		(in_pos_files yes)
-		(dnp no)
-		(property "Reference" "J15"
-			(at 171.196 116.332 0)
-			(show_name no)
-			(do_not_autoplace no)
-			(effects
-				(font
-					(size 1.27 1.27)
-				)
-			)
-		)
-		(property "Value" "Conn_01x04_Pin"
-			(at 171.196 118.872 0)
-			(show_name no)
-			(do_not_autoplace no)
-			(effects
-				(font
-					(size 1.27 1.27)
-				)
-			)
-		)
-		(property "Footprint" "Connector_PinHeader_2.54mm:PinHeader_1x04_P2.54mm_Vertical"
-			(at 165.1 107.95 0)
-			(hide yes)
-			(show_name no)
-			(do_not_autoplace no)
-			(effects
-				(font
-					(size 1.27 1.27)
-				)
-			)
-		)
-		(property "Datasheet" ""
-			(at 165.1 107.95 0)
-			(hide yes)
-			(show_name no)
-			(do_not_autoplace no)
-			(effects
-				(font
-					(size 1.27 1.27)
-				)
-			)
-		)
-		(property "Description" "Generic connector, single row, 01x04, script generated"
-			(at 165.1 107.95 0)
-			(hide yes)
-			(show_name no)
-			(do_not_autoplace no)
-			(effects
-				(font
-					(size 1.27 1.27)
-				)
-			)
-		)
-		(pin "1"
-		)
-		(pin "3"
-		)
-		(pin "2"
-		)
-		(pin "4"
-		)
-		(instances
-			(project "CLOCK"
-				(path "/e8d80103-6a56-4030-bccc-c2b7ae1d549d/dc044937-6056-4220-ad80-6587bb362b58"
-					(reference "J15")
 					(unit 1)
 				)
@@
 	)
 	(symbol
-		(lib_id "power:+3.3V")
-		(at 172.72 105.41 0)
+		(lib_id "power:GND")
+		(at 170.18 102.87 0)
 		(unit 1)
 		(body_style 1)
@@
 		(dnp no)
 		(fields_autoplaced yes)
-		(property "Reference" "#PWR050"
-			(at 172.72 109.22 0)
-			(hide yes)
-			(show_name no)
-			(do_not_autoplace no)
-			(effects
-				(font
-					(size 1.27 1.27)
-				)
-			)
-		)
-		(property "Value" "+3.3V"
-			(at 172.72 100.33 0)
+		(property "Reference" "#PWR0149"
+			(at 170.18 109.22 0)
+			(hide yes)
+			(show_name no)
+			(do_not_autoplace no)
+			(effects
+				(font
+					(size 1.27 1.27)
+				)
+			)
+		)
+		(property "Value" "GND"
+			(at 170.18 107.95 0)
+			(hide yes)
 			(show_name no)
 			(do_not_autoplace no)
@@
 		)
 		(property "Footprint" ""
-			(at 172.72 105.41 0)
+			(at 170.18 102.87 0)
 			(hide yes)
 			(show_name no)
@@
 		)
 		(property "Datasheet" ""
-			(at 172.72 105.41 0)
-			(hide yes)
-			(show_name no)
-			(do_not_autoplace no)
-			(effects
-				(font
-					(size 1.27 1.27)
-				)
-			)
-		)
-		(property "Description" "Power symbol creates a global label with name \"+3.3V\""
-			(at 172.72 105.41 0)
+			(at 170.18 102.87 0)
+			(hide yes)
+			(show_name no)
+			(do_not_autoplace no)
+			(effects
+				(font
+					(size 1.27 1.27)
+				)
+			)
+		)
+		(property "Description" "Power symbol creates a global label with name \"GND\" , ground"
+			(at 170.18 102.87 0)
 			(hide yes)
 			(show_name no)
@@
 			(project "CLOCK"
 				(path "/e8d80103-6a56-4030-bccc-c2b7ae1d549d/dc044937-6056-4220-ad80-6587bb362b58"
-					(reference "#PWR050")
+					(reference "#PWR0149")
 					(unit 1)
 				)

Commit message: sch update
Connections:
- net GPIO0: no longer names the net of U8.25 (PB12)
- net GPIO1: no longer names the net of U8.26 (PB13)
- net GPIO2: no longer names the net of U8.27 (PB14)
- no-connect marks 25 -> 28
Changed lines of the file:
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@@
+	)
+	(no_connect
+		(at 87.63 124.46)
 	)
 	(no_connect
@@
 	)
 	(no_connect
+		(at 87.63 119.38)
+	)
+	(no_connect
 		(at 123.19 91.44)
 	)
@@
 	)
 	(no_connect
+		(at 87.63 121.92)
+	)
+	(no_connect
 		(at 87.63 104.14)
 	)
@@
 	(wire
 		(pts
-			(xy 83.82 121.92) (xy 87.63 121.92)
-		)
-		(stroke
-			(width 0)
-			(type default)
-		)
-	)
-	(wire
-		(pts
 			(xy 68.58 91.44) (xy 73.66 91.44)
 		)
@@
 	(wire
 		(pts
-			(xy 83.82 124.46) (xy 87.63 124.46)
-		)
-		(stroke
-			(width 0)
-			(type default)
-		)
-	)
-	(wire
-		(pts
 			(xy 73.66 73.66) (xy 73.66 91.44)
 		)
@@
 		(pts
 			(xy 71.12 71.12) (xy 71.12 74.93)
-		)
-		(stroke
-			(width 0)
-			(type default)
-		)
-	)
-	(wire
-		(pts
-			(xy 83.82 119.38) (xy 87.63 119.38)
 		)
 		(stroke
@@
 			)
 			(justify left bottom)
-		)
-	)
-	(hierarchical_label "GPIO2"
-		(shape output)
-		(at 83.82 124.46 180)
-		(effects
-			(font
-				(size 1.27 1.27)
-			)
-			(justify right)
 		)
 	)
@@
 		(effects
 			(font
-				(size 1.27 1.27)
-			)
-			(justify right)
-		)
-	)
-	(hierarchical_label "GPIO1"
-		(shape output)
-		(at 83.82 121.92 180)
-		(effects
-			(font
-				(size 1.27 1.27)
-			)
-			(justify right)
-		)
-	)
-	(hierarchical_label "GPIO0"
-		(shape output)
-		(at 83.82 119.38 180)
-		(effects
-			(font

Commit message: sch and pcb update
Parts:
- added R35, R40, R42: 0, Resistor_SMD:R_0402_1005Metric, symbol Device:R
Connections:
- net PDN: now also R40.1; no longer U8.28 (PB15)
- net SCL: now also R42.1; no longer U8.21 (PB10)
- net SDA: now also R35.2; no longer U8.22 (PB11)
- new net: R35.1, U8.22 (PB11)
- new net: R40.2, U8.28 (PB15)
- new net: R42.2, U8.21 (PB10)
