File: hardware/schematic/v1.0/CLOCK_CORE/SIGNAL.kicad_sch (KiCad schematic)
At the start: 30 parts, among them J1 Conn_Coaxial

Commit message: sch and pcb update
Connections:
- net OUT2_N_RF: now reaches C5.1, R7.2, RF5.4 (SIG)
- net OUT3_N_RF: now reaches C7.1, R10.2, RF7.4 (SIG)
- net OUT1_N_RF: now reaches C4.2, R5.1, RF4.4 (SIG)
- net OUT2_P_RF: now reaches C6.2, R8.1, RF6.4 (SIG)
- net OUT3_P_RF: now reaches C8.2, R11.1, RF8.4 (SIG)
- net OUT0_P_RF: now reaches C2.2, R2.1, RF2.4 (SIG)
- net OUT0_N_RF: now reaches C1.1, R1.2, RF1.4 (SIG)
- net OUT1_P_RF: now reaches C3.1, R4.2, RF3.4 (SIG)
Changed lines of the file:
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@@
+		)
+	)
+	(label "OUT0_P_RF"
+		(at 76.2 68.58 0)
+		(effects
+			(font
+				(size 1.27 1.27)
+			)
+			(justify left bottom)
+		)
+	)
+	(label "OUT3_N_RF"
+		(at 207.01 107.95 0)
+		(effects
+			(font
+				(size 1.27 1.27)
+			)
+			(justify left bottom)
+		)
+	)
+	(label "OUT3_P_RF"
+		(at 215.9 143.51 0)
+		(effects
+			(font
+				(size 1.27 1.27)
+			)
+			(justify left bottom)
+		)
+	)
+	(label "OUT2_N_RF"
+		(at 207.01 34.29 0)
+		(effects
+			(font
+				(size 1.27 1.27)
+			)
+			(justify left bottom)
+		)
+	)
+	(label "OUT1_P_RF"
+		(at 67.31 107.95 0)
+		(effects
+			(font
+				(size 1.27 1.27)
+			)
+			(justify left bottom)
+		)
+	)
+	(label "OUT0_N_RF"
+		(at 67.31 33.02 0)
+		(effects
+			(font
+				(size 1.27 1.27)
+			)
+			(justify left bottom)
+		)
+	)
+	(label "OUT2_P_RF"
+		(at 215.9 69.85 0)
+		(effects
+			(font
+				(size 1.27 1.27)
+			)
+			(justify left bottom)
+		)
+	)
+	(label "OUT1_N_RF"
+		(at 76.2 143.51 0)
+		(effects
+			(font
+				(size 1.27 1.27)
+			)
+			(justify left bottom)
 		)
 	)

Commit message: sch and pcb update
Parts:
- added R31, R32, R33, R34, R35, R36, R37, R38: 0, Resistor_SMD:R_0402_1005Metric, symbol Device:R
Connections:
- net OUT0_N: now also R31.1; no longer C1.2, R3.2
- net OUT0_P: now also R32.1; no longer C2.1, R3.1
- net OUT1_N: now also R34.1; no longer C4.1, R6.1
- net OUT1_P: now also R33.1; no longer C3.2, R6.2
- net OUT2_N: now also R35.1; no longer C5.2, R9.2
- net OUT2_P: now also R36.1; no longer C6.1, R9.1
- net OUT3_N: now also R37.1; no longer C7.2, R12.2
- net OUT3_P: now also R38.1; no longer C8.1, R12.1
- net OUT0_N_RF renamed IPEX_O0_N
- net OUT0_P_RF renamed IPEX_O0_P
- net OUT1_N_RF renamed IPEX_O1_N
- net OUT1_P_RF renamed IPEX_O1_P
- net OUT2_N_RF renamed IPEX_O2_N
- net OUT2_P_RF renamed IPEX_O2_P
- net OUT3_N_RF renamed IPEX_O3_N
- net OUT3_P_RF renamed IPEX_O3_P
- new net O0_N: C1.2, R3.2, R31.2
- new net O0_P: C2.1, R3.1, R32.2
- new net O1_N: C4.1, R34.2, R6.1
- new net O1_P: C3.2, R33.2, R6.2
- new net O2_N: C5.2, R35.2, R9.2
- new net O2_P: C6.1, R36.2, R9.1
- new net O3_N: C7.2, R12.2, R37.2
- new net O3_P: C8.1, R12.1, R38.2

Commit message: sch and pcb update
Parts:
- C1, C2, C3, C4, C5, C6, C7, C8: footprint Capacitor_SMD:C_0402_1005Metric -> CLOCK_CORE:C_0402_1005Metric; symbol Device:C -> CLOCK_CORE:C
- J1: footprint Connector_Coaxial:SMA_Amphenol_132134-11_Vertical -> CLOCK_CORE:SMA_Amphenol_132134-11_Vertical; symbol Connector:Conn_Coaxial -> CLOCK_CORE:Conn_Coaxial
- R1, R10, R11, R12, R2, R3, R31, R32, R33, R34, R35, R36, R37, R38, R4, R5, R6, R7, R8, R9: footprint Resistor_SMD:R_0402_1005Metric -> CLOCK_CORE:R_0402_1005Metric; symbol Device:R -> CLOCK_CORE:R
- RF1, RF2, RF3, RF4, RF5, RF6, RF7, RF8, RF9: footprint JLCImport:KH-IPEX-K501-29 -> CLOCK_CORE:KH-IPEX-K501-29; symbol JLCImport:KH-IPEX-K501-29 -> CLOCK_CORE:KH-IPEX-K501-29

Commit message: sch and pcb update
Parts:
- R12, R3, R6, R9: value DNP -> 100; now not fitted
Changed lines of the file:
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@@
 		(on_board yes)
 		(in_pos_files yes)
-		(dnp no)
+		(dnp yes)
 		(property "Reference" "R9"
 			(at 240.284 53.594 0)
@@
 			)
 		)
-		(property "Value" "DNP"
+		(property "Value" "100"
 			(at 240.792 51.054 0)
 			(show_name no)
@@
 		(on_board yes)
 		(in_pos_files yes)
-		(dnp no)
+		(dnp yes)
 		(property "Reference" "R12"
 			(at 240.284 127.254 0)
@@
 			)
 		)
-		(property "Value" "DNP"
+		(property "Value" "100"
 			(at 240.792 124.714 0)
 			(show_name no)
@@
 		(on_board yes)
 		(in_pos_files yes)
-		(dnp no)
+		(dnp yes)
 		(property "Reference" "R3"
 			(at 100.584 52.324 0)
@@
 			)
 		)
-		(property "Value" "DNP"
+		(property "Value" "100"
 			(at 101.092 49.784 0)
 			(show_name no)
@@
 		(on_board yes)
 		(in_pos_files yes)
-		(dnp no)
+		(dnp yes)
 		(property "Reference" "R6"
 			(at 100.584 127.254 0)
@@
 			)
 		)
-		(property "Value" "DNP"
+		(property "Value" "100"
 			(at 101.092 124.714 0)
 			(show_name no)
