File: hardware/schematic/v1.0/CLOCK_CORE/LMK5B12204.kicad_sch (KiCad schematic)
At the start: 46 parts, among them U1 LMK5B12204

Commit message: sch update
Parts:
- removed H7: HX_PH254-01-03-Z-L11_5_PCB_PIN_HEADER, JLCImport:HX_PH254-01-03-Z-L11_5_PCB_PIN_HEADER, symbol JLCImport:HX_PH254-01-03-Z-L11_5_PCB_PIN_HEADER
- removed R41: 10K, Resistor_SMD:R_0402_1005Metric, symbol Device:R
Connections:
- net PDN renamed PLL_PG

Commit message: sch update
Changed lines of the file:
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@@
 	)
 	(hierarchical_label "OUT1_N"
-		(shape input)
+		(shape output)
 		(at 156.21 121.92 270)
 		(effects
@@
 	)
 	(hierarchical_label "OUT3_P"
-		(shape bidirectional)
+		(shape output)
 		(at 144.78 64.77 90)
 		(effects

Commit message: sch update
Changed lines of the file:
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@@
 		(property "Value" "GND"
 			(at 134.62 58.42 0)
+			(hide yes)
 			(show_name no)
 			(do_not_autoplace no)
@@
 		(property "Value" "GND"
 			(at 113.03 58.42 0)
-			(show_name no)
-			(do_not_autoplace no)
+			(hide yes)
+			(show_name no)
+			(do_not_autoplace no)
