File: hardware/schematic/v1.0/CLOCK_CORE/LMK5B12204.kicad_sch (KiCad schematic)
At the start: 44 parts, among them U5 LMK5B12204

Commit message: sch and pcb update
Connections:
- net HW_SW_CTRL: now reaches R24.2, U5.9 (HW_SW_CTRL)
- net SYNCN: now reaches H1.2, R25.2, U5.12 (GPIO0/SYNCN)
- net PLL_PG renamed PDN
- net XO_P renamed OCXO_OUT
Changed lines of the file:
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@@
+		)
+	)
+	(label "HW_SW_CTRL"
+		(at 121.92 99.06 0)
+		(effects
+			(font
+				(size 1.27 1.27)
+			)
+			(justify left bottom)
+		)
+	)
+	(label "SYNCN"
+		(at 109.22 106.68 0)
+		(effects
+			(font
+				(size 1.27 1.27)
+			)
+			(justify left bottom)
 		)
 	)
@@
 		)
 	)
-	(hierarchical_label "XO_P"
+	(hierarchical_label "OCXO_OUT"
 		(shape input)
 		(at 179.07 91.44 0)
@@
 		)
 	)
-	(hierarchical_label "PLL_PG"
+	(hierarchical_label "PDN"
 		(shape input)
 		(at 135.89 129.54 270)

Commit message: sch and pcb update
Parts:
- added C59: 100nF, Capacitor_SMD:C_0402_1005Metric, symbol Device:C
Connections:
- net GND: now also C59.1
- net VDDXO: now also C59.2

Commit message: sch and pcb update
Parts:
- C27, C28, C29, C30, C31, C32, C33, C34, C35, C36, C37, C38, C39, C40, C41, C42, C43, C44, C45, C46, C47, C48, C49, C50, C51, C52, C53, C54, C55, C59: footprint Capacitor_SMD:C_0402_1005Metric -> CLOCK_CORE:C_0402_1005Metric; symbol Device:C -> CLOCK_CORE:C
- D1, D2: footprint LED_SMD:LED_0603_1608Metric -> CLOCK_CORE:LED_0603_1608Metric; symbol Device:LED -> CLOCK_CORE:LED
- FB1, FB2, FB3, FB4, FB5, FB6, FB7: footprint Inductor_SMD:L_0603_1608Metric -> CLOCK_CORE:L_0603_1608Metric; symbol Device:FerriteBead_Small -> CLOCK_CORE:FerriteBead_Small
- H1: footprint JLCImport:HX_PH254-01-03-Z-L11_5_PCB_PIN_HEADER -> CLOCK_CORE:HX_PH254-01-03-Z-L11_5_PCB_PIN_HEADER; symbol JLCImport:HX_PH254-01-03-Z-L11_5_PCB_PIN_HEADER -> CLOCK_CORE:HX_PH254-01-03-Z-L11_5_PCB_PIN_HEADER
- R24: footprint Resistor_SMD:R_0402_1005Metric -> CLOCK_CORE:R_0402_1005Metric; symbol Device:R -> CLOCK_CORE:R
- R25, R26, R27: footprint Resistor_SMD:R_0603_1608Metric -> CLOCK_CORE:R_0603_1608Metric; symbol Device:R -> CLOCK_CORE:R
- U5: footprint Package_DFN_QFN:VQFN-48-1EP_7x7mm_P0.5mm_EP5.15x5.15mm_ThermalVias -> CLOCK_CORE:VQFN-48-1EP_7x7mm_P0.5mm_EP5.15x5.15mm_ThermalVias; symbol Counter:LMK5B12204 -> CLOCK_CORE:LMK5B12204
