File: hardware/schematic/v1.0/CLOCK_CORE/OCXO.kicad_sch (KiCad schematic)
At the start: 0 parts

Commit message: sch update
Parts:
- added C48: 10uF, Capacitor_SMD:C_0603_1608Metric, symbol Device:C
- added C49, C51, C52: 100nF, Capacitor_SMD:C_0402_1005Metric, symbol Device:C
- added C50: 1uF, Capacitor_SMD:C_0402_1005Metric, symbol Device:C
- added H1: HX_PH254-01-03-Z-L11_5_PCB_PIN_HEADER, JLCImport:HX_PH254-01-03-Z-L11_5_PCB_PIN_HEADER, symbol JLCImport:HX_PH254-01-03-Z-L11_5_PCB_PIN_HEADER
- added J12: Conn_Coaxial, Connector_Coaxial:SMA_Amphenol_132289_EdgeMount, symbol Connector:Conn_Coaxial
- added R13: 3296W-1-103_C48997937, Counter:3296W-1-103_C48997937, symbol Counter:3296W-1-103_C48997937
- added R33, R34: 1K, Resistor_SMD:R_0402_1005Metric, symbol Device:R
- added TP1: Volt TestPoint, TestPoint:TestPoint_Pad_D1.0mm, symbol Connector:TestPoint
- added TP2: TestPoint, TestPoint:TestPoint_Loop_D1.80mm_Drill1.0mm_Beaded, symbol Connector:TestPoint
- added U6: OCXO-10M, JLCImport:DOPFITKR2-10M, symbol Counter:OCXO-10M
Connections:
- new net: C52.1, J12.1 (In)
- new net: C51.1, R33.2, U6.3 (VCTRL)
- new net: C48.2, C49.1, C50.2, H1.2, TP1.1, U6.5 (VCC)
- new net: R13.3, U6.4 (VREF)
- new net: C52.2, R34.2
- new net: R13.2, R33.1
- new net +3.3V_OCXO: H1.1
- new net +5V_OCXO: H1.3
- new net GND: C48.1, C49.2, C50.1, C51.2, J12.2 (Ext), R13.1, TP2.1, U6.2 (GND)
- new net XO_P: R34.1, U6.1 (RF)
Other:
- note added: "50 OHM TRACE"
- note added: "OCXO"

Commit message: sch update
Changed lines of the file:
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@@
 		)
 	)
-	(global_label "XO_P"
+	(hierarchical_label "XO_P"
 		(shape output)
 		(at 101.6 91.44 180)
-		(fields_autoplaced yes)
 		(effects
 			(font
@@
 			(justify right)
 		)
-		(property "Intersheetrefs" "${INTERSHEET_REFS}"
-			(at 93.8372 91.44 0)
-			(hide yes)
-			(show_name no)
-			(do_not_autoplace no)
-			(effects
-				(font
-					(size 1.27 1.27)
-				)
-				(justify right)
-			)
-		)
 	)

Commit message: sch update
Parts:
- removed H1: HX_PH254-01-03-Z-L11_5_PCB_PIN_HEADER, JLCImport:HX_PH254-01-03-Z-L11_5_PCB_PIN_HEADER, symbol JLCImport:HX_PH254-01-03-Z-L11_5_PCB_PIN_HEADER
- removed U6: OCXO-10M, JLCImport:DOPFITKR2-10M, symbol Counter:OCXO-10M
- added U4: OCXO_25.4x25.4mm, JLCImport:DOPFITKR2-10M, symbol Counter:OCXO_25.4x25.4mm
- added U5: OCXO_20x20mm, JLCImport:OCXO_20x20mm, symbol Counter:OCXO_20x20mm
Connections:
- net GND: now also U4.2 (GND)
- net XO_P: now also U4.1 (RF)
- net at C51.1, R33.2: now also U4.3 (VCTRL)
- net OCXO_VCC: now reaches C48.2, C49.1, C50.2, TP1.1
- net OCXO_VCC: now also U4.5 (VCC)
- net at R13.3: now also U4.4 (VREF/NC)
Other:
- note added: "OCXO 20x20mm"
- note added: "OCXO 25.4x25.4mm"
- note removed: "OCXO"
- moved on the sheet: C48, C49, C50, C51, C52, J12, R13, R33, R34, TP1, TP2

Commit message: sch update
Connections:
- net XO_P is gone; now on net RF: R34.1, U4.1 (RF)
- net GND: now also U5.3 (GND)
- net OCXO_VCC: now also U5.1 (VCC)
- net VCTRL: now reaches C51.1, R33.2, U4.3 (VCTRL)
- net VCTRL: now also U5.4 (VCTRL/NC)
- net VREF: now reaches R13.3, U4.4 (VREF/NC)
- net VREF: now also U5.5 (VREF/NC)
- net RF: now reaches U5.2 (RF)
Other:
- moved on the sheet: C48, C49, C50, C52, J12, R34, TP1
