File: hardware/schematic/v1.0/CLOCK_CORE/OCXO.kicad_sch (KiCad schematic)
At the start: 13 parts, among them U1 OCXO_20x20mm, U2 OCXO_25.4x25.4mm

Commit message: sch and pcb update
Connections:
- net OCXO_MON: now reaches C9.2, R13.2
- net VCTRL_ADJ: now reaches R14.1, R15.2
- net OCXO_MON_RF: now reaches C9.1, RF10.4 (SIG)
- net RF renamed OCXO_OUT
Changed lines of the file:
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@@
 		)
 	)
-	(global_label "RF"
+	(label "OCXO_MON_RF"
+		(at 88.9 105.41 0)
+		(effects
+			(font
+				(size 1.27 1.27)
+			)
+			(justify left bottom)
+		)
+	)
+	(label "OCXO_MON"
+		(at 96.52 115.57 90)
+		(effects
+			(font
+				(size 1.27 1.27)
+			)
+			(justify left bottom)
+		)
+	)
+	(label "VCTRL_ADJ"
+		(at 118.11 147.32 270)
+		(effects
+			(font
+				(size 1.27 1.27)
+			)
+			(justify right bottom)
+		)
+	)
+	(global_label "OCXO_OUT"
 		(shape output)
 		(at 116.84 57.15 180)
@@
 		)
 	)
-	(global_label "RF"
+	(global_label "OCXO_OUT"
 		(shape input)
 		(at 110.49 115.57 90)
@@
 		)
 	)
-	(hierarchical_label "XO_P"
+	(hierarchical_label "OCXO_OUT"
 		(shape output)
 		(at 95.25 125.73 180)

Commit message: sch and pcb update
Parts:
- removed C11: 1uF, Capacitor_SMD:C_0402_1005Metric, symbol Device:C
Other:
- moved on the sheet: C12
Changed lines of the file:
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@@
+	)
+	(junction
+		(at 156.21 116.84)
+		(diameter 0)
+		(color 0 0 0 0)
 	)
 	(junction
@@
 	)
 	(junction
-		(at 160.02 116.84)
-		(diameter 0)
-		(color 0 0 0 0)
-	)
-	(junction
-		(at 167.64 125.73)
+		(at 160.02 125.73)
 		(diameter 0)
 		(color 0 0 0 0)
@@
 	)
 	(junction
-		(at 160.02 125.73)
-		(diameter 0)
-		(color 0 0 0 0)
-	)
-	(junction
 		(at 110.49 125.73)
 		(diameter 0)
@@
 	(wire
 		(pts
-			(xy 167.64 124.46) (xy 167.64 125.73)
+			(xy 160.02 124.46) (xy 160.02 125.73)
 		)
 		(stroke
@@
 	(wire
 		(pts
-			(xy 160.02 116.84) (xy 167.64 116.84)
+			(xy 160.02 125.73) (xy 175.26 125.73)
 		)
 		(stroke
@@
 		)
 	)
-	(wire
-		(pts
-			(xy 160.02 125.73) (xy 167.64 125.73)
-		)
-		(stroke
-			(width 0)
-			(type default)
-		)
-	)
 	(polyline
 		(pts
@@
 	(wire
 		(pts
-			(xy 160.02 115.57) (xy 160.02 116.84)
+			(xy 156.21 115.57) (xy 156.21 116.84)
 		)
 		(stroke
@@
 	(wire
 		(pts
-			(xy 152.4 116.84) (xy 160.02 116.84)
+			(xy 152.4 116.84) (xy 156.21 116.84)
 		)
 		(stroke
@@
 	(wire
 		(pts
-			(xy 167.64 125.73) (xy 175.26 125.73)
-		)
-		(stroke
-			(width 0)
-			(type default)
-		)
-	)
-	(wire
-		(pts
-			(xy 160.02 124.46) (xy 160.02 125.73)
+			(xy 156.21 116.84) (xy 160.02 116.84)
 		)
 		(stroke
@@
 	(symbol
 		(lib_id "Device:C")
-		(at 167.64 120.65 0)
+		(at 160.02 120.65 0)
 		(unit 1)
 		(body_style 1)
@@
 		(dnp no)
 		(property "Reference" "C12"
-			(at 171.958 118.11 0)
+			(at 164.338 118.11 0)
 			(show_name no)
 			(do_not_autoplace no)
@@
 		)
 		(property "Value" "10uF"
-			(at 174.244 123.444 0)
+			(at 166.624 123.444 0)
 			(show_name no)
 			(do_not_autoplace no)
@@
 		)
 		(property "Footprint" "Capacitor_SMD:C_0603_1608Metric"
-			(at 168.6052 124.46 0)
+			(at 160.9852 124.46 0)
 			(hide yes)
 			(show_name no)
@@
 		)
 		(property "Datasheet" ""
-			(at 167.64 120.65 0)
+			(at 160.02 120.65 0)
 			(hide yes)
 			(show_name no)
@@
 		)
 		(property "Description" "Unpolarized capacitor"
-			(at 167.64 120.65 0)
+			(at 160.02 120.65 0)
 			(hide yes)
 			(show_name no)
@@
 	(symbol
 		(lib_id "power:GND")
-		(at 160.02 115.57 180)
+		(at 156.21 115.57 180)
 		(unit 1)
 		(body_style 1)
@@
 		(fields_autoplaced yes)
 		(property "Reference" "#PWR03"
-			(at 160.02 109.22 0)
+			(at 156.21 109.22 0)
 			(hide yes)
 			(show_name no)
@@
 		)
 		(property "Value" "GND"
-			(at 160.02 110.49 0)
+			(at 156.21 110.49 0)
 			(hide yes)
 			(show_name no)
@@
 		)
 		(property "Footprint" ""
-			(at 160.02 115.57 0)
+			(at 156.21 115.57 0)
 			(hide yes)
 			(show_name no)
@@
 		)
 		(property "Datasheet" ""
-			(at 160.02 115.57 0)
+			(at 156.21 115.57 0)
 			(hide yes)
 			(show_name no)
@@
 		)
 		(property "Description" "Power symbol creates a global label with name \"GND\" , ground"
-			(at 160.02 115.57 0)
+			(at 156.21 115.57 0)
 			(hide yes)
 			(show_name no)
@@
 					(unit 1)
 				)
-			)
-		)
-	)
-	(symbol
-		(lib_id "Device:C")
-		(at 160.02 120.65 0)
-		(unit 1)
-		(body_style 1)
-		(exclude_from_sim no)
-		(in_bom yes)
-		(on_board yes)
-		(in_pos_files yes)
-		(dnp no)
-		(property "Reference" "C11"
-			(at 164.338 118.11 0)
-			(show_name no)
-			(do_not_autoplace no)
-			(effects
-				(font
-					(size 1.27 1.27)
-				)
-				(justify right)
-			)
-		)
-		(property "Value" "1uF"
-			(at 164.846 123.19 0)
-			(show_name no)
-			(do_not_autoplace no)
-			(effects
-				(font
-					(size 1.27 1.27)
-				)
-				(justify right)
-			)
-		)
-		(property "Footprint" "Capacitor_SMD:C_0402_1005Metric"
-			(at 160.9852 124.46 0)
-			(hide yes)
-			(show_name no)
-			(do_not_autoplace no)
-			(effects
-				(font
-					(size 1.27 1.27)
-				)
-			)
-		)
-		(property "Datasheet" ""
-			(at 160.02 120.65 0)
-			(hide yes)
-			(show_name no)
-			(do_not_autoplace no)
-			(effects
-				(font
-					(size 1.27 1.27)
-				)
-			)
-		)
-		(property "Description" "Unpolarized capacitor"
-			(at 160.02 120.65 0)
-			(hide yes)
-			(show_name no)
-			(do_not_autoplace no)
-			(effects
-				(font
-					(size 1.27 1.27)
-				)
-			)
-		)
-		(pin "1"
-		)
-		(pin "2"
-		)
-		(instances
-			(project "CLOCK_CORE"
-				(path "/a25f2a35-4889-4be5-9b80-12803bbbfe96/645fcd89-025a-4233-88ed-d1f363faa68e"
-					(reference "C11")
-					(unit 1)
-				)

Commit message: sch and pcb update
Parts:
- added C11: 100nF, Capacitor_SMD:C_0402_1005Metric, symbol Device:C
- added C56, C58: 10uF, Capacitor_SMD:C_0603_1608Metric, symbol Device:C
- added C57: 1uF, Capacitor_SMD:C_0603_1608Metric, symbol Device:C
- added R28: 10R, Resistor_SMD:R_0603_1608Metric, symbol Device:R
- added R29: 0R, Resistor_SMD:R_0603_1608Metric, symbol Device:R
- added U6: REF5040, JLCImport:REF5040, symbol JLCImport:REF5040
Connections:
- net GND: now also C11.1, C56.2, C57.2, C58.2, U6.4 (GND)
- net OCXO_VCC: now also R28.2
- net VREF: now also R29.2; no longer U1.5 (VREF/NC), U2.4 (VREF/NC)
- new net: C11.2, C56.1, R28.1, U6.2 (VIN)
- new net: C57.1, U6.5 (TRIM/NR)
- new net: C58.1, R29.1, U6.6 (VOUT)
- no-connect marks 0 -> 6
Other:
- note added: "VREF"

Commit message: sch and pcb update
Changed lines of the file:
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@@
 	(wire
 		(pts
-			(xy 264.16 46.99) (xy 264.16 49.53)
+			(xy 264.16 34.29) (xy 264.16 49.53)
 		)
 		(stroke
@@
 	)
 	(label "VREF"
-		(at 264.16 46.99 90)
+		(at 264.16 34.29 90)
 		(effects
 			(font

Commit message: sch and pcb update
Parts:
- U1: now not fitted
Other:
- note added: "OCXO 二选一"
Changed lines of the file:
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@@
+		)
+	)
+	(text "OCXO 二选一"
+		(exclude_from_sim no)
+		(at 48.768 50.292 0)
+		(effects
+			(font
+				(size 1.27 1.27)
+			)
+			(justify left bottom)
 		)
 	)
@@
 		(on_board yes)
 		(in_pos_files yes)
-		(dnp no)
+		(dnp yes)
 		(fields_autoplaced yes)
 		(property "Reference" "U1"

Commit message: sch and pcb update
Parts:
- added R30: 0R, Resistor_SMD:R_0402_1005Metric, symbol Device:R
- added R39: 0R, Resistor_SMD:R_0805_2012Metric, symbol Device:R
Connections:
- net OCXO_OUT: now also R30.1; no longer U1.2 (RF)
- net OCXO_VCC: now also R39.2; no longer U1.1 (VCC)
- new net: R30.2, U1.2 (RF)
- new net: R39.1, U1.1 (VCC)
Changed lines of the file:
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@@
+	(wire
+		(pts
+			(xy 115.57 53.34) (xy 119.38 53.34)
+		)
+		(stroke
+			(width 0)
+			(type default)
+		)
+	)
 	(wire
 		(pts
@@
 	(wire
 		(pts
-			(xy 116.84 53.34) (xy 119.38 53.34)
+			(xy 105.41 53.34) (xy 107.95 53.34)
 		)
 		(stroke
@@
 	(wire
 		(pts
+			(xy 114.3 66.04) (xy 114.3 64.77)
+		)
+		(stroke
+			(width 0)
+			(type default)
+		)
+	)
+	(wire
+		(pts
 			(xy 143.51 125.73) (xy 147.32 125.73)
 		)
@@
 	(wire
 		(pts
+			(xy 114.3 57.15) (xy 119.38 57.15)
+		)
+		(stroke
+			(width 0)
+			(type default)
+		)
+	)
+	(wire
+		(pts
 			(xy 110.49 125.73) (xy 118.11 125.73)
 		)
@@
 		(pts
 			(xy 215.9 45.72) (xy 215.9 46.99)
-		)
-		(stroke
-			(width 0)
-			(type default)
-		)
-	)
-	(wire
-		(pts
-			(xy 116.84 57.15) (xy 119.38 57.15)
 		)
 		(stroke
@@
 		)
 	)
-	(global_label "OCXO_OUT"
-		(shape output)
-		(at 116.84 57.15 180)
+	(global_label "OCXO_VCC"
+		(shape input)
+		(at 105.41 53.34 180)
 		(fields_autoplaced yes)
 		(effects
@@
 		)
 		(property "Intersheetrefs" "${INTERSHEET_REFS}"
-			(at 111.4962 57.15 0)
+			(at 92.6881 53.34 0)
 			(hide yes)
 			(show_name no)
@@
 		)
 	)
-	(global_label "OCXO_VCC"
-		(shape input)
-		(at 116.84 53.34 180)
+	(global_label "OCXO_OUT"
+		(shape output)
+		(at 114.3 66.04 270)
 		(fields_autoplaced yes)
 		(effects
@@
 		)
 		(property "Intersheetrefs" "${INTERSHEET_REFS}"
-			(at 104.1181 53.34 0)
+			(at 114.3 78.7619 90)
 			(hide yes)
 			(show_name no)
@@
 	(symbol
 		(lib_id "Device:R")
+		(at 114.3 60.96 180)
+		(unit 1)
+		(body_style 1)
+		(exclude_from_sim no)
+		(in_bom yes)
+		(on_board yes)
+		(in_pos_files yes)
+		(dnp no)
+		(property "Reference" "R30"
+			(at 112.776 59.69 0)
+			(show_name no)
+			(do_not_autoplace no)
+			(effects
+				(font
+					(size 1.27 1.27)
+				)
+				(justify left)
+			)
+		)
+		(property "Value" "0R"
+			(at 112.522 62.484 0)
+			(show_name no)
+			(do_not_autoplace no)
+			(effects
+				(font
+					(size 1.27 1.27)
+				)
+				(justify left)
+			)
+		)
+		(property "Footprint" "Resistor_SMD:R_0402_1005Metric"
+			(at 116.078 60.96 90)
+			(hide yes)
+			(show_name no)
+			(do_not_autoplace no)
+			(effects
+				(font
+					(size 1.27 1.27)
+				)
+			)
+		)
+		(property "Datasheet" ""
+			(at 114.3 60.96 0)
+			(hide yes)
+			(show_name no)
+			(do_not_autoplace no)
+			(effects
+				(font
+					(size 1.27 1.27)
+				)
+			)
+		)
+		(property "Description" "Resistor"
+			(at 114.3 60.96 0)
+			(hide yes)
+			(show_name no)
+			(do_not_autoplace no)
+			(effects
+				(font
+					(size 1.27 1.27)
+				)
+			)
+		)
+		(pin "2"
+		)
+		(pin "1"
+		)
+		(instances
+			(project "CLOCK_CORE"
+				(path "/a25f2a35-4889-4be5-9b80-12803bbbfe96/645fcd89-025a-4233-88ed-d1f363faa68e"
+					(reference "R30")
+					(unit 1)
+				)
+			)
+		)
+	)
+	(symbol
+		(lib_id "Device:R")
 		(at 215.9 50.8 180)
 		(unit 1)
@@
 					(unit 1)
 				)
+			)
+		)
+	)
+	(symbol
+		(lib_id "Device:R")
+		(at 111.76 53.34 270)
+		(unit 1)
+		(body_style 1)
+		(exclude_from_sim no)
+		(in_bom yes)
+		(on_board yes)
+		(in_pos_files yes)
+		(dnp no)
+		(property "Reference" "R39"
+			(at 109.728 50.546 90)
+			(show_name no)
+			(do_not_autoplace no)
+			(effects
+				(font
+					(size 1.27 1.27)
+				)
+				(justify left)
+			)
+		)
+		(property "Value" "0R"
+			(at 110.49 55.88 90)
+			(show_name no)
+			(do_not_autoplace no)
+			(effects
+				(font
+					(size 1.27 1.27)
+				)
+				(justify left)
+			)
+		)
+		(property "Footprint" "Resistor_SMD:R_0805_2012Metric"
+			(at 111.76 51.562 90)
+			(hide yes)
+			(show_name no)
+			(do_not_autoplace no)
+			(effects
+				(font
+					(size 1.27 1.27)
+				)
+			)
+		)
+		(property "Datasheet" ""
+			(at 111.76 53.34 0)
+			(hide yes)
+			(show_name no)
+			(do_not_autoplace no)
+			(effects
+				(font
+					(size 1.27 1.27)
+				)
+			)
+		)
+		(property "Description" "Resistor"
+			(at 111.76 53.34 0)
+			(hide yes)
+			(show_name no)
+			(do_not_autoplace no)
+			(effects
+				(font
+					(size 1.27 1.27)
+				)
+			)
+		)
+		(pin "2"
+		)
+		(pin "1"
+		)
+		(instances
+			(project "CLOCK_CORE"
+				(path "/a25f2a35-4889-4be5-9b80-12803bbbfe96/645fcd89-025a-4233-88ed-d1f363faa68e"
+					(reference "R39")
+					(unit 1)
+				)

Commit message: sch and pcb update
Changed lines of the file:
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@@
 	(text "OCXO 二选一"
 		(exclude_from_sim no)
-		(at 48.768 50.292 0)
+		(at 173.228 39.116 0)
 		(effects
 			(font

Commit message: sch and pcb update
Connections:
- net OCXO_VCC: no longer R28.2
- new net +5V: R28.2
Changed lines of the file:
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@@
 	(wire
 		(pts
-			(xy 264.16 34.29) (xy 264.16 49.53)
+			(xy 264.16 44.45) (xy 264.16 49.53)
 		)
 		(stroke
@@
 	)
 	(label "VREF"
-		(at 264.16 34.29 90)
+		(at 264.16 44.45 90)
 		(effects
 			(font
@@
 			)
 			(justify right)
-		)
-	)
-	(hierarchical_label "OCXO_VCC"
-		(shape input)
-		(at 215.9 45.72 90)
-		(effects
-			(font
-				(size 1.27 1.27)
-			)
-			(justify left)
 		)
 	)
@@
 					(unit 1)
 				)
+			)
+		)
+	)
+	(symbol
+		(lib_id "power:+5V")
+		(at 215.9 45.72 0)
+		(unit 1)
+		(body_style 1)
+		(exclude_from_sim no)
+		(in_bom yes)
+		(on_board yes)
+		(in_pos_files yes)
+		(dnp no)
+		(property "Reference" "#PWR0139"
+			(at 215.9 49.53 0)
+			(hide yes)
+			(show_name no)
+			(do_not_autoplace no)
+			(effects
+				(font
+					(size 1.27 1.27)
+				)
+			)
+		)
+		(property "Value" "+5V"
+			(at 214.122 41.656 0)
+			(show_name no)
+			(do_not_autoplace no)
+			(effects
+				(font
+					(size 1.27 1.27)
+				)
+				(justify left)
+			)
+		)
+		(property "Footprint" ""
+			(at 215.9 45.72 0)
+			(hide yes)
+			(show_name no)
+			(do_not_autoplace no)
+			(effects
+				(font
+					(size 1.27 1.27)
+				)
+			)
+		)
+		(property "Datasheet" ""
+			(at 215.9 45.72 0)
+			(hide yes)
+			(show_name no)
+			(do_not_autoplace no)
+			(effects
+				(font
+					(size 1.27 1.27)
+				)
+			)
+		)
+		(property "Description" ""
+			(at 215.9 45.72 0)
+			(hide yes)
+			(show_name no)
+			(do_not_autoplace no)
+			(effects
+				(font
+					(size 1.27 1.27)
+				)
+			)
+		)
+		(pin "1"
+		)
+		(instances
+			(project "CLOCK_CORE"
+				(path "/a25f2a35-4889-4be5-9b80-12803bbbfe96/645fcd89-025a-4233-88ed-d1f363faa68e"
+					(reference "#PWR0139")
+					(unit 1)
+				)
