File: hardware/schematic/v1.0/CLOCK_CORE/OCXO.kicad_sch (KiCad schematic)
At the start: 21 parts, among them U1 OCXO_20x20mm, U2 OCXO_25.4x25.4mm, U6 REF5040

Commit message: sch and pcb update
Parts:
- C10, C11, C13, C9: footprint Capacitor_SMD:C_0402_1005Metric -> CLOCK_CORE:C_0402_1005Metric; symbol Device:C -> CLOCK_CORE:C
- C12, C56, C57, C58: footprint Capacitor_SMD:C_0603_1608Metric -> CLOCK_CORE:C_0603_1608Metric; symbol Device:C -> CLOCK_CORE:C
- R13, R14, R30: footprint Resistor_SMD:R_0402_1005Metric -> CLOCK_CORE:R_0402_1005Metric; symbol Device:R -> CLOCK_CORE:R
- R15: footprint Counter:3296W-1-103_C48997937 -> CLOCK_CORE:3296W-1-103_C48997937; symbol Counter:3296W-1-103_C48997937 -> CLOCK_CORE:3296W-1-103_C48997937
- R28, R29: footprint Resistor_SMD:R_0603_1608Metric -> CLOCK_CORE:R_0603_1608Metric; symbol Device:R -> CLOCK_CORE:R
- R39: footprint Resistor_SMD:R_0805_2012Metric -> CLOCK_CORE:R_0805_2012Metric; symbol Device:R -> CLOCK_CORE:R
- RF10: footprint JLCImport:KH-IPEX-K501-29 -> CLOCK_CORE:KH-IPEX-K501-29; symbol JLCImport:KH-IPEX-K501-29 -> CLOCK_CORE:KH-IPEX-K501-29
- TP1, TP2: footprint TestPoint:TestPoint_Pad_D1.0mm -> CLOCK_CORE:TestPoint_Pad_D1.0mm; symbol Connector:TestPoint -> CLOCK_CORE:TestPoint
- U1: footprint JLCImport:OCXO_20x20mm -> CLOCK_CORE:OCXO_20x20mm; symbol Counter:OCXO_20x20mm -> CLOCK_CORE:OCXO_20x20mm
- U2: footprint JLCImport:DOPFITKR2-10M -> CLOCK_CORE:DOPFITKR2-10M; symbol Counter:OCXO_25.4x25.4mm -> CLOCK_CORE:OCXO_25.4x25.4mm
- U6: footprint JLCImport:REF5040 -> CLOCK_CORE:REF5040; symbol JLCImport:REF5040 -> CLOCK_CORE:REF5040
Changed lines of the file:
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@@
 	)
 	(symbol
-		(lib_id "power:GND")
+		(lib_id "CLOCK_CORE:GND")
 		(at 119.38 60.96 0)
 		(unit 1)
@@
 	)
 	(symbol
-		(lib_id "power:GND")
+		(lib_id "CLOCK_CORE:GND")
 		(at 101.6 138.43 270)
 		(unit 1)
@@
 	)
 	(symbol
-		(lib_id "power:GND")
+		(lib_id "CLOCK_CORE:GND")
 		(at 219.71 69.85 0)
 		(unit 1)
@@
 	)
 	(symbol
-		(lib_id "Counter:OCXO_25.4x25.4mm")
+		(lib_id "CLOCK_CORE:OCXO_25.4x25.4mm")
 		(at 129.54 129.54 0)
 		(unit 1)
@@
 			)
 		)
-		(property "Footprint" "JLCImport:DOPFITKR2-10M"
+		(property "Footprint" "CLOCK_CORE:DOPFITKR2-10M"
 			(at 129.032 113.284 0)
 			(hide yes)
@@
 	)
 	(symbol
-		(lib_id "Device:C")
+		(lib_id "CLOCK_CORE:C")
 		(at 106.68 138.43 270)
 		(unit 1)
@@
 			)
 		)
-		(property "Footprint" "Capacitor_SMD:C_0402_1005Metric"
+		(property "Footprint" "CLOCK_CORE:C_0402_1005Metric"
 			(at 102.87 139.3952 0)
 			(hide yes)
@@
 	)
 	(symbol
-		(lib_id "Device:C")
+		(lib_id "CLOCK_CORE:C")
 		(at 160.02 120.65 0)
 		(unit 1)
@@
 			)
 		)
-		(property "Footprint" "Capacitor_SMD:C_0603_1608Metric"
+		(property "Footprint" "CLOCK_CORE:C_0603_1608Metric"
 			(at 160.9852 124.46 0)
 			(hide yes)
@@
 	)
 	(symbol
-		(lib_id "power:GND")
+		(lib_id "CLOCK_CORE:GND")
 		(at 69.85 101.6 180)
 		(unit 1)
@@
 	)
 	(symbol
-		(lib_id "power:GND")
+		(lib_id "CLOCK_CORE:GND")
 		(at 57.15 114.3 270)
 		(unit 1)
@@
 	)
 	(symbol
-		(lib_id "power:GND")
+		(lib_id "CLOCK_CORE:GND")
 		(at 156.21 115.57 180)
 		(unit 1)
@@
 	)
 	(symbol
-		(lib_id "JLCImport:REF5040")
+		(lib_id "CLOCK_CORE:REF5040")
 		(at 242.57 57.15 0)
 		(unit 1)
@@
 			)
 		)
-		(property "Footprint" "JLCImport:REF5040"
+		(property "Footprint" "CLOCK_CORE:REF5040"
 			(at 242.57 57.15 0)
 			(hide yes)
@@
 	)
 	(symbol
-		(lib_id "power:+5V")
+		(lib_id "CLOCK_CORE:+5V")
 		(at 215.9 45.72 0)
 		(unit 1)
@@
 	)
 	(symbol
-		(lib_id "power:PWR_FLAG")
+		(lib_id "CLOCK_CORE:PWR_FLAG")
 		(at 137.16 148.59 90)
 		(unit 1)
@@
 	)
 	(symbol
-		(lib_id "Device:C")
+		(lib_id "CLOCK_CORE:C")
 		(at 152.4 120.65 180)
 		(unit 1)
@@
 			)
 		)
-		(property "Footprint" "Capacitor_SMD:C_0402_1005Metric"
+		(property "Footprint" "CLOCK_CORE:C_0402_1005Metric"
 			(at 151.4348 116.84 0)
 			(hide yes)
@@
 	)
 	(symbol
-		(lib_id "Device:R")
+		(lib_id "CLOCK_CORE:R")
 		(at 114.3 60.96 180)
 		(unit 1)
@@
 			)
 		)
-		(property "Footprint" "Resistor_SMD:R_0402_1005Metric"
+		(property "Footprint" "CLOCK_CORE:R_0402_1005Metric"
 			(at 116.078 60.96 90)
 			(hide yes)
@@
 	)
 	(symbol
-		(lib_id "Device:R")
+		(lib_id "CLOCK_CORE:R")
 		(at 215.9 50.8 180)
 		(unit 1)
@@
 			)
 		)
-		(property "Footprint" "Resistor_SMD:R_0603_1608Metric"
+		(property "Footprint" "CLOCK_CORE:R_0603_1608Metric"
 			(at 217.678 50.8 90)
 			(hide yes)
@@
 	)
 	(symbol
-		(lib_id "Device:C")
+		(lib_id "CLOCK_CORE:C")
 		(at 215.9 62.23 0)
 		(unit 1)
@@
 			)
 		)
-		(property "Footprint" "Capacitor_SMD:C_0603_1608Metric"
+		(property "Footprint" "CLOCK_CORE:C_0603_1608Metric"
 			(at 216.8652 66.04 0)
 			(hide yes)
@@
 	)
 	(symbol
-		(lib_id "power:GND")
+		(lib_id "CLOCK_CORE:GND")
 		(at 116.84 129.54 270)
 		(unit 1)
@@
 	)
 	(symbol
-		(lib_id "Device:C")
+		(lib_id "CLOCK_CORE:C")
 		(at 264.16 63.5 0)
 		(unit 1)
@@
 			)
 		)
-		(property "Footprint" "Capacitor_SMD:C_0603_1608Metric"
+		(property "Footprint" "CLOCK_CORE:C_0603_1608Metric"
 			(at 265.1252 67.31 0)
 			(hide yes)
@@
 	)
 	(symbol
-		(lib_id "power:GND")
+		(lib_id "CLOCK_CORE:GND")
 		(at 182.88 135.89 0)
 		(unit 1)
@@
 	)
 	(symbol
-		(lib_id "Device:R")
+		(lib_id "CLOCK_CORE:R")
 		(at 111.76 53.34 270)
 		(unit 1)
@@
 			)
 		)
-		(property "Footprint" "Resistor_SMD:R_0805_2012Metric"
+		(property "Footprint" "CLOCK_CORE:R_0805_2012Metric"
 			(at 111.76 51.562 90)
 			(hide yes)
@@
 	)
 	(symbol
-		(lib_id "Counter:OCXO_20x20mm")
+		(lib_id "CLOCK_CORE:OCXO_20x20mm")
 		(at 128.27 46.99 0)
 		(unit 1)
@@
 			)
 		)
-		(property "Footprint" "JLCImport:OCXO_20x20mm"
+		(property "Footprint" "CLOCK_CORE:OCXO_20x20mm"
 			(at 128.27 46.99 0)
 			(hide yes)
@@
 	)
 	(symbol
-		(lib_id "Device:R")
+		(lib_id "CLOCK_CORE:R")
 		(at 96.52 119.38 180)
 		(unit 1)
@@
 			)
 		)
-		(property "Footprint" "Resistor_SMD:R_0402_1005Metric"
+		(property "Footprint" "CLOCK_CORE:R_0402_1005Metric"
 			(at 98.298 119.38 90)
 			(hide yes)
@@
 	)
 	(symbol
-		(lib_id "Device:R")
+		(lib_id "CLOCK_CORE:R")
 		(at 118.11 143.51 180)
 		(unit 1)
@@
 			)
 		)
-		(property "Footprint" "Resistor_SMD:R_0402_1005Metric"
+		(property "Footprint" "CLOCK_CORE:R_0402_1005Metric"
 			(at 119.888 143.51 90)
 			(hide yes)
@@
 	)
 	(symbol
-		(lib_id "Device:C")
+		(lib_id "CLOCK_CORE:C")
 		(at 255.27 66.04 0)
 		(unit 1)
@@
 			)
 		)
-		(property "Footprint" "Capacitor_SMD:C_0603_1608Metric"
+		(property "Footprint" "CLOCK_CORE:C_0603_1608Metric"
 			(at 256.2352 69.85 0)
 			(hide yes)
@@
 	)
 	(symbol
-		(lib_id "power:GND")
+		(lib_id "CLOCK_CORE:GND")
 		(at 69.85 127 0)
 		(unit 1)
@@
 	)
 	(symbol
-		(lib_id "Device:C")
+		(lib_id "CLOCK_CORE:C")
 		(at 96.52 110.49 0)
 		(unit 1)
@@
 			)
 		)
-		(property "Footprint" "Capacitor_SMD:C_0402_1005Metric"
+		(property "Footprint" "CLOCK_CORE:C_0402_1005Metric"
 			(at 97.4852 114.3 0)
 			(hide yes)
@@
 	)
 	(symbol
-		(lib_id "Counter:3296W-1-103_C48997937")
+		(lib_id "CLOCK_CORE:3296W-1-103_C48997937")
 		(at 118.11 153.67 0)
 		(mirror y)
@@
 			)
 		)
-		(property "Footprint" "Counter:3296W-1-103_C48997937"
+		(property "Footprint" "CLOCK_CORE:3296W-1-103_C48997937"
 			(at 118.11 153.67 0)
 			(hide yes)
@@
 	)
 	(symbol
-		(lib_id "power:GND")
+		(lib_id "CLOCK_CORE:GND")
 		(at 113.03 153.67 270)
 		(unit 1)
@@
 	)
 	(symbol
-		(lib_id "power:GND")
+		(lib_id "CLOCK_CORE:GND")
 		(at 255.27 71.12 0)
 		(unit 1)
@@
 	)
 	(symbol
-		(lib_id "Device:R")
+		(lib_id "CLOCK_CORE:R")
 		(at 264.16 53.34 180)
 		(unit 1)
@@
 			)
 		)
-		(property "Footprint" "Resistor_SMD:R_0603_1608Metric"
+		(property "Footprint" "CLOCK_CORE:R_0603_1608Metric"
 			(at 265.938 53.34 90)
 			(hide yes)
@@
 	)
 	(symbol
-		(lib_id "Connector:TestPoint")
+		(lib_id "CLOCK_CORE:TestPoint")
 		(at 147.32 113.03 0)
 		(unit 1)
@@
 			)
 		)
-		(property "Footprint" "TestPoint:TestPoint_Pad_D1.0mm"
+		(property "Footprint" "CLOCK_CORE:TestPoint_Pad_D1.0mm"
 			(at 152.4 113.03 0)
 			(hide yes)
@@
 	)
 	(symbol
-		(lib_id "Device:C")
+		(lib_id "CLOCK_CORE:C")
 		(at 223.52 62.23 180)
 		(unit 1)
@@
 			)
 		)
-		(property "Footprint" "Capacitor_SMD:C_0402_1005Metric"
+		(property "Footprint" "CLOCK_CORE:C_0402_1005Metric"
 			(at 222.5548 58.42 0)
 			(hide yes)
@@
 	)
 	(symbol
-		(lib_id "Connector:TestPoint")
+		(lib_id "CLOCK_CORE:TestPoint")
 		(at 182.88 134.62 0)
 		(unit 1)
@@
 			)
 		)
-		(property "Footprint" "TestPoint:TestPoint_Pad_D1.0mm"
+		(property "Footprint" "CLOCK_CORE:TestPoint_Pad_D1.0mm"
 			(at 187.96 134.62 0)
 			(hide yes)
@@
 	)
 	(symbol
-		(lib_id "JLCImport:KH-IPEX-K501-29")
+		(lib_id "CLOCK_CORE:KH-IPEX-K501-29")
 		(at 69.85 114.3 270)
 		(unit 1)
@@
 			)
 		)
-		(property "Footprint" "JLCImport:KH-IPEX-K501-29"
+		(property "Footprint" "CLOCK_CORE:KH-IPEX-K501-29"
 			(at 69.85 114.3 0)
 			(hide yes)

Commit message: sch and pcb update
Parts:
- added R40, R41: 0, CLOCK_CORE:R_0402_1005Metric, symbol CLOCK_CORE:R
Connections:
- net GND: now also R41.2
- net OCXO_OUT: now also R40.2, R41.1; no longer R13.1, R30.1, U2.1 (RF)
- new net OCXO_FR: R13.1, R30.1, R40.1, U2.1 (RF)
Other:
- moved on the sheet: RF10
