File: hardware/schematic/v1.0/CLOCK_CORE/POWER.kicad_sch (KiCad schematic)
At the start: 0 parts

Commit message: sch update
Parts:
- added C73, C80: 10uF, Capacitor_SMD:C_0603_1608Metric, symbol Device:C
- added C74, C76, C82, C85: 100nF, Capacitor_SMD:C_0402_1005Metric, symbol Device:C
- added C75, C77, C81, C84: 22uF, Capacitor_SMD:C_0805_2012Metric, symbol Device:C
- added C78, C83: 10nF, Capacitor_SMD:C_0402_1005Metric, symbol Device:C
- added C79: 100uF, Capacitor_Tantalum_SMD:CP_EIA-3528-21_Kemet-B, symbol Device:C
- added CN1: LAIL-PHC2_54-2P-01-XH-L, JLCImport:LAIL-PHC2_54-2P-01-XH-L, symbol JLCImport:LAIL-PHC2_54-2P-01-XH-L
- added FB20: 220R@100MHz, Inductor_SMD:L_0603_1608Metric, symbol Device:FerriteBead_Small
- added R54, R60: 12.1K, Resistor_SMD:R_0402_1005Metric, symbol Device:R
- added R55, R61: 3.87K, Resistor_SMD:R_0402_1005Metric, symbol Device:R
- added R56, R59: 100K, Resistor_SMD:R_0402_1005Metric, symbol Device:R
- added R57, R58: 0, Resistor_SMD:R_0402_1005Metric, symbol Device:R
- added U2, U3: TPS7A5201RPSR, JLCImport:TPS7A5201RPSR, symbol JLCImport:TPS7A5201RPSR
Connections:
- new net: C83.2, R60.2, R61.1, U2.9 (FB)
- new net: C78.2, R54.2, R55.1, U3.9 (FB)
- new net: C76.1, U3.4 (NR/SS)
- new net: C82.1, U2.4 (NR/SS)
- new net +3.3V: C83.1, C84.1, R59.2, R60.1, U2.10 (OUT), U2.11 (OUT)
- new net +5V: C73.1, C74.1, C75.1, C81.1, CN1.1, FB20.1, U2.1 (IN), U2.2 (IN), U2.3 (EN), U3.1 (IN), U3.2 (IN), U3.3 (EN)
- new net 3.3V_OCXO: C77.1, C78.1, R54.1, R56.2, R58.2, U3.10 (OUT), U3.11 (OUT)
- new net GND: C73.2, C74.2, C75.2, C76.2, C77.2, C79.2, C80.2, C81.2, C82.2, C84.2, C85.2, CN1.2, R55.2, R61.2, U2.12 (GND), U2.5 (BIAS), U2.6 (GND), U2.7 (GND), U3.12 (GND), U3.5 (BIAS), U3.6 (GND), U3.7 (GND)
- new net OCXO_5V: C79.1, C80.1, C85.1, FB20.2, R57.1
- new net OCXO_PG: R56.1, U3.8 (PG)
- new net OCXO_VCC: R57.2, R58.1
- new net PLL_PG: R59.1, U2.8 (PG)
Other:
- note added: "OCXO 供电选配 (二者互斥, 严禁同装):"
- note added: "U2 TPS7A52 5V -> 3.3V 给LMK5B12204供电"
- note added: "U3 TPS7A52 5V -> 3.3V 仅 3.3V OCXO 时装配"
- note added: "装 R57 = 5V OCXO 直供 / 装 R58 = 3.3V OCXO 经 U3 稳压"

Commit message: sch update
Parts:
- removed C79: 100uF, Capacitor_Tantalum_SMD:CP_EIA-3528-21_Kemet-B, symbol Device:C
- removed FB20: 220R@100MHz, Inductor_SMD:L_0603_1608Metric, symbol Device:FerriteBead_Small
- added C9: TAJB107M010RNJ, JLCImport:TAJB107M010RNJ, symbol JLCImport:TAJB107M010RNJ
- R57: footprint Resistor_SMD:R_0402_1005Metric -> Resistor_SMD:R_0805_2012Metric
- R58: value 0 -> DNP; footprint Resistor_SMD:R_0402_1005Metric -> Resistor_SMD:R_0805_2012Metric
Connections:
- net OCXO_5V is gone; now on net +5V: C80.1, C85.1, R57.1
- net GND: now also C9.2
- net OCXO_VCC: now also C9.1
- net OCXO_PG: no longer names the net of R56.1, U3.8 (PG)

Commit message: sch update
Parts:
- added F1: BSMD1206C-1300T, JLCImport:BSMD1206C-1300T, symbol JLCImport:BSMD1206C-1300T
Connections:
- net +5V: now also F1.2; no longer CN1.1
- new net: CN1.1, F1.1
Other:
- moved on the sheet: CN1
