File: hardware/schematic/v1.0/CLOCK_CORE/POWER.kicad_sch (KiCad schematic)
At the start: 25 parts, among them CN1 LAIL-PHC2_54-2P-01-XH-L, U3 TPS7A5201RPSR, U4 TPS7A5201RPSR

Commit message: sch and pcb update
Connections:
- net LDO_3V3_FB: now reaches C20.2, R16.2, R17.1, U3.9 (FB)
- net +5V_IN: now reaches CN1.1, F1.1
- net LDO_OCXO_FB: now reaches C25.2, R21.2, R22.1, U4.9 (FB)
- net LDO_OCXO_NR: now reaches C26.1, U4.4 (NR/SS)
- net LDO_3V3_NR: now reaches C21.1, U3.4 (NR/SS)
- net LDO_OCXO_PG: now reaches R23.1, U4.8 (PG)
- net PLL_PG renamed PDN
Changed lines of the file:
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@@
 		)
 	)
-	(hierarchical_label "PLL_PG"
+	(label "LDO_3V3_NR"
+		(at 104.14 60.96 0)
+		(effects
+			(font
+				(size 1.27 1.27)
+			)
+			(justify left bottom)
+		)
+	)
+	(label "+5V_IN"
+		(at 34.29 52.07 0)
+		(effects
+			(font
+				(size 1.27 1.27)
+			)
+			(justify left bottom)
+		)
+	)
+	(label "LDO_OCXO_NR"
+		(at 101.6 134.62 0)
+		(effects
+			(font
+				(size 1.27 1.27)
+			)
+			(justify left bottom)
+		)
+	)
+	(label "LDO_OCXO_PG"
+		(at 138.43 154.94 0)
+		(effects
+			(font
+				(size 1.27 1.27)
+			)
+			(justify left bottom)
+		)
+	)
+	(label "LDO_3V3_FB"
+		(at 144.78 66.04 0)
+		(effects
+			(font
+				(size 1.27 1.27)
+			)
+			(justify left bottom)
+		)
+	)
+	(label "LDO_OCXO_FB"
+		(at 142.24 139.7 0)
+		(effects
+			(font
+				(size 1.27 1.27)
+			)
+			(justify left bottom)
+		)
+	)
+	(hierarchical_label "PDN"
 		(shape output)
 		(at 134.62 81.28 180)

Commit message: sch and pcb update
Parts:
- added D3, D4, D5: LED, LED_SMD:LED_0603_1608Metric, symbol Device:LED
Connections:
- net +5V: now also D3.2 (A)
- net 3.3V_OCXO: now also D5.2 (A)
- net GND: now also D3.1 (K), D4.1 (K), D5.1 (K)
- net OCXO_VCC: now also D4.2 (A)
Other:
- moved on the sheet: F1

Commit message: sch and pcb update
Parts:
- R20: now not fitted
Changed lines of the file:
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@@
 		(on_board yes)
 		(in_pos_files yes)
-		(dnp no)
+		(dnp yes)
 		(property "Reference" "R20"
 			(at 249.936 83.566 90)

Commit message: sch and pcb update
Connections:
- net +3.3V: now also D5.2 (A)
- net 3.3V_OCXO: no longer D5.2 (A)
Changed lines of the file:
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@@
 	(wire
 		(pts
+			(xy 181.61 55.88) (xy 181.61 57.15)
+		)
+		(stroke
+			(width 0)
+			(type default)
+		)
+	)
+	(wire
+		(pts
 			(xy 106.68 55.88) (xy 106.68 58.42)
 		)
@@
 	(wire
 		(pts
-			(xy 181.61 129.54) (xy 166.37 129.54)
-		)
-		(stroke
-			(width 0)
-			(type default)
-		)
-	)
-	(wire
-		(pts
-			(xy 181.61 132.08) (xy 181.61 129.54)
-		)
-		(stroke
-			(width 0)
-			(type default)
-		)
-	)
-	(wire
-		(pts
 			(xy 129.54 134.62) (xy 137.16 134.62)
 		)
@@
 	(wire
 		(pts
-			(xy 181.61 139.7) (xy 181.61 142.24)
+			(xy 181.61 64.77) (xy 181.61 67.31)
 		)
 		(stroke
@@
 	(wire
 		(pts
+			(xy 168.91 55.88) (xy 181.61 55.88)
+		)
+		(stroke
+			(width 0)
+			(type default)
+		)
+	)
+	(wire
+		(pts
 			(xy 160.02 55.88) (xy 168.91 55.88)
 		)
@@
 	)
 	(symbol
-		(lib_id "Device:LED")
-		(at 181.61 135.89 90)
+		(lib_id "Device:C")
+		(at 157.48 134.62 0)
 		(unit 1)
 		(body_style 1)
@@
 		(in_pos_files yes)
 		(dnp no)
-		(property "Reference" "D5"
-			(at 184.658 135.636 0)
-			(show_name no)
-			(do_not_autoplace no)
-			(effects
-				(font
-					(size 1.27 1.27)
-				)
-			)
-		)
-		(property "Value" "LED"
-			(at 178.054 135.89 0)
+		(property "Reference" "C25"
+			(at 158.242 132.334 0)
 			(show_name no)
 			(do_not_autoplace no)
@@
 					(size 1.27 1.27)
 				)
+				(justify left)
 			)
 		)
-		(property "Footprint" "LED_SMD:LED_0603_1608Metric"
-			(at 181.61 135.89 0)
-			(hide yes)
+		(property "Value" "10nF"
+			(at 158.75 136.906 0)
 			(show_name no)
 			(do_not_autoplace no)
@@
 					(size 1.27 1.27)
 				)
+				(justify left)
 			)
 		)
-		(property "Datasheet" ""
-			(at 181.61 135.89 0)
+		(property "Footprint" "Capacitor_SMD:C_0402_1005Metric"
+			(at 157.48 134.62 0)
 			(hide yes)
 			(show_name no)
@@
 			)
 		)
-		(property "Description" "Light emitting diode"
-			(at 181.61 135.89 0)
+		(property "Datasheet" "~"
+			(at 157.48 134.62 0)
 			(hide yes)
 			(show_name no)
@@
 			)
 		)
-		(property "Sim.Pins" "1=K 2=A"
-			(at 181.61 135.89 0)
+		(property "Description" ""
+			(at 157.48 134.62 0)
 			(hide yes)
 			(show_name no)
@@
 			(project "CLOCK_CORE"
 				(path "/a25f2a35-4889-4be5-9b80-12803bbbfe96/6e31b722-7b29-4340-8cba-f8ca04169b2e"
-					(reference "D5")
+					(reference "C25")
 					(unit 1)
 				)
@@
 	)
 	(symbol
-		(lib_id "Device:C")
-		(at 157.48 134.62 0)
+		(lib_id "power:GND")
+		(at 231.14 63.5 0)
 		(unit 1)
 		(body_style 1)
@@
 		(in_pos_files yes)
 		(dnp no)
-		(property "Reference" "C25"
-			(at 158.242 132.334 0)
+		(fields_autoplaced yes)
+		(property "Reference" "#PWR018"
+			(at 231.14 67.31 0)
+			(hide yes)
 			(show_name no)
 			(do_not_autoplace no)
@@
 					(size 1.27 1.27)
 				)
-				(justify left)
 			)
 		)
-		(property "Value" "10nF"
-			(at 158.75 136.906 0)
+		(property "Value" "GND"
+			(at 231.14 68.58 0)
+			(hide yes)
 			(show_name no)
 			(do_not_autoplace no)
@@
 					(size 1.27 1.27)
 				)
-				(justify left)
 			)
 		)
-		(property "Footprint" "Capacitor_SMD:C_0402_1005Metric"
-			(at 157.48 134.62 0)
+		(property "Footprint" ""
+			(at 231.14 63.5 0)
 			(hide yes)
 			(show_name no)
@@
 			)
 		)
-		(property "Datasheet" "~"
-			(at 157.48 134.62 0)
+		(property "Datasheet" ""
+			(at 231.14 63.5 0)
 			(hide yes)
 			(show_name no)
@@
 		)
 		(property "Description" ""
-			(at 157.48 134.62 0)
+			(at 231.14 63.5 0)
 			(hide yes)
 			(show_name no)
@@
 		(pin "1"
 		)
-		(pin "2"
-		)
 		(instances
 			(project "CLOCK_CORE"
 				(path "/a25f2a35-4889-4be5-9b80-12803bbbfe96/6e31b722-7b29-4340-8cba-f8ca04169b2e"
-					(reference "C25")
+					(reference "#PWR018")
 					(unit 1)
 				)
@@
 	)
 	(symbol
-		(lib_id "power:GND")
-		(at 231.14 63.5 0)
+		(lib_id "power:+5V")
+		(at 63.5 52.07 0)
 		(unit 1)
 		(body_style 1)
@@
 		(dnp no)
 		(fields_autoplaced yes)
-		(property "Reference" "#PWR018"
-			(at 231.14 67.31 0)
+		(property "Reference" "#PWR08"
+			(at 63.5 55.88 0)
 			(hide yes)
 			(show_name no)
@@
 			)
 		)
-		(property "Value" "GND"
-			(at 231.14 68.58 0)
-			(hide yes)
+		(property "Value" "+5V"
+			(at 63.5 46.99 0)
 			(show_name no)
 			(do_not_autoplace no)
@@
 		)
 		(property "Footprint" ""
-			(at 231.14 63.5 0)
+			(at 63.5 52.07 0)
 			(hide yes)
 			(show_name no)
@@
 		)
 		(property "Datasheet" ""
-			(at 231.14 63.5 0)
+			(at 63.5 52.07 0)
 			(hide yes)
 			(show_name no)
@@
 		)
 		(property "Description" ""
-			(at 231.14 63.5 0)
+			(at 63.5 52.07 0)
 			(hide yes)
 			(show_name no)
@@
 			(project "CLOCK_CORE"
 				(path "/a25f2a35-4889-4be5-9b80-12803bbbfe96/6e31b722-7b29-4340-8cba-f8ca04169b2e"
-					(reference "#PWR018")
+					(reference "#PWR08")
 					(unit 1)
 				)
@@
 	)
 	(symbol
-		(lib_id "power:+5V")
-		(at 63.5 52.07 0)
+		(lib_id "power:+3.3V")
+		(at 45.72 97.79 0)
 		(unit 1)
 		(body_style 1)
@@
 		(dnp no)
 		(fields_autoplaced yes)
-		(property "Reference" "#PWR08"
-			(at 63.5 55.88 0)
+		(property "Reference" "#PWR040"
+			(at 45.72 101.6 0)
 			(hide yes)
 			(show_name no)
@@
 			)
 		)
-		(property "Value" "+5V"
-			(at 63.5 46.99 0)
+		(property "Value" "+3.3V"
+			(at 45.72 92.71 0)
 			(show_name no)
 			(do_not_autoplace no)
@@
 		)
 		(property "Footprint" ""
-			(at 63.5 52.07 0)
+			(at 45.72 97.79 0)
 			(hide yes)
 			(show_name no)
@@
 		)
 		(property "Datasheet" ""
-			(at 63.5 52.07 0)
+			(at 45.72 97.79 0)
 			(hide yes)
 			(show_name no)
@@
 			)
 		)
-		(property "Description" ""
-			(at 63.5 52.07 0)
+		(property "Description" "Power symbol creates a global label with name \"+3.3V\""
+			(at 45.72 97.79 0)
 			(hide yes)
 			(show_name no)
@@
 			(project "CLOCK_CORE"
 				(path "/a25f2a35-4889-4be5-9b80-12803bbbfe96/6e31b722-7b29-4340-8cba-f8ca04169b2e"
-					(reference "#PWR08")
+					(reference "#PWR040")
 					(unit 1)
 				)
@@
 	)
 	(symbol
-		(lib_id "power:+3.3V")
-		(at 45.72 97.79 0)
+		(lib_id "Device:LED")
+		(at 181.61 60.96 90)
 		(unit 1)
 		(body_style 1)
@@
 		(in_pos_files yes)
 		(dnp no)
-		(fields_autoplaced yes)
-		(property "Reference" "#PWR040"
-			(at 45.72 101.6 0)
-			(hide yes)
+		(property "Reference" "D5"
+			(at 184.912 61.214 90)
 			(show_name no)
 			(do_not_autoplace no)
@@
 			)
 		)
-		(property "Value" "+3.3V"
-			(at 45.72 92.71 0)
+		(property "Value" "LED"
+			(at 184.404 57.404 90)
 			(show_name no)
 			(do_not_autoplace no)
@@
 			)
 		)
-		(property "Footprint" ""
-			(at 45.72 97.79 0)
+		(property "Footprint" "LED_SMD:LED_0603_1608Metric"
+			(at 181.61 60.96 0)
 			(hide yes)
 			(show_name no)
@@
 		)
 		(property "Datasheet" ""
-			(at 45.72 97.79 0)
+			(at 181.61 60.96 0)
 			(hide yes)
 			(show_name no)
@@
 			)
 		)
-		(property "Description" "Power symbol creates a global label with name \"+3.3V\""
-			(at 45.72 97.79 0)
+		(property "Description" "Light emitting diode"
+			(at 181.61 60.96 0)
+			(hide yes)
+			(show_name no)
+			(do_not_autoplace no)
+			(effects
+				(font
+					(size 1.27 1.27)
+				)
+			)
+		)
+		(property "Sim.Pins" "1=K 2=A"
+			(at 181.61 60.96 0)
 			(hide yes)
 			(show_name no)
@@
 		(pin "1"
 		)
+		(pin "2"
+		)
 		(instances
 			(project "CLOCK_CORE"
 				(path "/a25f2a35-4889-4be5-9b80-12803bbbfe96/6e31b722-7b29-4340-8cba-f8ca04169b2e"
-					(reference "#PWR040")
+					(reference "D5")
 					(unit 1)
 				)
@@
 	(symbol
 		(lib_id "power:GND")
-		(at 181.61 142.24 0)
+		(at 181.61 67.31 0)
 		(unit 1)
 		(body_style 1)
@@
 		(fields_autoplaced yes)
 		(property "Reference" "#PWR0133"
-			(at 181.61 146.05 0)
+			(at 181.61 71.12 0)
 			(hide yes)
 			(show_name no)
@@
 		)
 		(property "Value" "GND"
-			(at 181.61 147.32 0)
+			(at 181.61 72.39 0)
 			(hide yes)
 			(show_name no)
@@
 		)
 		(property "Footprint" ""
-			(at 181.61 142.24 0)
+			(at 181.61 67.31 0)
 			(hide yes)
 			(show_name no)
@@
 		)
 		(property "Datasheet" ""
-			(at 181.61 142.24 0)
+			(at 181.61 67.31 0)
 			(hide yes)
 			(show_name no)
@@
 		)
 		(property "Description" ""
-			(at 181.61 142.24 0)
+			(at 181.61 67.31 0)
 			(hide yes)
 			(show_name no)

Commit message: sch and pcb update
Other:
- moved on the sheet: C23, C24, C25, C26, R21, R22, R23, U4

Commit message: pcb update
Parts:
- R20: value DNP -> 0
Changed lines of the file:
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@@
 			)
 		)
-		(property "Value" "DNP"
+		(property "Value" "0"
 			(at 255.016 83.566 90)
 			(show_name no)

Commit message: sch and pcb update
Parts:
- C14, C18: footprint Capacitor_SMD:C_0603_1608Metric -> CLOCK_CORE:C_0603_1608Metric; symbol Device:C -> CLOCK_CORE:C
- C15, C19, C20, C21, C25, C26: footprint Capacitor_SMD:C_0402_1005Metric -> CLOCK_CORE:C_0402_1005Metric; symbol Device:C -> CLOCK_CORE:C
- C16, C17, C23, C24: footprint Capacitor_SMD:C_0805_2012Metric -> CLOCK_CORE:C_0805_2012Metric; symbol Device:C -> CLOCK_CORE:C
- C22: footprint JLCImport:TAJB107M010RNJ -> CLOCK_CORE:TAJB107M010RNJ; symbol JLCImport:TAJB107M010RNJ -> CLOCK_CORE:TAJB107M010RNJ
- CN1: footprint JLCImport:LAIL-PHC2_54-2P-01-XH-L -> CLOCK_CORE:LAIL-PHC2_54-2P-01-XH-L; symbol JLCImport:LAIL-PHC2_54-2P-01-XH-L -> CLOCK_CORE:LAIL-PHC2_54-2P-01-XH-L
- D3, D4, D5: footprint LED_SMD:LED_0603_1608Metric -> CLOCK_CORE:LED_0603_1608Metric; symbol Device:LED -> CLOCK_CORE:LED
- F1: footprint JLCImport:BSMD1206C-1300T -> CLOCK_CORE:BSMD1206C-1300T; symbol JLCImport:BSMD1206C-1300T -> CLOCK_CORE:BSMD1206C-1300T
- R16, R17, R18, R21, R22, R23: footprint Resistor_SMD:R_0402_1005Metric -> CLOCK_CORE:R_0402_1005Metric; symbol Device:R -> CLOCK_CORE:R
- R19, R20: footprint Resistor_SMD:R_0805_2012Metric -> CLOCK_CORE:R_0805_2012Metric; symbol Device:R -> CLOCK_CORE:R
- U3, U4: footprint JLCImport:TPS7A5201RPSR -> CLOCK_CORE:TPS7A5201RPSR; symbol JLCImport:TPS7A5201RPSR -> CLOCK_CORE:TPS7A5201RPSR

Commit message: Add a current-limiting resistor, sch and pcb update
Parts:
- added R42, R43, R46: 2.2K, CLOCK_CORE:R_0402_1005Metric, symbol CLOCK_CORE:R
Connections:
- net +3.3V: now also R43.1; no longer D5.2 (A)
- net +5V: now also R46.1; no longer D3.2 (A)
- net OCXO_VCC: now also R42.2; no longer D4.2 (A)
- new net: D4.2 (A), R42.1
- new net: D3.2 (A), R46.2
- new net: D5.2 (A), R43.2
