File: hardware/schematic/v1.0/CLOCK_CORE/CLOCK_CORE.kicad_sch (KiCad schematic)
At the start: 0 parts

Commit message: sch update
Other:
- sheet LMK5B12204 ports: added OUT0_N, OUT0_P, OUT1_N, OUT1_P, OUT2_N, OUT2_P, OUT3_N, OUT3_P, PLL_PG, PRIREF_P, XO_P; removed none
- sheet OCXO ports: added OCXO_VCC, XO_P; removed none
- sheet POWER ports: added OCXO_VCC, PLL_PG; removed none
- sheet SIGNAL ports: added OUT0_N, OUT0_P, OUT1_N, OUT1_P, OUT2_N, OUT2_P, OUT3_N, OUT3_P, PRIREF_P; removed none

Commit message: sch update
Other:
- added sheet DEBUG (DEBUG.kicad_sch)
- sheet LMK5B12204 ports: added SCL, SDA; removed none

Commit message: sch and pcb update
Other:
- sheet LMK5B12204 ports: added OCXO_OUT, PDN; removed PLL_PG, XO_P
- sheet OCXO ports: added OCXO_OUT; removed XO_P
- sheet POWER ports: added PDN; removed PLL_PG
Changed lines of the file:
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@@
 			)
 		)
-		(pin "XO_P" output
+		(pin "OCXO_OUT" output
 			(at 166.37 116.84 180)
 			(effects
@@
 			)
 		)
-		(pin "PLL_PG" output
+		(pin "PDN" output
 			(at 123.19 102.87 0)
 			(effects
@@
 			)
 		)
-		(pin "XO_P" input
+		(pin "OCXO_OUT" input
 			(at 156.21 116.84 0)
 			(effects
@@
 			)
 		)
-		(pin "PLL_PG" input
+		(pin "PDN" input
 			(at 134.62 102.87 180)
 			(effects
