File: hardware/schematic/v1.0/CLOCK_CORE/CLOCK_CORE.kicad_pcb (KiCad board)
At the start: 4 copper layers, 70 x 70 mm, 137 parts, among them CN1 LAIL-PHC2_54-2P-01-XH-L, J1 Conn_Coaxial, J3 Conn_01x04_Socket, U1 OCXO_20x20mm, U2 OCXO_25.4x25.4mm, U3 TPS7A5201RPSR, U4 TPS7A5201RPSR, U5 LMK5B12204, U6 REF5040

Commit message: pcb update
Parts:
- moved TP1 0.43 mm to (135.9, 66.3)
- moved RF9 0.34 mm to (162.7, 125.1)
Routing:
- net OCXO_VCC: track 3.84 -> 9.63 mm
Changed lines of the file:
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@@
 	(footprint "TestPoint:TestPoint_Pad_D1.0mm"
 		(layer "F.Cu")
-		(at 136.32 66.35)
+		(at 135.89 66.33)
 		(descr "SMD pad as test Point, diameter 1.0mm")
 		(tags "test point SMD pad")
@@
 	(footprint "JLCImport:KH-IPEX-K501-29"
 		(layer "F.Cu")
-		(at 162.65 125.40506)
+		(at 162.65 125.06494)
 		(descr "-40℃~+90℃ 1 1.25mm 2mm 3GHz 50Ω Board Side IPEX Male Pin SMD Coaxial Connectors (RF) ROHS")
 		(tags "ANT-SMD_KH-IPEX-K501-29 C411563 KH-IPEX-K501-29 Shenzhen Kinghelm Elec")
@@
 	)
 	(segment
+		(start 135.89 66.33)
+		(end 135.89 69.97008)
+		(width 0.8)
+		(locked yes)
+		(layer "F.Cu")
+		(net "OCXO_VCC")
+	)
+	(segment
 		(start 125.5 73.2)
 		(end 125.5 75.684998)
@@
 		(net "OCXO_VCC")
 	)
+	(segment
+		(start 135.89 69.97008)
+		(end 137.407 71.48708)
+		(width 0.8)
+		(locked yes)
+		(layer "F.Cu")
+		(net "OCXO_VCC")
+	)
 	(via
 		(at 135.79 79.1175)
@@
 		(polygon
 			(pts
-				(xy 163.41 63.04) (xy 170.77 63.04) (xy 170.77 63.92) (xy 163.41 63.92)
+				(xy 163.41 63.04) (xy 169.16 63.04) (xy 169.16 63.92) (xy 163.41 63.92)
 			)
 		)
@@
 			)
 		)
+	)
+	(zone
+		(net "+3.3V")
+		(layer "F.Cu")
+		(hatch edge 0.5)
+		(priority 11)
+		(connect_pads yes
+			(clearance 0.1)
+		)
+		(min_thickness 0.1)
+		(fill yes
+			(thermal_gap 0.5)
+			(thermal_bridge_width 0.5)
+			(island_removal_mode 0)
+		)
+		(polygon
+			(pts
+				(xy 130.99 85.91) (xy 131.45 85.91) (xy 131.45 90.2) (xy 128.25 90.2) (xy 128.25 91.57) (xy 132.67 91.57)
+				(xy 132.67 84.85) (xy 130.99 84.85)
+			)
+		)

Commit message: pcb update
Parts:
- moved TP2 8.29 mm to (162.6, 82.1)
- moved R27 1.05 mm to (168.8, 85.5)
- moved C26 0.64 mm to (123.5, 66.9)
- moved C52 0.25 mm to (145.4, 109.2)
Routing:
- net /DEBUG/SCL: track 0.00 -> 45.0 mm
- net /DEBUG/SDA: track 0.00 -> 42.1 mm
Changed lines of the file:
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@@
 		(capping no)
 		(filling no)
+		(zone_defaults)
 		(aux_axis_origin 111.35 58.6)
 		(grid_origin 111.35 58.6)
@@
 	)
 	(footprint "Resistor_SMD:R_0603_1608Metric"
+		(locked yes)
 		(layer "F.Cu")
 		(at 165.99 85.505 90)
@@
 	(footprint "Capacitor_SMD:C_0402_1005Metric"
 		(layer "F.Cu")
-		(at 145.65 109.19 90)
+		(at 145.4 109.19 90)
 		(descr "Capacitor SMD 0402 (1005 Metric), square (rectangular) end terminal, IPC-7351 nominal, (Body size source: IPC-SM-782 page 76, https://www.pcb-3d.com/wordpress/wp-content/uploads/ipc-sm-782a_amendment_1_and_2.pdf)")
 		(tags "capacitor")
@@
 	)
 	(footprint "Resistor_SMD:R_0603_1608Metric"
+		(locked yes)
 		(layer "F.Cu")
-		(at 167.79 85.53 90)
+		(at 168.84 85.51 90)
 		(descr "Resistor SMD 0603 (1608 Metric), square (rectangular) end terminal, IPC-7351 nominal, (Body size source: IPC-SM-782 page 72, https://www.pcb-3d.com/wordpress/wp-content/uploads/ipc-sm-782a_amendment_1_and_2.pdf)")
 		(tags "resistor")
@@
 	(footprint "Capacitor_SMD:C_0402_1005Metric"
 		(layer "F.Cu")
-		(at 122.85 67.010002 -90)
+		(at 123.49 66.93 -90)
 		(descr "Capacitor SMD 0402 (1005 Metric), square (rectangular) end terminal, IPC-7351 nominal, (Body size source: IPC-SM-782 page 76, https://www.pcb-3d.com/wordpress/wp-content/uploads/ipc-sm-782a_amendment_1_and_2.pdf)")
 		(tags "capacitor")
@@
 	(footprint "TestPoint:TestPoint_Pad_D1.0mm"
 		(layer "F.Cu")
-		(at 162.88 90.39)
+		(at 162.58 82.11)
 		(descr "SMD pad as test Point, diameter 1.0mm")
 		(tags "test point SMD pad")
@@
 	)
 	(segment
+		(start 170.15 81.59)
+		(end 175.859999 75.880001)
+		(width 0.15)
+		(layer "F.Cu")
+		(net "/DEBUG/SDA")
+	)
+	(segment
+		(start 169.535 86.335)
+		(end 170.15 85.72)
+		(width 0.15)
+		(layer "F.Cu")
+		(net "/DEBUG/SDA")
+	)
+	(segment
+		(start 170.15 85.72)
+		(end 170.15 81.59)
+		(width 0.15)
+		(layer "F.Cu")
+		(net "/DEBUG/SDA")
+	)
+	(segment
+		(start 168.84 86.67)
+		(end 168.84 86.335)
+		(width 0.15)
+		(layer "F.Cu")
+		(net "/DEBUG/SDA")
+	)
+	(segment
+		(start 168.84 86.335)
+		(end 169.535 86.335)
+		(width 0.15)
+		(layer "F.Cu")
+		(net "/DEBUG/SDA")
+	)
+	(segment
+		(start 149.15 99.32)
+		(end 153.71 94.76)
+		(width 0.15)
+		(layer "F.Cu")
+		(net "/DEBUG/SDA")
+	)
+	(segment
+		(start 153.71 94.76)
+		(end 160.75 94.76)
+		(width 0.15)
+		(layer "F.Cu")
+		(net "/DEBUG/SDA")
+	)
+	(segment
+		(start 160.75 94.76)
+		(end 168.84 86.67)
+		(width 0.15)
+		(layer "F.Cu")
+		(net "/DEBUG/SDA")
+	)
+	(segment
+		(start 149.15 100.075)
+		(end 149.15 99.32)
+		(width 0.15)
+		(layer "F.Cu")
+		(net "/DEBUG/SDA")
+	)
+	(segment
+		(start 175.859999 75.880001)
+		(end 178.2 75.880001)
+		(width 0.15)
+		(layer "F.Cu")
+		(net "/DEBUG/SDA")
+	)
+	(segment
+		(start 160.36 94.12)
+		(end 165.99 88.49)
+		(width 0.15)
+		(layer "F.Cu")
+		(net "/DEBUG/SCL")
+	)
+	(segment
+		(start 167.22 85.92)
+		(end 167.22 81.64)
+		(width 0.15)
+		(layer "F.Cu")
+		(net "/DEBUG/SCL")
+	)
+	(segment
+		(start 175.52 73.34)
+		(end 178.2 73.34)
+		(width 0.15)
+		(layer "F.Cu")
+		(net "/DEBUG/SCL")
+	)
+	(segment
+		(start 165.99 88.49)
+		(end 165.99 86.33)
+		(width 0.15)
+		(layer "F.Cu")
+		(net "/DEBUG/SCL")
+	)
+	(segment
+		(start 165.99 86.33)
+		(end 166.81 86.33)
+		(width 0.15)
+		(layer "F.Cu")
+		(net "/DEBUG/SCL")
+	)
+	(segment
+		(start 148.65 99.09)
+		(end 153.62 94.12)
+		(width 0.15)
+		(layer "F.Cu")
+		(net "/DEBUG/SCL")
+	)
+	(segment
+		(start 166.81 86.33)
+		(end 167.22 85.92)
+		(width 0.15)
+		(layer "F.Cu")
+		(net "/DEBUG/SCL")
+	)
+	(segment
+		(start 167.22 81.64)
+		(end 175.52 73.34)
+		(width 0.15)
+		(layer "F.Cu")
+		(net "/DEBUG/SCL")
+	)
+	(segment
+		(start 153.62 94.12)
+		(end 160.36 94.12)
+		(width 0.15)
+		(layer "F.Cu")
+		(net "/DEBUG/SCL")
+	)
+	(segment
+		(start 148.65 100.075)
+		(end 148.65 99.09)
+		(width 0.15)
+		(layer "F.Cu")
+		(net "/DEBUG/SCL")
+	)
+	(segment
 		(start 146.15 93.11)
 		(end 146.15 100.075)
@@
 	)
 	(zone
+		(net "+5V")
+		(layer "F.Cu")
+		(hatch edge 0.5)
+		(priority 12)
+		(connect_pads yes
+			(clearance 0.1)
+		)
+		(min_thickness 0.1)
+		(fill yes
+			(thermal_gap 0.5)
+			(thermal_bridge_width 0.5)
+			(island_removal_mode 0)
+		)
+		(polygon
+			(pts
+				(xy 120.72 65.44) (xy 120.72 69.32) (xy 122.79 69.32) (xy 122.79 72.7) (xy 124.22 72.7) (xy 124.22 68.59)
+				(xy 122.15 68.59) (xy 122.15 65.44)
+			)
+		)
+	)
+	(zone
 		(net "OCXO_VCC")
 		(locked yes)
@@
 	(zone
 		(net "+5V")
+		(locked yes)
 		(layer "F.Cu")
 		(name "+5V_2")
@@
 	(zone
 		(net "3.3V_OCXO")
+		(locked yes)
 		(layer "F.Cu")
 		(name "3.3V_OCXO")

Commit message: pcb update
Parts:
- moved C21 0.06 mm to (122.2, 87.2)
Routing:
- net VCTRL: track 9.34 -> 24.4 mm
- net /POWER/LDO_OCXO_FB: track 0.00 -> 5.42 mm
- net /POWER/LDO_3V3_NR: track 0.00 -> 2.11 mm
- net /POWER/LDO_OCXO_PG: track 0.00 -> 1.98 mm
- net Net-(U6-TRIM/NR): track 0.00 -> 1.80 mm
- net /POWER/LDO_OCXO_NR: track 0.00 -> 1.67 mm
Changed lines of the file:
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@@
 	(footprint "Capacitor_SMD:C_0402_1005Metric"
 		(layer "F.Cu")
-		(at 122.122748 87.204687 -90)
+		(at 122.18 87.204687 -90)
 		(descr "Capacitor SMD 0402 (1005 Metric), square (rectangular) end terminal, IPC-7351 nominal, (Body size source: IPC-SM-782 page 76, https://www.pcb-3d.com/wordpress/wp-content/uploads/ipc-sm-782a_amendment_1_and_2.pdf)")
 		(tags "capacitor")
@@
 	)
 	(segment
+		(start 128.428467 65.948467)
+		(end 128.7 66.22)
+		(width 0.2)
+		(locked yes)
+		(layer "F.Cu")
+		(net "/POWER/LDO_OCXO_FB")
+	)
+	(segment
+		(start 127.162126 65.948467)
+		(end 128.428467 65.948467)
+		(width 0.2)
+		(locked yes)
+		(layer "F.Cu")
+		(net "/POWER/LDO_OCXO_FB")
+	)
+	(segment
+		(start 131.15 66.29)
+		(end 131.4 66.54)
+		(width 0.2)
+		(locked yes)
+		(layer "F.Cu")
+		(net "/POWER/LDO_OCXO_FB")
+	)
+	(segment
+		(start 128.7 66.22)
+		(end 130.71 66.22)
+		(width 0.2)
+		(locked yes)
+		(layer "F.Cu")
+		(net "/POWER/LDO_OCXO_FB")
+	)
+	(segment
+		(start 130.78 66.29)
+		(end 131.15 66.29)
+		(width 0.2)
+		(locked yes)
+		(layer "F.Cu")
+		(net "/POWER/LDO_OCXO_FB")
+	)
+	(segment
+		(start 131.4 66.54)
+		(end 131.4 67.480002)
+		(width 0.2)
+		(locked yes)
+		(layer "F.Cu")
+		(net "/POWER/LDO_OCXO_FB")
+	)
+	(segment
+		(start 130.71 66.22)
+		(end 130.78 66.29)
+		(width 0.2)
+		(layer "F.Cu")
+		(net "/POWER/LDO_OCXO_FB")
+	)
+	(segment
 		(start 127.426692 111.654)
 		(end 127.453999 111.654)
@@
 	)
 	(segment
+		(start 157.47 89.50392)
+		(end 156.447 90.52692)
+		(width 0.5)
+		(locked yes)
+		(layer "F.Cu")
+		(net "VCTRL")
+	)
+	(segment
 		(start 157.47 75.9)
 		(end 154.55 72.98)
@@
 	)
 	(segment
+		(start 157.47 75.9)
+		(end 157.47 89.50392)
+		(width 0.5)
+		(locked yes)
+		(layer "F.Cu")
+		(net "VCTRL")
+	)
+	(segment
 		(start 161.15 74.369998)
 		(end 161.15 75.9)
@@
 	)
 	(segment
+		(start 123.491406 66.448594)
+		(end 123.49 66.45)
+		(width 0.15)
+		(layer "F.Cu")
+		(net "/POWER/LDO_OCXO_NR")
+	)
+	(segment
+		(start 125.162126 66.448594)
+		(end 123.491406 66.448594)
+		(width 0.2)
+		(locked yes)
+		(layer "F.Cu")
+		(net "/POWER/LDO_OCXO_NR")
+	)
+	(segment
+		(start 127.868594 66.448594)
+		(end 128.700002 67.280002)
+		(width 0.2)
+		(locked yes)
+		(layer "F.Cu")
+		(net "/POWER/LDO_OCXO_PG")
+	)
+	(segment
+		(start 128.700002 67.280002)
+		(end 128.8 67.280002)
+		(width 0.2)
+		(locked yes)
+		(layer "F.Cu")
+		(net "/POWER/LDO_OCXO_PG")
+	)
+	(segment
+		(start 127.162126 66.448594)
+		(end 127.868594 66.448594)
+		(width 0.2)
+		(locked yes)
+		(layer "F.Cu")
+		(net "/POWER/LDO_OCXO_PG")
+	)
+	(segment
 		(start 174.2 100.5)
 		(end 172.2 100.5)
@@
 	)
 	(segment
+		(start 124.285 86.72)
+		(end 122.184687 86.72)
+		(width 0.2)
+		(layer "F.Cu")
+		(net "/POWER/LDO_3V3_NR")
+	)
+	(segment
+		(start 122.184687 86.72)
+		(end 122.18 86.724687)
+		(width 0.2)
+		(layer "F.Cu")
+		(net "/POWER/LDO_3V3_NR")
+	)
+	(segment
 		(start 130.19 86.559999)
 		(end 130.19 87.65)
@@
 	)
 	(segment
+		(start 164.35 66.55)
+		(end 164.35 64.755)
+		(width 0.3)
+		(locked yes)
+		(layer "F.Cu")
+		(net "Net-(U6-TRIM{slash}NR)")
+	)
+	(segment
 		(start 172.2 108.96)
 		(end 172.2 110.13)
@@
 		(polygon
 			(pts
-				(xy 120.72 65.44) (xy 120.72 69.32) (xy 122.79 69.32) (xy 122.79 72.7) (xy 124.22 72.7) (xy 124.22 68.59)
-				(xy 122.15 68.59) (xy 122.15 65.44)
+				(xy 120.72 65.44) (xy 120.72 69.32) (xy 122.79 69.32) (xy 122.79 72.7) (xy 124.22 72.7) (xy 124.22 68.29)
+				(xy 122.15 68.29) (xy 122.15 65.44)
 			)
 		)

Commit message: add pdf and sch update
Parts:
- moved C49 0.29 mm to (136.9, 98.4)
Routing:
- net /LMK5B12204/PRIREF_P: track 0.00 -> 27.9 mm
- net VDDO2_3: track 0.00 -> 3.01 mm
- net +3.3V: vias 0 -> 8
- added copper zone on In2.Cu, net +3.3V
Changed lines of the file:
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@@
 	)
 	(footprint "Connector_Coaxial:SMA_Amphenol_132134-11_Vertical"
+		(locked yes)
 		(layer "F.Cu")
 		(at 162.64 117.94 -90)
@@
 	(footprint "Capacitor_SMD:C_0402_1005Metric"
 		(layer "F.Cu")
-		(at 136.85 98.6925 90)
+		(at 136.89 98.41 90)
 		(descr "Capacitor SMD 0402 (1005 Metric), square (rectangular) end terminal, IPC-7351 nominal, (Body size source: IPC-SM-782 page 76, https://www.pcb-3d.com/wordpress/wp-content/uploads/ipc-sm-782a_amendment_1_and_2.pdf)")
 		(tags "capacitor")
 		(property "Reference" "C49"
-			(at 1.33 0 180)
+			(at 0.0425 -0.84 270)
 			(layer "F.SilkS")
 			(effects
@@
 	)
 	(footprint "JLCImport:KH-IPEX-K501-29"
+		(locked yes)
 		(layer "F.Cu")
-		(at 162.65 125.06494)
+		(at 162.64 125.08494)
 		(descr "-40℃~+90℃ 1 1.25mm 2mm 3GHz 50Ω Board Side IPEX Male Pin SMD Coaxial Connectors (RF) ROHS")
 		(tags "ANT-SMD_KH-IPEX-K501-29 C411563 KH-IPEX-K501-29 Shenzhen Kinghelm Elec")
@@
 	)
 	(segment
+		(start 146.15 108.9)
+		(end 155.19 117.94)
+		(width 0.15)
+		(layer "F.Cu")
+		(net "/LMK5B12204/PRIREF_P")
+	)
+	(segment
+		(start 162.64 123.66)
+		(end 162.64 117.94)
+		(width 0.15)
+		(locked yes)
+		(layer "F.Cu")
+		(net "/LMK5B12204/PRIREF_P")
+	)
+	(segment
+		(start 146.15 106.95)
+		(end 146.15 108.9)
+		(width 0.15)
+		(layer "F.Cu")
+		(net "/LMK5B12204/PRIREF_P")
+	)
+	(segment
+		(start 155.19 117.94)
+		(end 162.64 117.94)
+		(width 0.15)
+		(layer "F.Cu")
+		(net "/LMK5B12204/PRIREF_P")
+	)
+	(segment
 		(start 126.918061 86.72)
 		(end 127.872748 87.674687)
@@
 	)
 	(segment
+		(start 140.2 99.7625)
+		(end 141.512501 99.7625)
+		(width 0.3)
+		(layer "F.Cu")
+		(net "VDDO2_3")
+	)
+	(segment
+		(start 138.5 99.7625)
+		(end 140.2 99.7625)
+		(width 0.3)
+		(layer "F.Cu")
+		(net "VDDO2_3")
+	)
+	(segment
 		(start 137.75322 102.8535)
 		(end 142.215248 102.8535)
@@
 		(net "/POWER/LDO_OCXO_FB")
 	)
+	(via
+		(at 136.6 96.4)
+		(size 0.6)
+		(drill 0.3)
+		(layers "F.Cu" "B.Cu")
+		(free yes)
+		(net "+3.3V")
+	)
+	(via
+		(at 132.56 91.17)
+		(size 0.6)
+		(drill 0.3)
+		(layers "F.Cu" "B.Cu")
+		(free yes)
+		(net "+3.3V")
+	)
+	(via
+		(at 137.3 96.4)
+		(size 0.6)
+		(drill 0.3)
+		(layers "F.Cu" "B.Cu")
+		(free yes)
+		(net "+3.3V")
+	)
+	(via
+		(at 137.3 97.1)
+		(size 0.6)
+		(drill 0.3)
+		(layers "F.Cu" "B.Cu")
+		(free yes)
+		(net "+3.3V")
+	)
+	(via
+		(at 131.8 90.45)
+		(size 0.6)
+		(drill 0.3)
+		(layers "F.Cu" "B.Cu")
+		(free yes)
+		(net "+3.3V")
+	)
+	(via
+		(at 132.56 90.45)
+		(size 0.6)
+		(drill 0.3)
+		(layers "F.Cu" "B.Cu")
+		(free yes)
+		(net "+3.3V")
+	)
+	(via
+		(at 131.8 91.17)
+		(size 0.6)
+		(drill 0.3)
+		(layers "F.Cu" "B.Cu")
+		(free yes)
+		(net "+3.3V")
+	)
+	(via
+		(at 136.6 97.1)
+		(size 0.6)
+		(drill 0.3)
+		(layers "F.Cu" "B.Cu")
+		(free yes)
+		(net "+3.3V")
+	)
 	(segment
 		(start 127.426692 111.654)
@@
 	(zone
 		(net "+3.3V")
+		(locked yes)
 		(layer "F.Cu")
 		(hatch edge 0.5)
@@
 		(polygon
 			(pts
-				(xy 130.99 85.91) (xy 131.45 85.91) (xy 131.45 90.2) (xy 128.25 90.2) (xy 128.25 91.57) (xy 132.67 91.57)
-				(xy 132.67 84.85) (xy 130.99 84.85)
+				(xy 130.99 85.91) (xy 131.45 85.91) (xy 131.45 90.2) (xy 128.25 90.2) (xy 128.25 91.57) (xy 132.91 91.57)
+				(xy 132.91 84.43) (xy 130.99 84.43)
 			)
 		)
@@
 	)
 	(zone
+		(net "+3.3V")
+		(layer "F.Cu")
+		(hatch edge 0.5)
+		(priority 13)
+		(connect_pads yes
+			(clearance 0.1)
+		)
+		(min_thickness 0.1)
+		(fill yes
+			(thermal_gap 0.5)
+			(thermal_bridge_width 0.5)
+			(island_removal_mode 0)
+		)
+		(polygon
+			(pts
+				(xy 136.2 96.02) (xy 136.2 98.3) (xy 137.67 98.3) (xy 137.67 96.02)
+			)
+		)
+	)
+	(zone
 		(net "GND")
 		(layer "In1.Cu")
@@
 			)
 		)
+	)
+	(zone
+		(net "+3.3V")
+		(locked yes)
+		(layer "In2.Cu")
+		(hatch edge 0.5)
+		(priority 14)
+		(connect_pads thru_hole_only
+			(clearance 0.1)
+		)
+		(min_thickness 0.1)
+		(fill yes
+			(thermal_gap 0.5)
+			(thermal_bridge_width 0.5)
+			(island_removal_mode 0)
+		)
+		(polygon
+			(pts
+				(xy 131.45 90.2) (xy 132.91 90.2) (xy 132.91 94.39) (xy 137.67 94.39) (xy 137.67 97.43) (xy 136.2 97.43)
+				(xy 136.2 95.589103) (xy 131.46 95.6)
+			)
+		)

Commit message: pcb update
Routing:
- net /OCXO/VREF: track 0.00 -> 13.1 mm
- net VDDO2_3: track 3.01 -> 5.27 mm
- net +3.3V: track 0.00 -> 1.72 mm, vias 8 -> 16
Changed lines of the file:
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@@
 		(capping no)
 		(filling no)
-		(zone_defaults)
 		(aux_axis_origin 111.35 58.6)
 		(grid_origin 111.35 58.6)
@@
 	)
 	(footprint "JLCImport:HX_PH254-01-03-Z-L11_5_PCB_PIN_HEADER"
+		(locked yes)
 		(layer "F.Cu")
 		(at 151.05 123.1125)
@@
 	)
 	(segment
+		(start 141.512501 100.432501)
+		(end 141.512501 99.7625)
+		(width 0.2)
+		(layer "F.Cu")
+		(net "VDDO2_3")
+	)
+	(segment
 		(start 138.5 99.7625)
 		(end 140.2 99.7625)
@@
 	)
 	(segment
+		(start 141.8425 100.7625)
+		(end 141.512501 100.432501)
+		(width 0.2)
+		(layer "F.Cu")
+		(net "VDDO2_3")
+	)
+	(segment
+		(start 142.9625 100.7625)
+		(end 141.8425 100.7625)
+		(width 0.2)
+		(layer "F.Cu")
+		(net "VDDO2_3")
+	)
+	(segment
 		(start 137.75322 102.8535)
 		(end 142.215248 102.8535)
@@
 		(net "/POWER/LDO_OCXO_FB")
 	)
+	(segment
+		(start 136.89 97.93)
+		(end 138.242502 97.93)
+		(width 0.3)
+		(layer "F.Cu")
+		(net "+3.3V")
+	)
+	(segment
+		(start 138.242502 97.93)
+		(end 138.5 98.187498)
+		(width 0.3)
+		(layer "F.Cu")
+		(net "+3.3V")
+	)
 	(via
 		(at 136.6 96.4)
@@
 	)
 	(via
+		(at 146.31 122.78)
+		(size 0.6)
+		(drill 0.3)
+		(layers "F.Cu" "B.Cu")
+		(locked yes)
+		(free yes)
+		(net "+3.3V")
+	)
+	(via
+		(at 146.31 123.48)
+		(size 0.6)
+		(drill 0.3)
+		(layers "F.Cu" "B.Cu")
+		(locked yes)
+		(free yes)
+		(net "+3.3V")
+	)
+	(via
 		(at 132.56 91.17)
 		(size 0.6)
@@
 	)
 	(via
+		(at 176 80.62)
+		(size 0.6)
+		(drill 0.3)
+		(layers "F.Cu" "B.Cu")
+		(locked yes)
+		(free yes)
+		(net "+3.3V")
+	)
+	(via
 		(at 137.3 97.1)
 		(size 0.6)
@@
 	)
 	(via
+		(at 145.61 122.78)
+		(size 0.6)
+		(drill 0.3)
+		(layers "F.Cu" "B.Cu")
+		(locked yes)
+		(free yes)
+		(net "+3.3V")
+	)
+	(via
 		(at 131.8 90.45)
 		(size 0.6)
@@
 	)
 	(via
+		(at 175.3 80.62)
+		(size 0.6)
+		(drill 0.3)
+		(layers "F.Cu" "B.Cu")
+		(locked yes)
+		(free yes)
+		(net "+3.3V")
+	)
+	(via
+		(at 176 81.32)
+		(size 0.6)
+		(drill 0.3)
+		(layers "F.Cu" "B.Cu")
+		(locked yes)
+		(free yes)
+		(net "+3.3V")
+	)
+	(via
+		(at 145.61 123.48)
+		(size 0.6)
+		(drill 0.3)
+		(layers "F.Cu" "B.Cu")
+		(locked yes)
+		(free yes)
+		(net "+3.3V")
+	)
+	(via
 		(at 132.56 90.45)
 		(size 0.6)
@@
 		(net "+3.3V")
 	)
+	(via
+		(at 175.3 81.32)
+		(size 0.6)
+		(drill 0.3)
+		(layers "F.Cu" "B.Cu")
+		(locked yes)
+		(free yes)
+		(net "+3.3V")
+	)
 	(segment
 		(start 127.426692 111.654)
@@
 	)
 	(segment
+		(start 168.45 65.15)
+		(end 168.45 74.91)
+		(width 0.5)
+		(locked yes)
+		(layer "F.Cu")
+		(net "/OCXO/VREF")
+	)
+	(segment
+		(start 168.45 74.91)
+		(end 167.47 75.89)
+		(width 0.5)
+		(locked yes)
+		(layer "F.Cu")
+		(net "/OCXO/VREF")
+	)
+	(segment
+		(start 167.47 75.89)
+		(end 165.55 75.89)
+		(width 0.5)
+		(locked yes)
+		(layer "F.Cu")
+		(net "/OCXO/VREF")
+	)
+	(segment
 		(start 164.35 66.55)
 		(end 164.35 64.755)
@@
 	)
 	(zone
+		(net "+3.3V")
+		(locked yes)
+		(layer "F.Cu")
+		(hatch edge 0.5)
+		(priority 15)
+		(connect_pads yes
+			(clearance 0.1)
+		)
+		(min_thickness 0.1)
+		(fill yes
+			(thermal_gap 0.5)
+			(thermal_bridge_width 0.5)
+			(island_removal_mode 0)
+		)
+		(polygon
+			(pts
+				(xy 149.41 122.27) (xy 145.13 122.27) (xy 145.13 123.96) (xy 149.41 123.96)
+			)
+		)
+	)
+	(zone
 		(net "OCXO_VCC")
 		(locked yes)
@@
 	)
 	(zone
+		(net "+3.3V")
+		(locked yes)
+		(layer "F.Cu")
+		(hatch edge 0.5)
+		(priority 15)
+		(connect_pads yes
+			(clearance 0.1)
+		)
+		(min_thickness 0.1)
+		(fill yes
+			(thermal_gap 0.5)
+			(thermal_bridge_width 0.5)
+			(island_removal_mode 0)
+		)
+		(polygon
+			(pts
+				(xy 177.83 80.11) (xy 174.82 80.11) (xy 174.82 81.8) (xy 177.83 81.8)
+			)
+		)
+	)
+	(zone
 		(net "Net-(U1-VCC)")
 		(locked yes)
@@
 		(polygon
 			(pts
-				(xy 131.45 90.2) (xy 132.91 90.2) (xy 132.91 94.39) (xy 137.67 94.39) (xy 137.67 97.43) (xy 136.2 97.43)
+				(xy 131.45 90.2) (xy 132.91 90.2) (xy 132.91 94.39) (xy 137.67 94.39) (xy 137.67 123.97) (xy 136.2 123.97)
 				(xy 136.2 95.589103) (xy 131.46 95.6)
 			)
 		)
+	)
+	(zone
+		(net "+3.3V")
+		(locked yes)
+		(layer "In2.Cu")
+		(hatch edge 0.5)
+		(priority 15)
+		(connect_pads yes
+			(clearance 0.1)
+		)
+		(min_thickness 0.1)
+		(fill yes
+			(thermal_gap 0.5)
+			(thermal_bridge_width 0.5)
+			(island_removal_mode 0)
+		)
+		(polygon
+			(pts
+				(xy 146.73 122.27) (xy 136.2 122.27) (xy 136.2 123.96) (xy 146.73 123.96)
+			)
+		)

Commit message: pcb update
Parts:
- moved C48 0.74 mm to (140.8, 101.2)
- moved C43 0.67 mm to (140.8, 106.6)
- moved C40 0.67 mm to (140.8, 104.2)
- moved C30 0.06 mm to (147.2, 98.2)
Routing:
- net VDDO2_3: track 5.27 -> 13.2 mm, vias 0 -> 3
- net LF1: track 0.00 -> 1.42 mm
- net LF2: track 0.00 -> 1.41 mm
- net GND: track 0.00 -> 0.91 mm, vias 0 -> 1

Commit message: pcb updaate
Parts:
- C51, C52: moved to B.Cu
- moved C52 0.39 mm to (145.3, 109.6)
- moved C51 0.38 mm to (144.3, 109.6)
Routing:
- net VDDDIG: track 0.00 -> 2.51 mm, vias 0 -> 1
- net VDDIN: track 0.00 -> 2.28 mm, vias 0 -> 1
Other:
- board text added: "N"
- board text added: "P"
