File: hardware/schematic/v1.0/CLOCK_CORE/CLOCK_CORE.kicad_pcb (KiCad board)
At the start: 4 copper layers, 70 x 70 mm, 137 parts, among them CN1 LAIL-PHC2_54-2P-01-XH-L, J1 Conn_Coaxial, J3 Conn_01x04_Socket, U1 OCXO_20x20mm, U2 OCXO_25.4x25.4mm, U3 TPS7A5201RPSR, U4 TPS7A5201RPSR, U5 LMK5B12204, U6 REF5040

Commit message: pcb update
Parts:
- moved C46 0.61 mm to (155.1, 99.1)
- moved C47 0.40 mm to (152.4, 99.8)
- moved C34 0.23 mm to (151.3, 104.7)
- moved FB6 0.21 mm to (153.8, 99.5)
- moved C37 0.06 mm to (151.3, 102.2)
Routing:
- net VDDO0_1: track 0.00 -> 11.4 mm, vias 0 -> 2
- net GND: track 0.91 -> 3.15 mm, vias 1 -> 3
- net STATUS0: track 0.00 -> 1.93 mm, vias 0 -> 1
- net +3.3V: track 1.72 -> 3.05 mm
Changed lines of the file:
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@@
 	)
 	(footprint "Capacitor_SMD:C_0402_1005Metric"
+		(locked yes)
 		(layer "F.Cu")
-		(at 152.062501 99.6825 -90)
+		(at 152.449999 99.76 -90)
 		(descr "Capacitor SMD 0402 (1005 Metric), square (rectangular) end terminal, IPC-7351 nominal, (Body size source: IPC-SM-782 page 76, https://www.pcb-3d.com/wordpress/wp-content/uploads/ipc-sm-782a_amendment_1_and_2.pdf)")
 		(tags "capacitor")
@@
 	)
 	(footprint "Inductor_SMD:L_0603_1608Metric"
+		(locked yes)
 		(layer "F.Cu")
-		(at 153.962501 99.374999 -90)
+		(at 153.7725 99.454999 -90)
 		(descr "Inductor SMD 0603 (1608 Metric), square (rectangular) end terminal, IPC-7351 nominal, (Body size source: http://www.tortai-tech.com/upload/download/2011102023233369053.pdf)")
 		(tags "inductor")
@@
 	)
 	(footprint "Capacitor_SMD:C_0402_1005Metric"
+		(locked yes)
 		(layer "F.Cu")
-		(at 155.462501 99.63 90)
+		(at 155.1 99.14 90)
 		(descr "Capacitor SMD 0402 (1005 Metric), square (rectangular) end terminal, IPC-7351 nominal, (Body size source: IPC-SM-782 page 76, https://www.pcb-3d.com/wordpress/wp-content/uploads/ipc-sm-782a_amendment_1_and_2.pdf)")
 		(tags "capacitor")
@@
 	)
 	(footprint "Capacitor_SMD:C_0402_1005Metric"
+		(locked yes)
 		(layer "B.Cu")
-		(at 151.212501 102.1825 -90)
+		(at 151.27 102.18 -90)
 		(descr "Capacitor SMD 0402 (1005 Metric), square (rectangular) end terminal, IPC-7351 nominal, (Body size source: IPC-SM-782 page 76, https://www.pcb-3d.com/wordpress/wp-content/uploads/ipc-sm-782a_amendment_1_and_2.pdf)")
 		(tags "capacitor")
@@
 	)
 	(footprint "Capacitor_SMD:C_0402_1005Metric"
+		(locked yes)
 		(layer "B.Cu")
-		(at 151.212501 104.8925 90)
+		(at 151.27 104.67 90)
 		(descr "Capacitor SMD 0402 (1005 Metric), square (rectangular) end terminal, IPC-7351 nominal, (Body size source: IPC-SM-782 page 76, https://www.pcb-3d.com/wordpress/wp-content/uploads/ipc-sm-782a_amendment_1_and_2.pdf)")
 		(tags "capacitor")
@@
 		(net "OCXO_VCC")
 	)
+	(segment
+		(start 151.62 99.28)
+		(end 151.43 99.09)
+		(width 0.3)
+		(locked yes)
+		(layer "F.Cu")
+		(net "GND")
+	)
+	(segment
+		(start 155.1 99.62)
+		(end 155.83 99.62)
+		(width 0.3)
+		(locked yes)
+		(layer "F.Cu")
+		(net "GND")
+	)
+	(segment
+		(start 152.449999 99.28)
+		(end 151.62 99.28)
+		(width 0.3)
+		(locked yes)
+		(layer "F.Cu")
+		(net "GND")
+	)
+	(segment
+		(start 155.83 99.62)
+		(end 156.12 99.33)
+		(width 0.3)
+		(locked yes)
+		(layer "F.Cu")
+		(net "GND")
+	)
+	(via
+		(at 151.43 99.09)
+		(size 0.5)
+		(drill 0.3)
+		(layers "F.Cu" "B.Cu")
+		(locked yes)
+		(net "GND")
+	)
+	(via
+		(at 156.12 99.33)
+		(size 0.5)
+		(drill 0.3)
+		(layers "F.Cu" "B.Cu")
+		(net "GND")
+	)
 	(via
 		(at 139.92 100.77)
@@
 	)
 	(segment
+		(start 142.54 106.95)
+		(end 143.65 106.95)
+		(width 0.2)
+		(layer "F.Cu")
+		(net "STATUS0")
+	)
+	(segment
+		(start 141.96 107.53)
+		(end 142.54 106.95)
+		(width 0.2)
+		(layer "F.Cu")
+		(net "STATUS0")
+	)
+	(via
+		(at 141.96 107.53)
+		(size 0.6)
+		(drill 0.3)
+		(layers "F.Cu" "B.Cu")
+		(net "STATUS0")
+	)
+	(segment
 		(start 144.425 108.285)
 		(end 144.39 108.285)
@@
 	)
 	(segment
+		(start 149.8375 103.7625)
+		(end 150.9675 103.7625)
+		(width 0.2)
+		(locked yes)
+		(layer "F.Cu")
+		(net "VDDO0_1")
+	)
+	(segment
+		(start 150.9675 103.7625)
+		(end 151.27 103.46)
+		(width 0.2)
+		(locked yes)
+		(layer "F.Cu")
+		(net "VDDO0_1")
+	)
+	(segment
+		(start 151.0725 103.2625)
+		(end 151.27 103.46)
+		(width 0.2)
+		(locked yes)
+		(layer "F.Cu")
+		(net "VDDO0_1")
+	)
+	(segment
+		(start 149.8375 103.2625)
+		(end 151.0725 103.2625)
+		(width 0.2)
+		(locked yes)
+		(layer "F.Cu")
+		(net "VDDO0_1")
+	)
+	(segment
+		(start 152.449999 100.24)
+		(end 153.77 100.24)
+		(width 0.5)
+		(locked yes)
+		(layer "F.Cu")
+		(net "VDDO0_1")
+	)
+	(segment
+		(start 152.449999 100.24)
+		(end 151.53 100.24)
+		(width 0.3)
+		(locked yes)
+		(layer "F.Cu")
+		(net "VDDO0_1")
+	)
+	(segment
+		(start 153.77 100.24)
+		(end 153.7725 100.2425)
+		(width 0.2)
+		(locked yes)
+		(layer "F.Cu")
+		(net "VDDO0_1")
+	)
+	(via
+		(at 151.27 103.46)
+		(size 0.5)
+		(drill 0.3)
+		(layers "F.Cu" "B.Cu")
+		(locked yes)
+		(net "VDDO0_1")
+	)
+	(via
+		(at 151.53 100.24)
+		(size 0.5)
+		(drill 0.3)
+		(layers "F.Cu" "B.Cu")
+		(locked yes)
+		(net "VDDO0_1")
+	)
+	(segment
+		(start 151.27 103.46)
+		(end 151.27 104.19)
+		(width 0.2)
+		(layer "B.Cu")
+		(net "VDDO0_1")
+	)
+	(segment
+		(start 152.36 101.25)
+		(end 151.53 100.42)
+		(width 0.3)
+		(locked yes)
+		(layer "B.Cu")
+		(net "VDDO0_1")
+	)
+	(segment
+		(start 151.27 103.46)
+		(end 152.15 103.46)
+		(width 0.3)
+		(locked yes)
+		(layer "B.Cu")
+		(net "VDDO0_1")
+	)
+	(segment
+		(start 151.53 100.42)
+		(end 151.53 100.24)
+		(width 0.3)
+		(layer "B.Cu")
+		(net "VDDO0_1")
+	)
+	(segment
+		(start 152.36 103.25)
+		(end 152.36 101.25)
+		(width 0.3)
+		(locked yes)
+		(layer "B.Cu")
+		(net "VDDO0_1")
+	)
+	(segment
+		(start 152.15 103.46)
+		(end 152.36 103.25)
+		(width 0.3)
+		(locked yes)
+		(layer "B.Cu")
+		(net "VDDO0_1")
+	)
+	(segment
+		(start 151.27 103.46)
+		(end 151.27 102.66)
+		(width 0.2)
+		(layer "B.Cu")
+		(net "VDDO0_1")
+	)
+	(segment
 		(start 162.558999 97.259)
 		(end 160.56072 97.259)
@@
 	)
 	(segment
+		(start 155.1 98.66)
+		(end 153.779998 98.66)
+		(width 0.3)
+		(locked yes)
+		(layer "F.Cu")
+		(net "+3.3V")
+	)
+	(segment
 		(start 138.242502 97.93)
 		(end 138.5 98.187498)
@@
 		(layer "F.Cu")
 		(net "+3.3V")
+	)
+	(segment
+		(start 153.779998 98.66)
+		(end 153.7725 98.667498)
+		(width 0.3)
+		(locked yes)
+		(layer "F.Cu")
+		(net "+3.3V")
