File: hardware/schematic/v1.0/CLOCK_CORE/CLOCK_CORE.kicad_pcb (KiCad board)
At the start: 4 copper layers, 70 x 70 mm, 137 parts, among them CN1 LAIL-PHC2_54-2P-01-XH-L, J1 Conn_Coaxial, J3 Conn_01x04_Socket, U1 OCXO_20x20mm, U2 OCXO_25.4x25.4mm, U3 TPS7A5201RPSR, U4 TPS7A5201RPSR, U5 LMK5B12204, U6 REF5040

Commit message: pcb update
Routing:
- net +3.3V: vias 22 -> 28
- added copper zone on B.Cu, net +3.3V
Changed lines of the file:
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@@
 	)
 	(footprint "LED_SMD:LED_0603_1608Metric"
+		(locked yes)
 		(layer "F.Cu")
 		(at 130 123)
@@
 	)
 	(footprint "LED_SMD:LED_0603_1608Metric"
+		(locked yes)
 		(layer "F.Cu")
 		(at 130 120.6)
@@
 		(tags "capacitor")
 		(property "Reference" "C38"
-			(at 0.03 -0.95 0)
+			(at 1.872501 0.0025 0)
 			(layer "B.SilkS")
 			(effects
@@
 		(tags "capacitor")
 		(property "Reference" "C35"
-			(at 0.03 -1 0)
+			(at -1.8 0 0)
 			(layer "B.SilkS")
 			(effects
@@
 	)
 	(via
+		(at 139.89 94.7)
+		(size 0.5)
+		(drill 0.3)
+		(layers "F.Cu" "B.Cu")
+		(free yes)
+		(net "+3.3V")
+	)
+	(via
+		(at 148.36 93.02)
+		(size 0.5)
+		(drill 0.3)
+		(layers "F.Cu" "B.Cu")
+		(locked yes)
+		(free yes)
+		(net "+3.3V")
+	)
+	(via
+		(at 152.33 93.04)
+		(size 0.5)
+		(drill 0.3)
+		(layers "F.Cu" "B.Cu")
+		(locked yes)
+		(free yes)
+		(net "+3.3V")
+	)
+	(via
+		(at 149.03 93.02)
+		(size 0.5)
+		(drill 0.3)
+		(layers "F.Cu" "B.Cu")
+		(locked yes)
+		(free yes)
+		(net "+3.3V")
+	)
+	(via
 		(at 140.42 116.64)
 		(size 0.5)
@@
 	)
 	(via
+		(at 153 93.04)
+		(size 0.5)
+		(drill 0.3)
+		(layers "F.Cu" "B.Cu")
+		(locked yes)
+		(free yes)
+		(net "+3.3V")
+	)
+	(via
+		(at 139.33 94.71)
+		(size 0.5)
+		(drill 0.3)
+		(layers "F.Cu" "B.Cu")
+		(free yes)
+		(net "+3.3V")
+	)
+	(via
 		(at 140.41 117.16)
 		(size 0.5)
@@
 		(start 139.72 95.68)
 		(end 141.115002 95.68)
-		(width 0.3)
+		(width 0.4)
 		(layer "B.Cu")
 		(net "+3.3V")
@@
 		(drill 0.3)
 		(layers "F.Cu" "B.Cu")
+		(locked yes)
 		(free yes)
 		(net "+5V")
@@
 		(drill 0.3)
 		(layers "F.Cu" "B.Cu")
+		(locked yes)
 		(free yes)
 		(net "+5V")
@@
 		(drill 0.3)
 		(layers "F.Cu" "B.Cu")
+		(locked yes)
 		(free yes)
 		(net "+5V")
@@
 		(drill 0.3)
 		(layers "F.Cu" "B.Cu")
+		(locked yes)
 		(free yes)
 		(net "+5V")
@@
 	(zone
 		(net "+5V")
+		(locked yes)
 		(layer "F.Cu")
 		(hatch edge 0.5)
@@
 		(polygon
 			(pts
-				(xy 151.63 63.48) (xy 154.5 63.48) (xy 154.5 65.45) (xy 151.63 65.45)
+				(xy 151.628414 63.51) (xy 154.498414 63.51) (xy 154.498414 65.48) (xy 151.628414 65.48)
 			)
 		)
@@
 	)
 	(zone
+		(net "+3.3V")
+		(layer "B.Cu")
+		(hatch edge 0.5)
+		(priority 20)
+		(connect_pads yes
+			(clearance 0.1)
+		)
+		(min_thickness 0.1)
+		(fill yes
+			(thermal_gap 0.5)
+			(thermal_bridge_width 0.5)
+			(island_removal_mode 0)
+		)
+		(polygon
+			(pts
+				(xy 138.97 94.38) (xy 138.97 95.98) (xy 140.21 95.98) (xy 140.21 94.38)
+			)
+		)
+	)
+	(zone
+		(net "+3.3V")
+		(layer "B.Cu")
+		(hatch edge 0.5)
+		(priority 23)
+		(connect_pads yes
+			(clearance 0.1)
+		)
+		(min_thickness 0.1)
+		(fill yes
+			(thermal_gap 0.5)
+			(thermal_bridge_width 0.5)
+			(island_removal_mode 0)
+		)
+		(polygon
+			(pts
+				(xy 150.8 93.71) (xy 150.8 94.44) (xy 153.28 94.44) (xy 153.28 92.69) (xy 152.07 92.69) (xy 152.07 93.71)
+			)
+		)
+	)
+	(zone
+		(net "+3.3V")
+		(locked yes)
+		(layer "B.Cu")
+		(hatch edge 0.5)
+		(priority 23)
+		(connect_pads yes
+			(clearance 0.1)
+		)
+		(min_thickness 0.1)
+		(fill yes
+			(thermal_gap 0.5)
+			(thermal_bridge_width 0.5)
+			(island_removal_mode 0)
+		)
+		(polygon
+			(pts
+				(xy 146.84 93.66) (xy 146.84 94.39) (xy 149.32 94.39) (xy 149.32 92.64) (xy 148.11 92.64) (xy 148.11 93.66)
+			)
+		)
+	)
+	(zone
 		(net "GND")
 		(layer "In1.Cu")
@@
 	(zone
 		(net "+5V")
+		(locked yes)
 		(layer "In2.Cu")
 		(hatch edge 0.5)
@@
 		(layer "In2.Cu")
 		(hatch edge 0.5)
+		(priority 22)
+		(connect_pads yes
+			(clearance 0.1)
+		)
+		(min_thickness 0.1)
+		(fill yes
+			(thermal_gap 0.5)
+			(thermal_bridge_width 0.5)
+			(island_removal_mode 0)
+		)
+		(polygon
+			(pts
+				(xy 136.2 94.95) (xy 136.2 92.6) (xy 154.53 92.6) (xy 154.53 93.47) (xy 137.66 93.47) (xy 137.66 94.95)
+			)
+		)
+	)
+	(zone
+		(net "+3.3V")
+		(layer "In2.Cu")
+		(hatch edge 0.5)
 		(priority 16)
 		(connect_pads
@@
 			)
 		)
+	)
+	(zone
+		(net "+3.3V")
+		(layer "In2.Cu")
+		(hatch edge 0.5)
+		(priority 21)
+		(connect_pads yes
+			(clearance 0.1)
+		)
+		(min_thickness 0.1)
+		(fill yes
+			(thermal_gap 0.5)
+			(thermal_bridge_width 0.5)
+			(island_removal_mode 0)
+		)
+		(polygon
+			(pts
+				(xy 137.42 94.39) (xy 140.21 94.39) (xy 140.21 95.11) (xy 137.42 95.11)
+			)
+		)

Commit message: pcb update
Parts:
- moved TP2 1.42 mm to (161.6, 81.1)
Routing:
- net +3.3V: track 11.1 -> 13.6 mm, vias 28 -> 32
- net GND: track 2.05 -> 0.91 mm, vias 2 -> 1
Changed lines of the file:
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@@
 		(tags "resistor")
 		(property "Reference" "R26"
-			(at 2.425 0 90)
+			(at -0.245 -1.21 90)
 			(layer "F.SilkS")
 			(effects
@@
 		(tags "resistor")
 		(property "Reference" "R27"
-			(at 2.45 0 90)
+			(at -0.11 -1.21 90)
 			(layer "F.SilkS")
 			(effects
@@
 	)
 	(footprint "Capacitor_SMD:C_0402_1005Metric"
+		(locked yes)
 		(layer "F.Cu")
 		(at 143.55 97.42 -90)
@@
 	(footprint "TestPoint:TestPoint_Pad_D1.0mm"
 		(layer "F.Cu")
-		(at 162.58 82.11)
+		(at 161.56 81.12)
 		(descr "SMD pad as test Point, diameter 1.0mm")
 		(tags "test point SMD pad")
@@
 	)
 	(footprint "Capacitor_SMD:C_0402_1005Metric"
+		(locked yes)
 		(layer "F.Cu")
 		(at 148.17 97.5 -90)
@@
 		(tags "capacitor")
 		(property "Reference" "C46"
-			(at 1.45 0 180)
+			(at 0.02 0.93 270)
 			(layer "F.SilkS")
 			(effects
@@
 		(net "OCXO_VCC")
 	)
-	(segment
-		(start 155.1 99.62)
-		(end 155.83 99.62)
-		(width 0.3)
-		(locked yes)
-		(layer "F.Cu")
-		(net "GND")
-	)
-	(segment
-		(start 155.83 99.62)
-		(end 156.12 99.33)
-		(width 0.3)
-		(locked yes)
-		(layer "F.Cu")
-		(net "GND")
-	)
-	(via
-		(at 156.12 99.33)
-		(size 0.5)
-		(drill 0.3)
-		(layers "F.Cu" "B.Cu")
-		(net "GND")
-	)
 	(via
 		(at 139.92 100.77)
@@
 	)
 	(segment
+		(start 168.84 84.685)
+		(end 168.84 83.415)
+		(width 0.3)
+		(layer "F.Cu")
+		(net "+3.3V")
+	)
+	(segment
 		(start 136.89 97.93)
 		(end 138.242502 97.93)
@@
 	)
 	(segment
+		(start 165.99 84.68)
+		(end 165.99 83.41)
+		(width 0.3)
+		(layer "F.Cu")
+		(net "+3.3V")
+	)
+	(segment
 		(start 149.4 120.0625)
 		(end 148.8675 120.0625)
@@
 	)
 	(via
-		(at 132.56 91.17)
+		(at 132.57 91.24)
 		(size 0.6)
 		(drill 0.3)
@@
 	)
 	(via
+		(at 168.84 83.415)
+		(size 0.5)
+		(drill 0.3)
+		(layers "F.Cu" "B.Cu")
+		(net "+3.3V")
+	)
+	(via
 		(at 140.41 117.16)
 		(size 0.5)
@@
 	)
 	(via
-		(at 131.8 90.45)
+		(at 131.81 90.52)
 		(size 0.6)
 		(drill 0.3)
@@
 	)
 	(via
-		(at 132.56 90.45)
+		(at 132.57 90.52)
 		(size 0.6)
 		(drill 0.3)
@@
 	)
 	(via
-		(at 131.8 91.17)
+		(at 155.66 97.47)
+		(size 0.5)
+		(drill 0.3)
+		(layers "F.Cu" "B.Cu")
+		(free yes)
+		(net "+3.3V")
+	)
+	(via
+		(at 165.99 83.41)
+		(size 0.5)
+		(drill 0.3)
+		(layers "F.Cu" "B.Cu")
+		(net "+3.3V")
+	)
+	(via
+		(at 131.81 91.24)
 		(size 0.6)
 		(drill 0.3)
@@
 	)
 	(via
+		(at 155.12 97.48)
+		(size 0.5)
+		(drill 0.3)
+		(layers "F.Cu" "B.Cu")
+		(free yes)
+		(net "+3.3V")
+	)
+	(via
 		(at 146.14 117.15)
 		(size 0.5)
@@
 	)
 	(zone
+		(net "+3.3V")
+		(layer "F.Cu")
+		(hatch edge 0.5)
+		(priority 26)
+		(connect_pads yes
+			(clearance 0.1)
+		)
+		(min_thickness 0.1)
+		(fill yes
+			(thermal_gap 0.5)
+			(thermal_bridge_width 0.5)
+			(island_removal_mode 0)
+		)
+		(polygon
+			(pts
+				(xy 154.79 96.88) (xy 154.79 99.04) (xy 156.04 99.04) (xy 156.04 96.88)
+			)
+		)
+	)
+	(zone
 		(net "+5V")
 		(layer "F.Cu")
@@
 		(layer "In2.Cu")
 		(hatch edge 0.5)
+		(priority 25)
+		(connect_pads yes
+			(clearance 0.1)
+		)
+		(min_thickness 0.1)
+		(fill yes
+			(thermal_gap 0.5)
+			(thermal_bridge_width 0.5)
+			(island_removal_mode 0)
+		)
+		(polygon
+			(pts
+				(xy 169.71 83.89) (xy 168.01 83.89) (xy 168.01 80.29) (xy 176.35 80.29) (xy 176.35 81.73) (xy 169.71 81.73)
+			)
+		)
+	)
+	(zone
+		(net "+3.3V")
+		(locked yes)
+		(layer "In2.Cu")
+		(hatch edge 0.5)
 		(priority 14)
 		(connect_pads thru_hole_only
@@
 		(layer "In2.Cu")
 		(hatch edge 0.5)
+		(priority 24)
+		(connect_pads yes
+			(clearance 0.1)
+		)
+		(min_thickness 0.1)
+		(fill yes
+			(thermal_gap 0.5)
+			(thermal_bridge_width 0.5)
+			(island_removal_mode 0)
+		)
+		(polygon
+			(pts
+				(xy 163.12 93.46) (xy 161.73 93.46) (xy 161.73 82.89) (xy 169.71 82.89) (xy 169.71 83.89) (xy 163.12 83.89)
+			)
+		)
+	)
+	(zone
+		(net "+3.3V")
+		(locked yes)
+		(layer "In2.Cu")
+		(hatch edge 0.5)
+		(priority 27)
+		(connect_pads yes
+			(clearance 0.1)
+		)
+		(min_thickness 0.1)
+		(fill yes
+			(thermal_gap 0.5)
+			(thermal_bridge_width 0.5)
+			(island_removal_mode 0)
+		)
+		(polygon
+			(pts
+				(xy 154.79 93.25) (xy 154.79 97.8) (xy 156.04 97.8) (xy 156.04 93.25)
+			)
+		)
+	)
+	(zone
+		(net "+3.3V")
+		(locked yes)
+		(layer "In2.Cu")
+		(hatch edge 0.5)
 		(priority 15)
 		(connect_pads yes
@@
 	(zone
 		(net "+3.3V")
+		(locked yes)
 		(layer "In2.Cu")
 		(hatch edge 0.5)
@@
 		(polygon
 			(pts
-				(xy 136.2 94.95) (xy 136.2 92.6) (xy 154.53 92.6) (xy 154.53 93.47) (xy 137.66 93.47) (xy 137.66 94.95)
+				(xy 136.2 94.95) (xy 136.2 92.6) (xy 163.12 92.6) (xy 163.12 93.6) (xy 137.66 93.6) (xy 137.66 94.95)
 			)
 		)

Commit message: pcb update
Routing:
- net /DEBUG/SDA: track 19.6 -> 43.0 mm
- net /DEBUG/SCL: track 23.6 -> 45.6 mm
Changed lines of the file:
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@@
-	)
-	(segment
-		(start 149.15 100.075)
-		(end 150.245 100.075)
-		(width 0.15)
-		(layer "F.Cu")
-		(net "/DEBUG/SDA")
 	)
 	(segment
@@
 	)
 	(segment
-		(start 150.245 100.075)
-		(end 150.91 99.41)
-		(width 0.15)
+		(start 152.19 98.31)
+		(end 152.19 98.54)
+		(width 0.2)
 		(layer "F.Cu")
 		(net "/DEBUG/SDA")
@@
 	)
 	(segment
+		(start 150.655 100.075)
+		(end 149.15 100.075)
+		(width 0.2)
+		(layer "F.Cu")
+		(net "/DEBUG/SDA")
+	)
+	(segment
+		(start 152.19 98.54)
+		(end 150.655 100.075)
+		(width 0.2)
+		(layer "F.Cu")
+		(net "/DEBUG/SDA")
+	)
+	(segment
 		(start 175.859999 75.880001)
 		(end 178.2 75.880001)
@@
 	)
 	(via
-		(at 150.91 99.41)
-		(size 0.5)
+		(at 152.19 98.31)
+		(size 0.6)
 		(drill 0.3)
 		(layers "F.Cu" "B.Cu")
@@
 	)
 	(segment
+		(start 152.19 98.31)
+		(end 156.6 93.9)
+		(width 0.2)
+		(layer "B.Cu")
+		(net "/DEBUG/SDA")
+	)
+	(segment
+		(start 168.84 88.61)
+		(end 168.84 87.825)
+		(width 0.2)
+		(layer "B.Cu")
+		(net "/DEBUG/SDA")
+	)
+	(segment
+		(start 163.55 93.9)
+		(end 168.84 88.61)
+		(width 0.2)
+		(layer "B.Cu")
+		(net "/DEBUG/SDA")
+	)
+	(segment
+		(start 156.6 93.9)
+		(end 163.55 93.9)
+		(width 0.2)
+		(layer "B.Cu")
+		(net "/DEBUG/SDA")
+	)
+	(segment
 		(start 148.65 100.075)
 		(end 148.65 99.637501)
@@
 		(net "/DEBUG/SCL")
 	)
+	(segment
+		(start 161.68 93.17)
+		(end 165.99 88.86)
+		(width 0.2)
+		(layer "B.Cu")
+		(net "/DEBUG/SCL")
+	)
+	(segment
+		(start 155.75 93.17)
+		(end 161.68 93.17)
+		(width 0.2)
+		(layer "B.Cu")
+		(net "/DEBUG/SCL")
+	)
+	(segment
+		(start 165.99 88.86)
+		(end 165.99 87.82)
+		(width 0.2)
+		(layer "B.Cu")
+		(net "/DEBUG/SCL")
+	)
+	(segment
+		(start 151.4 98.69)
+		(end 151.4 97.52)
+		(width 0.2)
+		(layer "B.Cu")
+		(net "/DEBUG/SCL")
+	)
+	(segment
+		(start 151.4 97.52)
+		(end 155.75 93.17)
+		(width 0.2)
+		(layer "B.Cu")
+		(net "/DEBUG/SCL")
+	)
+	(segment
+		(start 150.89 99.2)
+		(end 151.4 98.69)
+		(width 0.2)
+		(layer "B.Cu")
+		(net "/DEBUG/SCL")
+	)
+	(segment
+		(start 150 99.2)
+		(end 150.89 99.2)
+		(width 0.2)
+		(layer "B.Cu")
+		(net "/DEBUG/SCL")
+	)

Commit message: pcb update
Parts:
- moved TP1 0.39 mm to (135.9, 66.7)
Routing:
- net GND: track 0.91 -> 109.8 mm, vias 1 -> 89
- net +3.3V: track 13.6 -> 16.9 mm

Commit message: pcb update
Routing:
- net +5V: track 0.00 -> 1.14 mm
Changed lines of the file:
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@@
 		(tags "capacitor")
 		(property "Reference" "C27"
-			(at -1.52 0 180)
+			(at -0.2 -0.89 270)
 			(layer "F.SilkS")
 			(effects
@@
 		(tags "capacitor")
 		(property "Reference" "C52"
-			(at -1.52 0 0)
+			(at -0.01 0.93 90)
 			(layer "B.SilkS")
 			(effects
@@
 		(tags "capacitor")
 		(property "Reference" "C51"
-			(at -1.52 0 0)
+			(at -0.02 -0.83 270)
 			(layer "B.SilkS")
 			(effects
@@
 		(net "/POWER/+5V_IN")
 	)
+	(segment
+		(start 125.381406 65.448594)
+		(end 125.162126 65.667874)
+		(width 0.3)
+		(locked yes)
+		(layer "F.Cu")
+		(net "+5V")
+	)
+	(segment
+		(start 125.387126 65.448594)
+		(end 125.381406 65.448594)
+		(width 0.3)
+		(locked yes)
+		(layer "F.Cu")
+		(net "+5V")
+	)
+	(segment
+		(start 124.285 85.945)
+		(end 124.285 86.195)
+		(width 0.3)
+		(locked yes)
+		(layer "F.Cu")
+		(net "+5V")
+	)
+	(segment
+		(start 124.51 85.72)
+		(end 124.285 85.945)
+		(width 0.3)
+		(locked yes)
+		(layer "F.Cu")
+		(net "+5V")
+	)
+	(segment
+		(start 125.162126 65.667874)
+		(end 125.162126 65.923594)
+		(width 0.3)
+		(locked yes)
+		(layer "F.Cu")
+		(net "+5V")
+	)
 	(via

Commit message: pcb update
Routing:
- net /LMK5B12204/PDN: track 3.50 -> 96.9 mm, vias 0 -> 2
- net GND: track 109.8 -> 110.6 mm
Changed lines of the file:
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@@
 	)
 	(footprint "Capacitor_SMD:C_0402_1005Metric"
-		(locked yes)
 		(layer "F.Cu")
 		(at 151.3 106.87 90)
@@
 		(tags "capacitor")
 		(property "Reference" "C45"
-			(at 0.03 1.1 90)
+			(at 0 1.96 90)
 			(layer "F.SilkS")
 			(effects
@@
 	)
 	(footprint "Connector_PinHeader_2.54mm:PinHeader_1x04_P2.54mm_Vertical"
+		(locked yes)
 		(layer "F.Cu")
 		(at 178.2 80.96 180)
@@
 	)
 	(via
-		(at 152.17 106.05)
+		(at 153.26 105.51)
 		(size 0.6)
 		(drill 0.3)
@@
 	)
 	(segment
+		(start 151.27 105.15)
+		(end 151.63 105.51)
+		(width 0.3)
+		(layer "B.Cu")
+		(net "GND")
+	)
+	(segment
 		(start 151.27 101.295)
 		(end 150.7375 100.7625)
@@
 	)
 	(segment
-		(start 151.27 105.15)
-		(end 152.17 106.05)
-		(width 0.3)
-		(layer "B.Cu")
-		(net "GND")
-	)
-	(segment
 		(start 147.25 96.8)
 		(end 147.41 96.96)
@@
 	)
 	(segment
+		(start 151.63 105.51)
+		(end 153.26 105.51)
+		(width 0.3)
+		(layer "B.Cu")
+		(net "GND")
+	)
+	(segment
 		(start 145.29 110.04)
 		(end 145.29 110.79)
@@
 	)
 	(segment
-		(start 138.34 109.56)
-		(end 138.34 116.01)
+		(start 139.99 107.91)
+		(end 136.42 111.48)
 		(width 0.2)
 		(layer "B.Cu")
@@
 	)
 	(segment
-		(start 133.75 120.6)
-		(end 132.16 120.6)
+		(start 141.58 107.91)
+		(end 139.99 107.91)
 		(width 0.2)
 		(layer "B.Cu")
@@
 	)
 	(segment
-		(start 139.99 107.91)
-		(end 138.34 109.56)
+		(start 136.42 111.48)
+		(end 136.42 117.93)
 		(width 0.2)
 		(layer "B.Cu")
@@
 	)
 	(segment
-		(start 141.58 107.91)
-		(end 139.99 107.91)
+		(start 136.42 117.93)
+		(end 133.75 120.6)
 		(width 0.2)
 		(layer "B.Cu")
@@
 	)
 	(segment
-		(start 138.34 116.01)
-		(end 133.75 120.6)
+		(start 133.75 120.6)
+		(end 132.16 120.6)
 		(width 0.2)
 		(layer "B.Cu")
@@
 	)
 	(segment
-		(start 133.74 123)
-		(end 132.19 123)
+		(start 137.33 119.41)
+		(end 133.74 123)
 		(width 0.2)
 		(layer "B.Cu")
@@
 	)
 	(segment
-		(start 141.16 108.74)
-		(end 139.82 110.08)
+		(start 137.33 112.57)
+		(end 137.33 119.41)
 		(width 0.2)
 		(layer "B.Cu")
@@
 	)
 	(segment
-		(start 139.82 116.92)
-		(end 133.74 123)
+		(start 141.16 108.74)
+		(end 137.33 112.57)
 		(width 0.2)
 		(layer "B.Cu")
@@
 	)
 	(segment
-		(start 139.82 110.08)
-		(end 139.82 116.92)
+		(start 133.74 123)
+		(end 132.19 123)
 		(width 0.2)
 		(layer "B.Cu")
@@
 	)
 	(segment
+		(start 127.872748 87.674687)
+		(end 127.872748 88.067252)
+		(width 0.3)
+		(layer "F.Cu")
+		(net "/LMK5B12204/PDN")
+	)
+	(segment
 		(start 126.918061 86.72)
 		(end 127.872748 87.674687)
@@
 	)
 	(segment
+		(start 151.3 106.39)
+		(end 152.3 106.39)
+		(width 0.3)
+		(layer "F.Cu")
+		(net "/LMK5B12204/PDN")
+	)
+	(segment
 		(start 151.1725 106.2625)
 		(end 151.3 106.39)
@@
 	)
 	(segment
+		(start 127.872748 88.067252)
+		(end 126.98 88.96)
+		(width 0.3)
+		(layer "F.Cu")
+		(net "/LMK5B12204/PDN")
+	)
+	(segment
 		(start 126.285 86.72)
 		(end 126.918061 86.72)
@@
 		(net "/LMK5B12204/PDN")
 	)
+	(via
+		(at 152.3 106.39)
+		(size 0.5)
+		(drill 0.3)
+		(layers "F.Cu" "B.Cu")
+		(net "/LMK5B12204/PDN")
+	)
+	(via
+		(at 126.98 88.96)
+		(size 0.5)
+		(drill 0.3)
+		(layers "F.Cu" "B.Cu")
+		(net "/LMK5B12204/PDN")
+	)
+	(segment
+		(start 153.58 106.39)
+		(end 152.3 106.39)
+		(width 0.3)
+		(layer "In2.Cu")
+		(net "/LMK5B12204/PDN")
+	)
+	(segment
+		(start 124.4 90.41)
+		(end 124.4 121.93)
+		(width 0.3)
+		(layer "In2.Cu")
+		(net "/LMK5B12204/PDN")
+	)
+	(segment
+		(start 157.13 109.94)
+		(end 153.58 106.39)
+		(width 0.3)
+		(layer "In2.Cu")
+		(net "/LMK5B12204/PDN")
+	)
+	(segment
+		(start 157.13 124.55)
+		(end 157.13 109.94)
+		(width 0.3)
+		(layer "In2.Cu")
+		(net "/LMK5B12204/PDN")
+	)
+	(segment
+		(start 124.4 121.93)
+		(end 128.59 126.12)
+		(width 0.3)
+		(layer "In2.Cu")
+		(net "/LMK5B12204/PDN")
+	)
+	(segment
+		(start 126.98 88.96)
+		(end 125.85 88.96)
+		(width 0.3)
+		(layer "In2.Cu")
+		(net "/LMK5B12204/PDN")
+	)
+	(segment
+		(start 128.59 126.12)
+		(end 155.56 126.12)
+		(width 0.3)
+		(layer "In2.Cu")
+		(net "/LMK5B12204/PDN")
+	)
+	(segment
+		(start 125.85 88.96)
+		(end 124.4 90.41)
+		(width 0.3)
+		(layer "In2.Cu")
+		(net "/LMK5B12204/PDN")
+	)
+	(segment
+		(start 155.56 126.12)
+		(end 157.13 124.55)
+		(width 0.3)
+		(layer "In2.Cu")
+		(net "/LMK5B12204/PDN")
+	)

Commit message: pcb update
Routing:
- net 3.3V_OCXO: track 0.00 -> 5.83 mm, vias 0 -> 2
- net VDDIN: track 3.68 -> 9.29 mm, vias 1 -> 2
- net VDDDIG: track 0.00 -> 1.16 mm, vias 0 -> 1
Changed lines of the file:
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@@
 		(tags "resistor")
 		(property "Reference" "R23"
-			(at 0.01 1.05 0)
+			(at 0 0.889998 0)
 			(layer "F.SilkS")
 			(effects
@@
 	)
 	(segment
-		(start 144.15 107.387499)
-		(end 143.727499 107.81)
+		(start 141.92 108.74)
+		(end 141.16 108.74)
 		(width 0.15)
 		(layer "F.Cu")
@@
 	)
 	(segment
-		(start 142.28 108.74)
-		(end 141.16 108.74)
+		(start 144.15 106.95)
+		(end 144.15 107.387499)
 		(width 0.15)
 		(layer "F.Cu")
@@
 	)
 	(segment
-		(start 144.15 106.95)
-		(end 144.15 107.387499)
+		(start 144.15 107.387499)
+		(end 143.727499 107.81)
 		(width 0.15)
 		(layer "F.Cu")
@@
 	)
 	(segment
-		(start 143.21 107.81)
-		(end 142.28 108.74)
+		(start 142.85 107.81)
+		(end 141.92 108.74)
 		(width 0.15)
 		(layer "F.Cu")
@@
 	(segment
 		(start 143.727499 107.81)
-		(end 143.21 107.81)
+		(end 142.85 107.81)
 		(width 0.15)
 		(layer "F.Cu")
@@
 	)
 	(segment
+		(start 142.462501 112.7)
+		(end 142.462501 113.8625)
+		(width 0.3)
+		(layer "F.Cu")
+		(net "VDDDIG")
+	)
+	(via
+		(at 142.462501 112.7)
+		(size 0.5)
+		(drill 0.3)
+		(layers "F.Cu" "B.Cu")
+		(net "VDDDIG")
+	)
+	(segment
+		(start 144.529998 112.4275)
+		(end 144.529998 111.650002)
+		(width 0.3)
+		(layer "F.Cu")
+		(net "VDDIN")
+	)
+	(segment
 		(start 145.649999 107.930001)
 		(end 145.649999 106.95)
@@
 	)
 	(segment
+		(start 144.529998 111.650002)
+		(end 144.53 111.65)
+		(width 0.3)
+		(layer "F.Cu")
+		(net "VDDIN")
+	)
+	(segment
 		(start 144.529998 113.827499)
 		(end 144.532499 113.83)
@@
 	)
 	(via
+		(at 144.53 111.65)
+		(size 0.5)
+		(drill 0.3)
+		(layers "F.Cu" "B.Cu")
+		(net "VDDIN")
+	)
+	(via
 		(at 145.430172 108.476012)
 		(size 0.5)
@@
 	)
 	(segment
+		(start 146.15 111.2)
+		(end 146.15 109.19584)
+		(width 0.3)
+		(layer "In2.Cu")
+		(net "VDDIN")
+	)
+	(segment
+		(start 145.7 111.65)
+		(end 146.15 111.2)
+		(width 0.3)
+		(layer "In2.Cu")
+		(net "VDDIN")
+	)
+	(segment
+		(start 146.15 109.19584)
+		(end 145.430172 108.476012)
+		(width 0.3)
+		(layer "In2.Cu")
+		(net "VDDIN")
+	)
+	(segment
+		(start 144.53 111.65)
+		(end 145.7 111.65)
+		(width 0.3)
+		(layer "In2.Cu")
+		(net "VDDIN")
+	)
+	(segment
 		(start 146.15 108.9)
 		(end 155.19 117.94)
@@
 	)
 	(segment
+		(start 129.82 67.280002)
+		(end 129.82 68.77)
+		(width 0.3)
+		(layer "F.Cu")
+		(net "3.3V_OCXO")
+	)
+	(via
+		(at 129.69 64.48)
+		(size 0.6)
+		(drill 0.3)
+		(layers "F.Cu" "B.Cu")
+		(free yes)
+		(net "3.3V_OCXO")
+	)
+	(via
+		(at 129.82 68.77)
+		(size 0.5)
+		(drill 0.3)
+		(layers "F.Cu" "B.Cu")
+		(net "3.3V_OCXO")
+	)
+	(segment
+		(start 129.69 64.48)
+		(end 129.69 68.64)
+		(width 0.3)
+		(layer "In2.Cu")
+		(net "3.3V_OCXO")
+	)
+	(segment
+		(start 129.69 68.64)
+		(end 129.82 68.77)
+		(width 0.3)
+		(layer "In2.Cu")
+		(net "3.3V_OCXO")
+	)
+	(segment

Commit message: pcb update
Parts:
- moved C51 0.49 mm to (144.2, 110.0)
Routing:
- net VDDDIG: track 1.16 -> 8.90 mm, vias 1 -> 2
- net GND: track 110.6 -> 111.1 mm, vias 89 -> 88
Changed lines of the file:
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@@
 	(footprint "Capacitor_SMD:C_0402_1005Metric"
 		(layer "B.Cu")
-		(at 144.28 109.56 90)
+		(at 144.17 110.04 90)
 		(descr "Capacitor SMD 0402 (1005 Metric), square (rectangular) end terminal, IPC-7351 nominal, (Body size source: IPC-SM-782 page 76, https://www.pcb-3d.com/wordpress/wp-content/uploads/ipc-sm-782a_amendment_1_and_2.pdf)")
 		(tags "capacitor")
@@
 	)
 	(via
-		(at 144.28 110.79)
-		(size 0.6)
-		(drill 0.3)
-		(layers "F.Cu" "B.Cu")
-		(net "GND")
-	)
-	(via
 		(at 178.2 112.5)
 		(size 0.6)
@@
 	)
 	(segment
+		(start 144.17 110.52)
+		(end 145.02 110.52)
+		(width 0.3)
+		(layer "B.Cu")
+		(net "GND")
+	)
+	(segment
 		(start 146.51 96.8)
 		(end 147.25 96.8)
@@
 	)
 	(segment
-		(start 144.28 110.04)
-		(end 144.28 110.79)
-		(width 0.3)
-		(layer "B.Cu")
-		(net "GND")
-	)
-	(segment
 		(start 150.1375 94.0975)
 		(end 150.1375 93.2975)
@@
 	)
 	(segment
+		(start 145.02 110.52)
+		(end 145.29 110.79)
+		(width 0.3)
+		(layer "B.Cu")
+		(net "GND")
+	)
+	(segment
 		(start 140.83 100.77)
 		(end 139.92 100.77)
@@
 	)
 	(segment
+		(start 145.15 107.9)
+		(end 144.31 108.74)
+		(width 0.2)
+		(layer "F.Cu")
+		(net "VDDDIG")
+	)
+	(segment
+		(start 145.15 106.95)
+		(end 145.15 107.9)
+		(width 0.2)
+		(layer "F.Cu")
+		(net "VDDDIG")
+	)
+	(segment
 		(start 142.462501 112.7)
 		(end 142.462501 113.8625)
@@
 	)
 	(via
+		(at 144.31 108.74)
+		(size 0.5)
+		(drill 0.3)
+		(layers "F.Cu" "B.Cu")
+		(net "VDDDIG")
+	)
+	(via
 		(at 142.462501 112.7)
 		(size 0.5)
 		(drill 0.3)
 		(layers "F.Cu" "B.Cu")
+		(locked yes)
+		(net "VDDDIG")
+	)
+	(segment
+		(start 144.17 108.88)
+		(end 144.31 108.74)
+		(width 0.3)
+		(layer "B.Cu")
+		(net "VDDDIG")
+	)
+	(segment
+		(start 144.17 109.56)
+		(end 144.17 108.88)
+		(width 0.3)
+		(layer "B.Cu")
+		(net "VDDDIG")
+	)
+	(segment
+		(start 144.31 110.6)
+		(end 144.31 108.74)
+		(width 0.3)
+		(locked yes)
+		(layer "In2.Cu")
+		(net "VDDDIG")
+	)
+	(segment
+		(start 142.462501 112.7)
+		(end 142.462501 112.447499)
+		(width 0.3)
+		(locked yes)
+		(layer "In2.Cu")
+		(net "VDDDIG")
+	)
+	(segment
+		(start 142.462501 112.447499)
+		(end 144.31 110.6)
+		(width 0.3)
+		(locked yes)
+		(layer "In2.Cu")
 		(net "VDDDIG")
 	)
@@
 		(end 146.15 109.19584)
 		(width 0.3)
+		(locked yes)
 		(layer "In2.Cu")
 		(net "VDDIN")
@@
 		(end 146.15 111.2)
 		(width 0.3)
+		(locked yes)
 		(layer "In2.Cu")
 		(net "VDDIN")
@@
 		(end 145.430172 108.476012)
 		(width 0.3)
+		(locked yes)
 		(layer "In2.Cu")
 		(net "VDDIN")
@@
 		(end 145.7 111.65)
 		(width 0.3)
+		(locked yes)
 		(layer "In2.Cu")
 		(net "VDDIN")
