File: hardware/schematic/v1.0/CLOCK_CORE/DEBUG.kicad_sch (KiCad schematic)
At the start: 1 part, among them J2 Conn_01x04_Socket

Commit message: sch and pcb update
Parts:
- added H2, H3, H4, H5: MountingHole_Pad, MountingHole:MountingHole_3.2mm_M3_Pad, symbol Mechanical:MountingHole_Pad
- renumbered J2 to J3
Connections:
- net GND: now also H2.1, H3.1, H4.1, H5.1
Other:
- note added: "HOLE"

Commit message: sch and pcb update
Other:
- note added: "I2C"
Changed lines of the file:
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@@
 	(generator_version "10.0")
 	(paper "A4")
+	(text "I2C"
+		(exclude_from_sim no)
+		(at 163.83 107.696 0)
+		(effects
+			(font
+				(size 2.54 2.54)
+			)
+		)
+	)
 	(text "HOLE"
 		(exclude_from_sim no)
@@
 	(polyline
 		(pts
+			(xy 105.41 73.66) (xy 105.41 111.76)
+		)
+		(stroke
+			(width 0)
+			(type dash)
+		)
+	)
+	(polyline
+		(pts
 			(xy 20.32 186.69) (xy 88.9 186.69)
 		)
@@
 		)
 	)
+	(polyline
+		(pts
+			(xy 105.41 111.76) (xy 173.99 111.76)
+		)
+		(stroke
+			(width 0)
+			(type dash)
+		)
+	)
+	(polyline
+		(pts
+			(xy 173.99 73.66) (xy 173.99 111.76)
+		)
+		(stroke
+			(width 0)
+			(type dash)
+		)
+	)
+	(polyline
+		(pts
+			(xy 105.41 73.66) (xy 173.99 73.66)
+		)
+		(stroke
+			(width 0)
+			(type dash)
+		)
+	)

Commit message: sch and pcb update
Parts:
- H2, H3, H4, H5: footprint MountingHole:MountingHole_3.2mm_M3_Pad -> CLOCK_CORE:MountingHole_3.2mm_M3_Pad; symbol Mechanical:MountingHole_Pad -> CLOCK_CORE:MountingHole_Pad
- J3: footprint Connector_PinHeader_2.54mm:PinHeader_1x04_P2.54mm_Vertical -> CLOCK_CORE:PinHeader_1x04_P2.54mm_Vertical; symbol Connector:Conn_01x04_Socket -> CLOCK_CORE:Conn_01x04_Socket
Changed lines of the file:
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@@
 	)
 	(symbol
-		(lib_id "power:GND")
+		(lib_id "CLOCK_CORE:GND")
 		(at 64.77 176.53 0)
 		(unit 1)
@@
 	)
 	(symbol
-		(lib_id "Mechanical:MountingHole_Pad")
+		(lib_id "CLOCK_CORE:MountingHole_Pad")
 		(at 31.75 158.75 0)
 		(unit 1)
@@
 			)
 		)
-		(property "Footprint" "MountingHole:MountingHole_3.2mm_M3_Pad"
+		(property "Footprint" "CLOCK_CORE:MountingHole_3.2mm_M3_Pad"
 			(at 31.75 158.75 0)
 			(hide yes)
@@
 	)
 	(symbol
-		(lib_id "power:GND")
+		(lib_id "CLOCK_CORE:GND")
 		(at 31.75 176.53 0)
 		(unit 1)
@@
 	)
 	(symbol
-		(lib_id "Mechanical:MountingHole_Pad")
+		(lib_id "CLOCK_CORE:MountingHole_Pad")
 		(at 31.75 173.99 0)
 		(unit 1)
@@
 			)
 		)
-		(property "Footprint" "MountingHole:MountingHole_3.2mm_M3_Pad"
+		(property "Footprint" "CLOCK_CORE:MountingHole_3.2mm_M3_Pad"
 			(at 31.75 173.99 0)
 			(hide yes)
@@
 	)
 	(symbol
-		(lib_id "power:GND")
+		(lib_id "CLOCK_CORE:GND")
 		(at 134.62 92.71 270)
 		(unit 1)
@@
 	)
 	(symbol
-		(lib_id "power:GND")
+		(lib_id "CLOCK_CORE:GND")
 		(at 31.75 161.29 0)
 		(unit 1)
@@
 	)
 	(symbol
-		(lib_id "Connector:Conn_01x04_Socket")
+		(lib_id "CLOCK_CORE:Conn_01x04_Socket")
 		(at 140.97 92.71 0)
 		(unit 1)
@@
 			)
 		)
-		(property "Footprint" "Connector_PinHeader_2.54mm:PinHeader_1x04_P2.54mm_Vertical"
+		(property "Footprint" "CLOCK_CORE:PinHeader_1x04_P2.54mm_Vertical"
 			(at 140.97 92.71 0)
 			(hide yes)
@@
 	)
 	(symbol
-		(lib_id "Mechanical:MountingHole_Pad")
+		(lib_id "CLOCK_CORE:MountingHole_Pad")
 		(at 64.77 173.99 0)
 		(unit 1)
@@
 			)
 		)
-		(property "Footprint" "MountingHole:MountingHole_3.2mm_M3_Pad"
+		(property "Footprint" "CLOCK_CORE:MountingHole_3.2mm_M3_Pad"
 			(at 64.77 173.99 0)
 			(hide yes)
@@
 	)
 	(symbol
-		(lib_id "power:GND")
+		(lib_id "CLOCK_CORE:GND")
 		(at 64.77 161.29 0)
 		(unit 1)
@@
 	)
 	(symbol
-		(lib_id "power:+3.3V")
+		(lib_id "CLOCK_CORE:+3.3V")
 		(at 134.62 90.17 0)
 		(unit 1)
@@
 	)
 	(symbol
-		(lib_id "Mechanical:MountingHole_Pad")
+		(lib_id "CLOCK_CORE:MountingHole_Pad")
 		(at 64.77 158.75 0)
 		(unit 1)
@@
 			)
 		)
-		(property "Footprint" "MountingHole:MountingHole_3.2mm_M3_Pad"
+		(property "Footprint" "CLOCK_CORE:MountingHole_3.2mm_M3_Pad"
 			(at 64.77 158.75 0)
 			(hide yes)
