File: hardware/schematic/v1.0/CLOCK_CORE/_restore_backup_2026-09-12T13-45-48-352/CLOCK_CORE.kicad_pcb (KiCad board)
At the start: 2 copper layers, 70 x 60 mm, 117 parts, among them CN1 LAIL-PHC2_54-2P-01-XH-L, J1 Conn_Coaxial, J3 Conn_01x04_Socket, U1 OCXO_20x20mm, U2 OCXO_25.4x25.4mm, U3 TPS7A5201RPSR, U4 TPS7A5201RPSR, U5 LMK5B12204

Commit message: sch and pcb update
Parts:
- removed H2, H3, H4, H5: MountingHole_Pad, MountingHole:MountingHole_3.2mm_M3_Pad
- removed RF10: KH-IPEX-K501-29, JLCImport:KH-IPEX-K501-29
- added J2: Conn_Coaxial, Connector_Coaxial:SMA_Amphenol_132289_EdgeMount, F.Cu at (175.0, 69.2)
- TP2: footprint TestPoint:TestPoint_Pad_D1.0mm -> TestPoint:TestPoint_Loop_D1.80mm_Drill1.0mm_Beaded
- moved RF8 66.0 mm to (140.5, 90.6), turned to 0 degrees
- moved RF7 65.4 mm to (140.5, 85.6), turned to 0 degrees
- moved RF9 64.9 mm to (142.8, 70.4)
- moved J1 64.9 mm to (135.6, 70.4)
- moved R11 63.1 mm to (144.4, 103.0), turned to 0 degrees
- moved R10 62.7 mm to (144.4, 101.0), turned to 0 degrees
- moved R7 61.6 mm to (141.5, 103.0), turned to 0 degrees
- moved R8 60.9 mm to (141.5, 105.0), turned to 0 degrees
- moved R9 59.0 mm to (144.4, 99.0), turned to 0 degrees
- moved R12 58.3 mm to (144.4, 105.0), turned to 0 degrees
- moved RF5 57.7 mm to (135.4, 90.6), turned to 0 degrees
- moved RF6 57.7 mm to (135.4, 95.5), turned to 0 degrees
- moved J3 57.3 mm to (109.3, 121.2), turned to 90 degrees
- moved R13 45.9 mm to (131.6, 76.5), turned to 0 degrees
- moved C16 44.9 mm to (81.3, 114.0)
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