File: hardware/schematic/v1.0/CLOCK_CORE/_restore_backup_2026-09-12T13-45-48-352/OCXO.kicad_sch (KiCad schematic)
At the start: 13 parts, among them U1 OCXO_20x20mm, U2 OCXO_25.4x25.4mm

Commit message: sch and pcb update
Parts:
- removed RF10: KH-IPEX-K501-29, JLCImport:KH-IPEX-K501-29, symbol JLCImport:KH-IPEX-K501-29
- added J2: Conn_Coaxial, Connector_Coaxial:SMA_Amphenol_132289_EdgeMount, symbol Connector:Conn_Coaxial
- TP2: footprint TestPoint:TestPoint_Pad_D1.0mm -> TestPoint:TestPoint_Loop_D1.80mm_Drill1.0mm_Beaded
Connections:
- net GND: now also J2.2 (Ext)
- net at C9.1: now also J2.1 (In)
