File: hardware/schematic/v1.0/CLOCK_CORE/_restore_backup_2026-09-12T15-52-04-893/CLOCK_CORE.kicad_pcb (KiCad board)
At the start: 2 copper layers, 70 x 60 mm, 117 parts, among them CN1 LAIL-PHC2_54-2P-01-XH-L, J1 Conn_Coaxial, J3 Conn_01x04_Socket, U1 OCXO_20x20mm, U2 OCXO_25.4x25.4mm, U3 TPS7A5201RPSR, U4 TPS7A5201RPSR, U5 LMK5B12204

Commit message: sch and pcb update
Parts:
- moved C35 84.9 mm to (151.4, 162.9), turned to 90 degrees
- moved C36 79.6 mm to (153.4, 162.9), turned to 90 degrees
- moved C43 79.3 mm to (151.4, 160.1), turned to 90 degrees
- moved C44 69.0 mm to (153.4, 160.1), turned to 90 degrees
- moved D1 63.8 mm to (118.6, 173.2)
- moved D2 60.0 mm to (118.6, 170.8)
- moved H1 56.5 mm to (130.4, 173.7)
- moved C52 54.0 mm to (123.2, 165.6)
- moved C51 53.9 mm to (122.3, 164.7)
- moved C27 53.6 mm to (121.3, 163.6)
- moved FB1 53.5 mm to (131.5, 164.6), turned to 0 degrees
- moved C48 53.1 mm to (119.5, 161.6)
- moved C49 53.1 mm to (114.0, 158.4)
- moved C50 53.1 mm to (117.1, 157.8)
- moved C55 53.1 mm to (118.8, 157.8)
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